File: mini48-stm32/can_brd_1.sch (KiCad schematic (older format))
At the start: 7 parts, among them P201 CONN_4, P202 JUMPER, U201 SN65HVD230

Commit message: lib path
Parts:
- C201: symbol C -> Device:C
- C202: symbol CP1 -> Device:CP1
- P202: symbol JUMPER -> Device:Jumper
- R201, R202: symbol R -> Device:R
- U201: symbol SN65HVD230 -> art-electro-ic:SN65HVD230
Changed lines of the file:
@@
-EESchema Schematic File Version 2
-LIBS:power
-LIBS:device
-LIBS:conn
-LIBS:linear
-LIBS:regul
-LIBS:art-electro-stm32
-LIBS:art-electro-ic
-LIBS:art-electro-power
-LIBS:transistors
-LIBS:art-electro-conn
-LIBS:mini48-stm32-cache
-EELAYER 27 0
+EESchema Schematic File Version 4
+EELAYER 30 0
 EELAYER END
 $Descr A4 11693 8268
@@
 $EndDescr
 $Comp
-L CP1 C202
+L Device:CP1 C202
 U 1 1 52CAD8F6
 P 3550 3250
@@
 $EndComp
 $Comp
-L C C201
+L Device:C C201
 U 1 1 52CAD8F7
 P 3550 2700
@@
 $EndComp
 $Comp
-L GND #PWR033
+L power:GND #PWR033
 U 1 1 52CAD8F8
 P 3550 3450
@@
 $EndComp
 $Comp
-L GND #PWR034
+L power:GND #PWR034
 U 1 1 52CAD8F9
 P 3550 2500
@@
 $EndComp
 $Comp
-L GND #PWR035
+L power:GND #PWR035
 U 1 1 52CADB40
 P 4950 2500
@@
 NoConn ~ 4900 1200
 $Comp
-L R R201
+L Device:R R201
 U 1 1 52CADB46
 P 4000 1850
@@
 $EndComp
 $Comp
-L GND #PWR036
+L power:GND #PWR036
 U 1 1 52CADB51
 P 3750 1850
@@
 $EndComp
 $Comp
-L GND #PWR037
+L power:GND #PWR037
 U 1 1 52CADB3B
 P 2200 1650
@@
 	5050 1200 5050 1100
 $Comp
-L SN65HVD230 U201
+L art-electro-ic:SN65HVD230 U201
 U 1 1 52CD2CA4
 P 4800 1850
@@
 $EndComp
 $Comp
-L R R202
+L Device:R R202
 U 1 1 52CD2DE2
 P 5975 2625
@@
 $EndComp
 $Comp
-L JUMPER P202
+L Device:Jumper P202
 U 1 1 52CD2DEF
 P 6650 2625
@@
 CANH
 $Comp
-L GND #PWR038
+L power:GND #PWR038
 U 1 1 54959C55
 P 6350 3300
