File: mini48-stm32/can_brd_1.sch (KiCad schematic (older format))
At the start: 7 parts, among them P201 CONN_4, P202 JUMPER, U201 SN65HVD230

Commit message: progress
Parts:
- C201: footprint SM0805 -> Capacitor_SMD:C_0805_2012Metric; JLC PN (none) -> C111492; MPN (none) -> CC0805JRX7R9BB104
- C202: footprint SM0805 -> Capacitor_SMD:C_0805_2012Metric; JLC PN (none) -> C123621; MPN (none) -> 0805B472K500CT
- P201: symbol CONN_4 -> Connector_Generic:Conn_01x04; JLC PN (none) -> DNP
- P202: JLC PN (none) -> DNP
- R201: footprint SM0805 -> Resistor_SMD:R_0805_2012Metric; JLC PN (none) -> C212284; MPN (none) -> RMS10FT1002
- R202: footprint SM0805 -> Resistor_SMD:R_0805_2012Metric; JLC PN (none) -> C149652; MPN (none) -> CRH0805J120RP05Z
- U201: footprint SO8E -> Package_SO:SO-8_3.9x4.9mm_P1.27mm; symbol art-electro-ic:SN65HVD230 -> mini48-stm32-rescue:SN65HVD230-art-electro-ic; JLC PN (none) -> C12084; MPN (none) -> SN65HVD230DR
Connections:
- wire segments 17 -> 18
Other:
- moved on the sheet: C201, C202, P202, R201, R202, U201
