File: mini48-stm32/mini48-stm32.sch (KiCad schematic (older format))
At the start: 29 parts, among them J1 MINI-USB, P1 CONN_20, P2 CONN_20, U1 STM32F103C8, U2 NUF2101MT1G, U3 LM2937, X1 8MHz, X2 32768KHz

Commit message: lib path
Parts:
- C1, C10, C11, C12, C2, C3, C4, C5, C6, C7, C9: symbol C -> Device:C
- C8: symbol CP1 -> Device:CP1
- D1, D4: symbol LED_0805 -> art-electro-conn:LED_0805
- J1: symbol MINI-USB -> art-electro-conn:MINI-USB
- R1, R2, R3, R6, R7: symbol R -> Device:R
- U1: symbol STM32F103C8 -> art-electro-stm32:STM32F103C8
- U2: symbol NUF2101MT1G -> art-electro-ic:NUF2101MT1G
- U3: symbol LM2937 -> art-electro-power:LM2937
- X1, X2: symbol CRYSTAL -> Device:Crystal
Connections:
- wire segments 130 -> 133
