File: mini48-stm32/mini48-stm32.sch (KiCad schematic (older format))
At the start: 29 parts, among them J1 MINI-USB, P1 CONN_20, P2 CONN_20, U1 STM32F103C8, U2 NUF2101MT1G, U3 LM2937, X1 8MHz, X2 32768KHz

Commit message: progress
Parts:
- removed P1, P2: CONN_20, PIN_ARRAY_20X1, symbol CONN_20
- added J2, J3: Conn_01x20, mini48-stm32:PIN_ARRAY_20X1, symbol Connector_Generic:Conn_01x20
- added J4: Conn_02x03_Odd_Even, Connector:Tag-Connect_TC2030-IDC-NL_2x03_P1.27mm_Vertical, symbol Connector_Generic:Conn_02x03_Odd_Even
- C1: footprint SM0805 -> Capacitor_SMD:C_0805_2012Metric; JLC PN (none) -> C123621; MPN (none) -> 0805B472K500CT
- C10, C11, C7: footprint SM0805 -> Capacitor_SMD:C_0805_2012Metric; JLC PN (none) -> C106838; MPN (none) -> CC0805ZKY5V9BB105
- C12: footprint SM0805 -> Capacitor_SMD:C_0805_2012Metric; JLC PN (none) -> C117956; MPN (none) -> GRM21BR71A106KA73L
- C2, C3: footprint SM0805 -> Capacitor_SMD:C_0805_2012Metric; JLC PN (none) -> C113825; MPN (none) -> CC0805JRNPO9BN180
- C4, C5: value 18pF -> 12pF; footprint SM0805 -> Capacitor_SMD:C_0805_2012Metric; JLC PN (none) -> C0805; MPN (none) -> CC0805JRNPO9BN120
- C6, C9: footprint SM0805 -> Capacitor_SMD:C_0805_2012Metric; JLC PN (none) -> C111492; MPN (none) -> CC0805JRX7R9BB104
- C8: footprint CP_elec_4x5.3 -> Capacitor_SMD:CP_Elec_4x5.3; JLC PN (none) -> C124129; MPN (none) -> GRM21BR61A476ME15L
- D1: symbol art-electro-conn:LED_0805 -> mini48-stm32-rescue:LED_0805-art-electro-conn; JLC PN (none) -> C693904; MPN (none) -> MHS171UGCT
- D2, D3: footprint SM0805-diode -> Diode_SMD:D_SOD-123; symbol DIODESCH -> Device:D_Schottky; JLC PN (none) -> C82288; MPN (none) -> PMEG2010ER,115
- D4: symbol art-electro-conn:LED_0805 -> mini48-stm32-rescue:LED_0805-art-electro-conn; JLC PN (none) -> C99870; MPN (none) -> 17-21/BHC-AP1Q2/3T
- J1: symbol art-electro-conn:MINI-USB -> mini48-stm32-rescue:MINI-USB-art-electro-conn; JLC PN (none) -> C2681563; MPN (none) -> MINI 5PTP
- R1, R3, R7: footprint SM0805 -> Resistor_SMD:R_0805_2012Metric; JLC PN (none) -> C218388; MPN (none) -> ARG05FTC1001
- R2: footprint SM0805 -> Resistor_SMD:R_0805_2012Metric; JLC PN (none) -> C230655; MPN (none) -> ERJ6GEYJ105V
- R6: footprint SM0805 -> Resistor_SMD:R_0805_2012Metric; JLC PN (none) -> C212284; MPN (none) -> RMS10FT1002
- U1: footprint lqfp48 -> Package_QFP:LQFP-48_7x7mm_P0.5mm; symbol art-electro-stm32:STM32F103C8 -> mini48-stm32-rescue:STM32F103C8-art-electro-stm32; JLC PN (none) -> C8734; MPN (none) -> STM32F103C8T6
- U2: symbol art-electro-ic:NUF2101MT1G -> mini48-stm32-rescue:NUF2101MT1G-art-electro-ic; JLC PN (none) -> C2827654; MPN (none) -> USBLC6-2SC6
- U3: footprint SOT223 -> Package_TO_SOT_SMD:SOT-223; symbol art-electro-power:LM2937 -> mini48-stm32-rescue:LM2937-art-electro-power; JLC PN (none) -> C140265; MPN (none) -> LM2937IMP-3.3/NOPB
- X1: JLC PN (none) -> C111806; MPN (none) -> E49A8E00000FE10CO
- X2: value 32768KHz -> 32.768KHz; footprint MC-306 -> mini48-stm32:SMD2012; JLC PN (none) -> C280831; MPN (none) -> NX2012SA-32.768KHz-EXS00A-MU00311
Connections:
- net labels added: PA13,TMS, PA14,TSK, PA15,TDI, PB3,TDO, PB4,NTRST
- net labels removed: PA13, PA14, PA15, PB3, PB4
- wire segments 133 -> 158
Other:
- moved on the sheet: C12, C2, C3, C6, C7, D4, R1, R6, R7, U1, U3, X1

Commit message: progress
Parts:
- U2: footprint SOT-457 -> Package_TO_SOT_SMD:SOT-23-6
- X1: footprint HC-49V -> Crystal:Crystal_SMD_HC49-SD; JLC PN C111806 -> C106809; MPN E49A8E00000FE10CO -> X49SM8MSD2SI
- X2: footprint mini48-stm32:SMD2012 -> mini48-stm32:SMD2012-2P; JLC PN C280831 -> C515343; MPN NX2012SA-32.768KHz-EXS00A-MU00311 -> TFX-03-32.768K
Changed lines of the file:
@@
 F 0 "X2" H 1525 5250 60  0000 C CNN
 F 1 "32.768KHz" H 1525 4950 60  0000 C CNN
-F 2 "mini48-stm32:SMD2012" H 1525 5100 60  0001 C CNN
+F 2 "mini48-stm32:SMD2012-2P" H 1525 5100 60  0001 C CNN
 F 3 "~" H 1525 5100 60  0000 C CNN
-F 4 "C280831" H 1525 5100 50  0001 C CNN "JLC PN"
-F 5 "NX2012SA-32.768KHz-EXS00A-MU00311" H 1525 5100 50  0001 C CNN "MPN"
+F 4 "C515343" H 1525 5100 50  0001 C CNN "JLC PN"
+F 5 "TFX-03-32.768K" H 1525 5100 50  0001 C CNN "MPN"
 	1    1525 5100
 	0    1    1    0
@@
 F 0 "X1" H 1675 2150 60  0000 C CNN
 F 1 "8MHz" H 1675 1850 60  0000 C CNN
-F 2 "HC-49V" H 1675 2000 60  0001 C CNN
+F 2 "Crystal:Crystal_SMD_HC49-SD" H 1675 2000 60  0001 C CNN
 F 3 "~" H 1675 2000 60  0000 C CNN
-F 4 "C111806" H 1675 2000 50  0001 C CNN "JLC PN"
-F 5 "E49A8E00000FE10CO" H 1675 2000 50  0001 C CNN "MPN"
+F 4 "C106809" H 1675 2000 50  0001 C CNN "JLC PN"
+F 5 "X49SM8MSD2SI" H 1675 2000 50  0001 C CNN "MPN"
 	1    1675 2000
 	0    1    1    0
@@
 F 0 "U2" H 4175 7450 70  0000 C CNN
 F 1 "NUF2101MT1G" H 4075 6650 70  0000 C CNN
-F 2 "SOT-457" H 4075 7050 60  0001 C CNN
+F 2 "Package_TO_SOT_SMD:SOT-23-6" H 4075 7050 60  0001 C CNN
 F 3 "~" H 4075 7050 60  0000 C CNN
 F 4 "C2827654" H 4075 7050 50  0001 C CNN "JLC PN"
