File: mini48-stm32/mini48-stm32.kicad_pcb (KiCad board)
At the start: 2 copper layers, 78.9 x 19.8 mm, 36 parts, among them J1 MINI-USB, P1 CONN_20, P2 CONN_20, P201 CONN_4, P202 JUMPER, U1 STM32F103C8, U2 NUF2101MT1G, U201 SN65HVD230, U3 LM2937, X1 8MHz, X2 32768KHz

Commit message: progress
Parts:
- removed P1, P2: CONN_20, PIN_ARRAY_20X1
- added J2: Conn_01x20, mini48-stm32:PIN_ARRAY_20X1, F.Cu at (136.4, 96.5)
- added J3: Conn_01x20, mini48-stm32:PIN_ARRAY_20X1, F.Cu at (136.4, 81.3)
- added J4: Conn_02x03_Odd_Even, Connector:Tag-Connect_TC2030-IDC-NL_2x03_P1.27mm_Vertical, F.Cu at (148.8, 84.7)
- C1, C10, C11, C12, C2, C201, C202, C3, C6, C7, C9: footprint SM0805 -> Capacitor_SMD:C_0805_2012Metric
- C4, C5: footprint SM0805 -> Capacitor_SMD:C_0805_2012Metric; moved to F.Cu
- C8: footprint CP_elec_4x5.3 -> Capacitor_SMD:CP_Elec_4x5.3
- D2, D3: footprint SM0805-diode -> Diode_SMD:D_SOD-123
- R1, R2, R201, R202, R3, R6, R7: footprint SM0805 -> Resistor_SMD:R_0805_2012Metric
- U1: footprint lqfp48 -> Package_QFP:LQFP-48_7x7mm_P0.5mm
- U201: footprint SO8E -> Package_SO:SO-8_3.9x4.9mm_P1.27mm
- U3: footprint SOT223 -> Package_TO_SOT_SMD:SOT-223
- X2: value 32768KHz -> 32.768KHz; footprint MC-306 -> mini48-stm32:SMD2012; moved to F.Cu
- moved C9 27.6 mm to (156.7, 92.8), turned to 270 degrees
- moved C11 9.63 mm to (160.7, 92.8), turned to 270 degrees
- moved R7 9.43 mm to (115.8, 92.7), turned to 90 degrees
- moved C6 9.12 mm to (113.8, 92.7), turned to 270 degrees
- moved R1 8.89 mm to (111.8, 92.7), turned to 90 degrees
- moved C4 7.79 mm to (126.0, 94.0), turned to 0 degrees
- moved D4 6.87 mm to (114.8, 89.9)
- moved C5 5.92 mm to (126.0, 91.9), turned to 0 degrees
- moved R6 3.12 mm to (116.3, 83.6)
- moved X2 3.10 mm to (128.8, 93.5), turned to 90 degrees
- moved R202 1.72 mm to (177.3, 83.0)
- moved C10 1.34 mm to (158.7, 92.8), turned to 270 degrees
- moved D1 1.27 mm to (183.3, 95.6)
- moved C201 1.22 mm to (167.7, 83.6)
- moved U201 1.20 mm to (172.5, 84.0), turned to 0 degrees
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Connections:
- net /CAN BUS/3.3V renamed /VCC
- net /CAN BUS/CANH renamed /CANH
- net /CAN BUS/CANL renamed /CANL
- net /CAN BUS/CAN_RX renamed /CANRX
- net /CAN BUS/CAN_TX renamed /CANTX
- C12 pad 1: N-0000016 -> Net-(C12-Pad1)
- D2 pad 1: /VIN -> Net-(C12-Pad1)
- D2 pad 2: N-0000016 -> /VIN
- D3 pad 1: /CAN BUS/5V -> Net-(C12-Pad1)
- D3 pad 2: N-0000016 -> /+5v
- J1 pad 1: /CAN BUS/5V -> /+5v
- P201 pad 1: /CAN BUS/5V -> /+5v
- R3 pad 1: /CAN BUS/5V -> /+5v
- U1 pad 34: /PA13 -> /PA13,TMS
- U1 pad 37: /PA14 -> /PA14,TSK
- U1 pad 38: /PA15 -> /PA15,TDI
- U1 pad 39: /PB3 -> /PB3,TDO
- U1 pad 40: /PB4 -> /PB4,NTRST
- U2 pad 5: /CAN BUS/5V -> /+5v
- U3 pad 1: N-0000016 -> Net-(C12-Pad1)
Routing:
- net GND: track 129.8 -> 45.2 mm, vias 29 -> 41
- net /PB4,NTRST: track 0.00 -> 26.0 mm, vias 0 -> 2
- net /PB3,TDO: track 0.00 -> 24.7 mm, vias 0 -> 2
- net /VCC: track 150.7 -> 131.7 mm, vias 0 -> 4
- net /PA14,TSK: track 0.00 -> 18.3 mm, vias 0 -> 2
- net /CAN BUS/5V: track 16.8 -> 0.00 mm
- net /+5v: track 0.00 -> 16.1 mm
- net /PA13,TMS: track 0.00 -> 13.4 mm, vias 0 -> 2
- net N-0000016: track 13.3 -> 0.00 mm
- net Net-(C12-Pad1): track 0.00 -> 11.1 mm
- net /PB4: track 8.46 -> 0.00 mm
- net /Reset: track 35.1 -> 28.1 mm, vias 1 -> 0
- net /PB3: track 6.13 -> 0.00 mm
- net /PC15_OSC32_OUT: track 12.7 -> 6.90 mm, vias 1 -> 0
- net /PA13: track 4.22 -> 0.00 mm
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Other:
- rule via_min_drill: 0.508 -> 0.3
- rule via_min_size: 0.889 -> 0.6
- board text added: "rev 0.3"
- board text removed: "3V3 GND VBAT RESET PA1 PA4 PA5 PA6 PA7 PB0 PB2 PB10 PB11 VIN"
- board text removed: "PB7 PB5 PB4 PB3 PA15 PA12 USBDP PA11 USBDM PA10 PA9 PA8 PA15 PA14 PB13 PB12"
- board text removed: "rev 0.2"

Commit message: progress
Other:
- board size 78.9 x 19.8 mm -> 78.9 x 20.3 mm
Changed lines of the file:
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@@
   )
   (setup
-    (last_trace_width 0.254)
+    (last_trace_width 0.1524)
     (user_trace_width 0.254)
     (user_trace_width 0.508)
@@
     (effects (font (size 1.016 1.016) (thickness 0.2032)) (justify left mirror))
   )
-  (gr_line (start 109.474 98.806) (end 109.474 78.994) (angle 90) (layer Edge.Cuts) (width 0.15))
-  (gr_line (start 188.341 98.806) (end 109.474 98.806) (angle 90) (layer Edge.Cuts) (width 0.15))
-  (gr_line (start 188.341 78.994) (end 188.341 98.806) (angle 90) (layer Edge.Cuts) (width 0.15))
-  (gr_line (start 109.474 78.994) (end 188.341 78.994) (angle 90) (layer Edge.Cuts) (width 0.15))
+  (gr_line (start 109.474 98.9) (end 109.474 78.6) (angle 90) (layer Edge.Cuts) (width 0.15))
+  (gr_line (start 188.341 98.9) (end 109.474 98.9) (angle 90) (layer Edge.Cuts) (width 0.15))
+  (gr_line (start 188.341 78.6) (end 188.341 98.9) (angle 90) (layer Edge.Cuts) (width 0.15))
+  (gr_line (start 109.474 78.6) (end 188.341 78.6) (angle 90) (layer Edge.Cuts) (width 0.15))
   (via (at 131.8274 85.7486) (size 0.6) (drill 0.3) (layers F.Cu B.Cu) (net 1))
   (segment (start 131.8274 85.7487) (end 131.8274 85.7486) (width 0.254) (layer F.Cu) (net 1))

Commit message: progress
Parts:
- C4, C5: value 18pF -> 12pF
- U2: footprint SOT-457 -> Package_TO_SOT_SMD:SOT-23-6
- X1: footprint HC-49V -> Crystal:Crystal_SMD_HC49-SD
- X2: footprint mini48-stm32:SMD2012 -> mini48-stm32:SMD2012-2P
- moved C3 8.16 mm to (122.4, 92.5), turned to 90 degrees
- moved D4 1.42 mm to (113.7, 89.1), turned to 90 degrees
- moved X1 1.00 mm to (121.6, 87.9)
- moved C2 0.74 mm to (118.8, 92.5), turned to 90 degrees
- moved X2 0.68 mm to (128.9, 92.8)
- turned U2 to 0 degrees
Routing:
- net /VCC: track 131.7 -> 134.3 mm
- net GND: track 45.2 -> 43.7 mm, vias 41 -> 42
- net /PD1: track 18.0 -> 16.8 mm, vias 1 -> 2
- net Net-(D4-Pad1): track 1.87 -> 2.99 mm
- net /VBAT: track 17.8 -> 16.9 mm
- net /PD0: track 19.5 -> 20.0 mm, vias 1 -> 2
