File: mini48-stm32/mini48-stm32.kicad_sch (KiCad schematic)
At the start: 30 parts, among them J1 MINI-USB, J2 Conn_01x20, J3 Conn_01x20, J4 Conn_02x03_Odd_Even, U1 STM32F103C8, U2 NUF2101MT1G, U3 LM2937, X1 8MHz, X2 32768KHz

Commit message: #273 X2 and #272 kiCad 7.0
Parts:
- X2: value 32768KHz -> 32.768KHz
