File: GDI-4ch/GDI-4ch.kicad_pcb (KiCad board)
At the start: 4 copper layers, 380.4 x 234.8 mm, 165 parts, among them J14 CONN_01X03, J15 CONN_01X01, J3 CONN_02X08, J4 CONN_02X08, J7 CONN_01X03, P1 368255-2, Q1 BUK9230-100B, Q10 BUK9230-100B, Q11 BUK9230-100B, Q12 BUK9230-100B, Q2 BUK9230-100B, Q3 BUK9230-100B, Q4 BUK9230-100B, Q5 BUK9230-100B, Q6 BUK9230-100B, Q7 BUK9230-100B, Q8 BUK9230-100B, Q9 BUK9230-100B, U1 MC33816, Y2 1MHz

Commit message: UPD sch
Parts:
- removed C1: 100nF, Capacitor_SMD:C_0603_1608Metric
- removed C10, C11, C13, C8: 0.1uF, rusefi_lib:C_0805
- removed C12: 4.7uF, rusefi_lib:C_0805
- removed C14, C15: 1000uF, Capacitors_ThroughHole:CP_Radial_D22.0mm_P10.00mm_SnapIn
- removed C16, C17: 220nF, rusefi_lib:C_0805
- removed C19, C35, C36, C37, C38, C55, C56, C57, C58, C63, C71: 1000pF, rusefi_lib:C_0805
- removed C21, C22: 390uF, Capacitors_ThroughHole:CP_Radial_D16.0mm_P7.50mm
- removed C23, C24, C28, C59, C60, C73: 330pF, rusefi_lib:C_0805
- removed C25, C27: 0.22uF, rusefi_lib:C_0805
- removed C26: 470pF, rusefi_lib:C_0805
- removed C39, C40, C41, C42, C64: 0.33uF, rusefi_lib:C_0805
- removed C43, C44, C45, C46, C47, C48, C49, C50, C65, C67: 4700pF, rusefi_lib:C_0805
- removed C9: 1uF, rusefi_lib:C_0805
- removed D1, D18, D19, D2, D20, D21, D22, D23, D24, D25, D26, D27, D28, D29, D3, D31, D32, D33, D4, D5, D6, D7, D8: LED_Small, LED_SMD:LED_0805_2012Metric
- removed D10, D11: SBR10200CTL, Package_TO_SOT_SMD:TO-252-2
- removed D12, D13, D14, D15, D16, D17: STPS2H100UY, Diodes_SMD:D_SMB
- removed D30, D35, D36, D37, D38: 5.7V, Diode_SMD:D_MicroMELF_Handsoldering
- removed D34: STTH802G-TR, Package_TO_SOT_SMD:TO-263-2
- removed D9: FFD10UP20S, Package_TO_SOT_SMD:TO-252-2
- removed J14, J7: CONN_01X03, Pin_Headers:Pin_Header_Straight_1x03_Pitch2.54mm
- removed J15: CONN_01X01, Connector_Pin:Pin_D1.4mm_L8.5mm_W2.8mm_FlatFork
- removed J3, J4: CONN_02X08, Pin_Headers:Pin_Header_Straight_2x08_Pitch2.54mm
- removed L1: 6uH, rusefi_lib:744710610-Inductor
- removed L2: 10uH, rusefi_lib:IHLP6767GZER100M01
- removed Q1, Q10, Q11, Q12, Q2, Q3, Q4, Q5, Q6, Q7, Q8, Q9: BUK9230-100B, Package_TO_SOT_SMD:TO-252-2
- removed R1, R2, R25, R27, R28, R29, R3, R30, R31, R32, R33, R34, R35, R36, R37, R39, R4, R40, R5, R6, R7, R8: 1k, rusefi_lib:R_0805
- removed R10, R9: 5.1R, rusefi_lib:R_0805
- removed R11, R13, R14, R15, R16, R17, R18, R19, R20, R23, R24, R41: 10R, rusefi_lib:R_0805
- removed R12, R21, R22, R26: 0R010, Resistors_SMD:R_1206_HandSoldering
- removed R38, R44: 10k, Resistor_SMD:R_0603_1608Metric
- removed R42: 1k, Resistor_SMD:R_0805_2012Metric
- removed R43, R45: 0R010, Resistor_SMD:R_1206_3216Metric_Pad1.42x1.75mm_HandSolder
- removed TP101, TP102, TP103, TP104, TP23, TP24, TP3, TP4, TP5, TP6, TP7, TP8: CONN_01X01, Connector_Pin:Pin_D0.7mm_L6.5mm_W1.8mm_FlatFork
- removed U1: MC33816, Package_QFP:LQFP-64-1EP_10x10mm_P0.5mm_EP5x5mm_ThermalVias
- removed Y2: 1MHz, Oscillator:Oscillator_SMD_Diodes_FN-4Pin_7.0x5.0mm
Routing:
- net Vdrive: track 290.7 -> 0.00 mm, vias 5 -> 0
- net Net-(C21-Pad2): track 230.5 -> 0.00 mm, vias 6 -> 0
- net +BATT: track 214.0 -> 0.00 mm, vias 1 -> 0
- net /5V: track 177.0 -> 0.00 mm, vias 2 -> 0
- net GND: track 164.4 -> 0.00 mm, vias 277 -> 31
- net /H3: track 163.3 -> 0.00 mm, vias 2 -> 0
- net /H1: track 152.4 -> 0.00 mm, vias 3 -> 0
- net /H_PUMP: track 139.4 -> 0.00 mm, vias 2 -> 0
- net /L_PUMP: track 130.7 -> 0.00 mm, vias 2 -> 0
- net /L4: track 114.0 -> 0.00 mm, vias 2 -> 0
- net Net-(C37-Pad2): track 108.2 -> 0.00 mm, vias 3 -> 0
- net Net-(C71-Pad2): track 108.0 -> 0.00 mm, vias 1 -> 0
- net Net-(C35-Pad2): track 99.8 -> 0.00 mm
- net Net-(C60-Pad1): track 98.0 -> 0.00 mm, vias 2 -> 0
- net Net-(C10-Pad1): track 96.9 -> 0.00 mm
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- removed copper zone on B.Cu, net GND
- removed copper zone on F.Cu, net GND
- removed copper zone on In1.Cu, net GND
- removed copper zone on In2.Cu, net GND
Other:
- board size 380.4 x 234.8 mm -> 164 x 118 mm
- board text removed: "0"
- board text removed: "1"
- board text removed: "3"
- board text removed: "3.3V"
- board text removed: "4"
- board text removed: "4 layer board stackup is as follows: 0 is top min 1 oz copper (1.4 mil) min 6.7 mil prepreg FR4 1 is GND min 0.5 oz copper (0.7 mil) min 47 mil core FR4 2 is PWR min 0.5 oz copper (0.7 mil) min 6.7 mil prepreg FR4 3 is bottom min 1 oz copper (1.4 mil)"
- board text removed: "5V"
- board text removed: "CBS"
- board text removed: "CLK"
- board text removed: "CSB"
- board text removed: "DBG"
- board text removed: "DRIVEN"
- board text removed: "DRVEN"
- board text removed: "ECLK"
- board text removed: "EXT"
- board text removed: "EXT-CLK"
- board text removed: "EXT-DBG"
- board text removed: "EXT1"
- board text removed: "EXT2"
- board text removed: "FLAG-0"
- board text removed: "FLAG-1"
- board text removed: "FLAG-2"
- board text removed: "FLAG0"
- board text removed: "FLAG1"
- board text removed: "FLAG2"
- board text removed: "GND"
- board text removed: "HI LOW"
- board text removed: "INJ1 B1"
- board text removed: "INJ2 B1"
- board text removed: "INJ3 B2"
- board text removed: "INJ4 B2"
- board text removed: "IRQB"
- board text removed: "MC33816 for rusEFI.com R0.3.3"
- board text removed: "MISO"
- board text removed: "MOSI"
- board text removed: "NC"
- board text removed: "OA_1"
- board text removed: "OA_2"
- board text removed: "PUMP"
- board text removed: "RESETB"
- board text removed: "RSTB"
- board text removed: "SCLK"
- board text removed: "STAR1"
- board text removed: "STAR2"
- board text removed: "STAR3"
- board text removed: "STAR4"
- board text removed: "STAR5"
- board text removed: "STAR6"
- board text removed: "START1"
- board text removed: "START2"
- board text removed: "START3"
- board text removed: "START4"
- board text removed: "START5"
- board text removed: "START6"
- board text removed: "VBAT"
- board text removed: "VBAT-EXT"
- board text removed: "VCCIO"
- board text removed: "VCCP"
- board text removed: "VPWR"
- board text removed: "Vbat"
- board text removed: "Vboost"
- board text removed: "Y1-3"

Commit message: Upd PCB
Parts:
- added C1: 100n, hellen-one-common:C0603, F.Cu at (-8.09, 108.7)
- added C10: 330p, hellen-one-common:C0603, F.Cu at (112.0, 120.8)
- added C11: 330p, hellen-one-common:C0603, F.Cu at (113.8, 122.2)
- added C12: 4.7u, hellen-one-common:C0603, F.Cu at (-29.0, 128.3)
- added C13: 330p, hellen-one-common:C0603, F.Cu at (115.5, 120.8)
- added C14: 390uF, Capacitor_SMD:CP_Elec_16x17.5, F.Cu at (213.5, 119.0)
- added C15: 390uF, Capacitor_SMD:CP_Elec_16x17.5, F.Cu at (213.5, 100.2)
- added C16: 390uF, Capacitor_SMD:CP_Elec_16x17.5, F.Cu at (213.5, 81.5)
- added C17: 0.22uF, Capacitor_SMD:C_0805_2012Metric, F.Cu at (14.4, 69.0)
- added C18: 1000pF, Capacitor_SMD:C_0603_1608Metric, F.Cu at (29.2, 61.8)
- added C19: 1000pF, Capacitor_SMD:C_0603_1608Metric, F.Cu at (-85.6, 123.5)
- added C2: 47p, Capacitor_SMD:C_0402_1005Metric, F.Cu at (43.7, 57.0)
- added C20: 100n, Capacitor_SMD:C_0402_1005Metric, F.Cu at (0.16, 100.8)
- added C21: 390uF, Capacitor_SMD:CP_Elec_16x17.5, F.Cu at (175.5, 118.5)
- added C22: 390uF, Capacitor_SMD:CP_Elec_16x17.5, F.Cu at (193.2, 107.0)
- added C23: 100n, hellen-one-common:C0603, F.Cu at (121.5, 113.8)
- added C24: 330p, hellen-one-common:C0603, F.Cu at (118.8, 120.0)
- added C25: 390uF, Capacitor_SMD:CP_Elec_16x17.5, F.Cu at (157.2, 118.5)
- added C26: 4.7u, hellen-one-common:C0603, F.Cu at (121.5, 111.2)
- added C27: 390uF, Capacitor_SMD:CP_Elec_16x17.5, F.Cu at (193.2, 84.8)
- added C28: 100n, hellen-one-common:C0603, F.Cu at (121.5, 112.5)
- added C29: 1000pF, Capacitor_SMD:C_0603_1608Metric, F.Cu at (-10.7, 94.0)
- added C3: 47p, Capacitor_SMD:C_0402_1005Metric, F.Cu at (-16.7, 118.5)
- added C30: 1000pF, Capacitor_SMD:C_0603_1608Metric, F.Cu at (-36.5, 124.0)
- added C31: 10u, Capacitor_SMD:C_0805_2012Metric, F.Cu at (212.5, 64.2)
- added C32: 100n, hellen-one-common:C0603, F.Cu at (108.5, 121.5)
- added C33: 10u, Capacitor_SMD:C_0805_2012Metric, F.Cu at (216.0, 68.4)
- added C34: 100n, hellen-one-common:C0603, F.Cu at (110.0, 121.5)
- added C35: 1000pF, Capacitor_SMD:C_0603_1608Metric, F.Cu at (13.6, 76.8)
- added C36: 1000pF, Capacitor_SMD:C_0603_1608Metric, F.Cu at (31.4, 56.8)
- added C37: 1000pF, Capacitor_SMD:C_0603_1608Metric, F.Cu at (-31.4, 118.5)
- added C38: 1000pF, Capacitor_SMD:C_0603_1608Metric, F.Cu at (-14.5, 102.6)
- added C39: 0.33uF, Capacitor_SMD:C_0603_1608Metric, F.Cu at (108.5, 103.5)
- added C4: 10u, Capacitor_SMD:C_0805_2012Metric, F.Cu at (212.6, 61.2)
- added C40: 0.33uF, Capacitor_SMD:C_0603_1608Metric, F.Cu at (112.5, 103.5)
- added C41: 0.33uF, Capacitor_SMD:C_0603_1608Metric, F.Cu at (110.5, 102.0)
- added C42: 0.33uF, Capacitor_SMD:C_0603_1608Metric, F.Cu at (114.5, 102.0)
- added C43: 4700p, hellen-one-common:C0603, F.Cu at (95.5, 54.5)
- added C44: 4700p, hellen-one-common:C0603, F.Cu at (91.5, 54.5)
- added C45: 4700p, hellen-one-common:C0603, F.Cu at (114.5, 54.5)
- added C46: 4700p, hellen-one-common:C0603, F.Cu at (110.5, 54.5)
- added C47: 4700p, hellen-one-common:C0603, F.Cu at (122.0, 54.5)
- added C48: 4700p, hellen-one-common:C0603, F.Cu at (118.3, 54.5)
- added C49: 4700p, hellen-one-common:C0603, F.Cu at (134.0, 54.5)
- added C5: 1000pF, Capacitor_SMD:C_0603_1608Metric, F.Cu at (-1.45, 88.2)
- added C50: 4700p, hellen-one-common:C0603, F.Cu at (126.0, 54.5)
- added C51: 1000pF, Capacitor_SMD:C_0603_1608Metric, F.Cu at (-19.4, 104.8)
- added C52: 1000pF, Capacitor_SMD:C_0603_1608Metric, F.Cu at (93.5, 70.0)
- added C53: 1000pF, Capacitor_SMD:C_0603_1608Metric, F.Cu at (89.0, 58.5)
- added C54: 1000pF, Capacitor_SMD:C_0603_1608Metric, F.Cu at (102.5, 80.0)
- added C55: 1000pF, Capacitor_SMD:C_0603_1608Metric, F.Cu at (98.5, 70.0)
- added C56: 1000pF, Capacitor_SMD:C_0603_1608Metric, F.Cu at (119.5, 68.5)
- added C57: 1000pF, Capacitor_SMD:C_0603_1608Metric, F.Cu at (108.7, 66.5)
- added C58: 1000pF, Capacitor_SMD:C_0603_1608Metric, F.Cu at (140.7, 78.0)
- added C59: 100n, hellen-one-common:C0603, F.Cu at (105.8, 121.5)
- added C6: 1000pF, Capacitor_SMD:C_0603_1608Metric, F.Cu at (-15.4, 105.1)
- added C60: 330p, hellen-one-common:C0603, F.Cu at (181.5, 103.8)
- added C61: 1000pF, Capacitor_SMD:C_0603_1608Metric, F.Cu at (127.0, 78.1)
- added C62: 1000pF, Capacitor_SMD:C_0603_1608Metric, F.Cu at (131.7, 66.5)
- added C63: 1000pF, Capacitor_SMD:C_0603_1608Metric, F.Cu at (148.0, 78.0)
- added C64: 0.33uF, Capacitor_SMD:C_0603_1608Metric, F.Cu at (116.5, 103.5)
- added C65: 4700p, hellen-one-common:C0603, F.Cu at (130.0, 54.5)
- added C66: 100nF, Capacitor_SMD:C_0402_1005Metric, F.Cu at (24.3, 76.7)
- added C67: 4700p, hellen-one-common:C0603, F.Cu at (138.0, 54.5)
- added C68: 10u, Capacitor_SMD:C_0805_2012Metric, F.Cu at (223.5, 68.4)
- added C69: 100nF, Capacitor_SMD:C_0402_1005Metric, F.Cu at (-20.7, 121.7)
- added C7: 1000pF, Capacitor_SMD:C_0603_1608Metric, F.Cu at (-12.7, 96.8)
- added C70: 100nF, Capacitor_SMD:C_0402_1005Metric, F.Cu at (13.6, 88.5)
- added C71: 1000pF, Capacitor_SMD:C_0603_1608Metric, F.Cu at (-46.5, 131.4)
- added C72: 100nF, Capacitor_SMD:C_0402_1005Metric, F.Cu at (-4.38, 106.5)
- added C73: 330p, hellen-one-common:C0603, F.Cu at (126.3, 130.5)
- added C74: 470p, hellen-one-common:C0603, F.Cu at (179.0, 101.0)
- added C75: 100n, hellen-one-common:C0603, F.Cu at (40.5, 58.4)
- added C76: 100n, hellen-one-common:C0603, F.Cu at (-3.55, 102.6)
- added C77: 100n, hellen-one-common:C0603, F.Cu at (-39.9, 133.6)
- added C78: 100n, hellen-one-common:C0603, F.Cu at (0.79, 98.8)
- added C79: 100n, hellen-one-common:C0603, F.Cu at (21.1, 78.2)
- added C8: 100n, hellen-one-common:C0603, F.Cu at (30.0, 69.7)
- added C80: 0.22uF, Capacitor_SMD:C_0805_2012Metric, F.Cu at (168.8, 105.5)
- added C81: 0.22uF, Capacitor_SMD:C_0805_2012Metric, F.Cu at (133.2, 130.0)
- added C82: 0.22uF, Capacitor_SMD:C_0805_2012Metric, F.Cu at (133.6, 125.0)
- added C83: 390uF, Capacitor_SMD:CP_Elec_16x17.5, F.Cu at (175.5, 84.8)
- added C9: 1u, hellen-one-common:C0603, F.Cu at (107.2, 121.5)
- added D1: SMCJ22CA, Diode_SMD:D_SMC, F.Cu at (219.5, 54.0)
- added D10: SBR10200CTL, Package_TO_SOT_SMD:TO-252-2, F.Cu at (93.5, 62.1)
- added D11: SBR10200CTL, Package_TO_SOT_SMD:TO-252-2, F.Cu at (118.0, 62.1)
- added D12: STPS2H100UY, Diode_SMD:D_SMB, F.Cu at (107.0, 60.5)
- added D13: STPS2H100UY, Diode_SMD:D_SMB, F.Cu at (134.0, 60.5)
- added D14: STPS2H100UY, Diode_SMD:D_SMB, F.Cu at (124.0, 60.5)
- added D15: STPS2H100UY, Diode_SMD:D_SMB, F.Cu at (129.0, 60.5)
- added D16: STPS2H100UY, Diode_SMD:D_SMB, F.Cu at (139.0, 60.5)
- added D18: SRV05-4, Package_TO_SOT_SMD:SOT-23-6, F.Cu at (28.0, 50.3)
- added D19: WHITE, LED_SMD:LED_0603_1608Metric, F.Cu at (227.0, 68.5)
- added D2: ZMM5V6, Diode_SMD:D_MiniMELF, F.Cu at (201.0, 58.8)
- added D20: BLUE, LED_SMD:LED_0603_1608Metric, F.Cu at (-98.1, 133.6)
- added D21: GREEN, LED_SMD:LED_0603_1608Metric, F.Cu at (-62.0, 101.0)
- added D28: LED_Small, LED_SMD:LED_0805_2012Metric, F.Cu at (-40.0, 118.7)
- added D3: ZMM5V6, Diode_SMD:D_MiniMELF, F.Cu at (198.0, 53.0)
- added D30: 5.7V, Diode_SMD:D_MicroMELF_Handsoldering, F.Cu at (-48.6, 122.8)
- added D31: LED_Small, LED_SMD:LED_0805_2012Metric, F.Cu at (21.0, 61.5)
- added D32: LED_Small, LED_SMD:LED_0805_2012Metric, F.Cu at (32.8, 50.0)
- added D33: LED_Small, LED_SMD:LED_0805_2012Metric, F.Cu at (-10.1, 91.3)
- added D34: STTH802G-TR, Package_TO_SOT_SMD:TO-263-2, F.Cu at (160.5, 77.2)
- added D35: 5.7V, Diode_SMD:D_MicroMELF_Handsoldering, F.Cu at (8.88, 69.0)
- added D36: 5.7V, Diode_SMD:D_MicroMELF_Handsoldering, F.Cu at (22.1, 55.1)
- added D37: 5.7V, Diode_SMD:D_MicroMELF_Handsoldering, F.Cu at (-29.2, 107.5)
- added D38: 5.7V, Diode_SMD:D_MicroMELF_Handsoldering, F.Cu at (-38.9, 115.7)
- added D4: ZMM5V6, Diode_SMD:D_MiniMELF, F.Cu at (201.0, 53.0)
- added D5: D_Schottky, Diode_SMD:D_SMA, F.Cu at (188.5, 58.0)
- added D6: D_Schottky, Diode_SMD:D_SMA, F.Cu at (196.0, 58.0)
- added D7: SRV05-4, Package_TO_SOT_SMD:SOT-23-6, F.Cu at (-85.0, 120.0)
- added D8: SRV05-4, Package_TO_SOT_SMD:SOT-23-6, F.Cu at (-51.1, 131.1)
- added D9: STPS2H100UY, Diode_SMD:D_SMB, F.Cu at (112.0, 60.5)
- added F1: Fuse-Pad-Pad, hellen-one-common:PAD-1206-PAD, F.Cu at (209.5, 51.5)
- added J1: Conn_02x02_Odd_Even, Connector_PinHeader_2.54mm:PinHeader_2x02_P2.54mm_Vertical, F.Cu at (-47.1, 116.5)
- added J14: CONN_01X03, Connector_PinHeader_2.54mm:PinHeader_1x03_P2.54mm_Vertical, F.Cu at (-73.1, 127.4)
- added J15: CONN_01X01, Connector_Pin:Pin_D1.4mm_L8.5mm_W2.8mm_FlatFork, F.Cu at (15.3, 64.2)
- added J2: FTSH-107-01-F-DV-K, Connector_PinHeader_1.27mm:PinHeader_2x07_P1.27mm_Vertical_SMD, F.Cu at (-65.1, 125.9)
- added J3: TC2030, Connector:Tag-Connect_TC2030-IDC-NL_2x03_P1.27mm_Vertical, F.Cu at (-7.22, 78.2)
- added J4: Conn_01x06, Connector_PinHeader_2.54mm:PinHeader_1x06_P2.54mm_Vertical, F.Cu at (-79.8, 102.0)
- added L1: 6.8uH, Inductor_SMD:L_Wuerth_HCI-1350, F.Cu at (192.5, 125.0)
- added L2: 10uH, Inductor_SMD:L_Vishay_IHLP-6767, F.Cu at (157.2, 96.5)
- added P10: Pad, hellen-one-common:PAD-TH, F.Cu at (-23.4, 118.7)
- added P11: Pad, hellen-one-common:PAD-TH, F.Cu at (44.7, 52.1)
- added P12: Pad, hellen-one-common:PAD-TH, F.Cu at (17.5, 76.8)
- added P13: Pad, hellen-one-common:PAD-TH, F.Cu at (26.4, 69.9)
- added P14: Pad, hellen-one-common:PAD-TH, F.Cu at (51.3, 47.1)
- added P15: Pad, hellen-one-common:PAD-TH, F.Cu at (13.5, 80.0)
- added P16: Pad, hellen-one-common:PAD-TH, F.Cu at (-37.1, 129.6)
- added P17: Pad, hellen-one-common:PAD-TH, F.Cu at (-6.59, 99.7)
- added P18: Pad, hellen-one-common:PAD-TH, F.Cu at (12.9, 83.7)
- added P19: Pad, hellen-one-common:PAD-TH, F.Cu at (-16.6, 111.7)
- added P2: Pad, hellen-one-common:PAD-TH, F.Cu at (17.3, 80.6)
- added P20: Pad, hellen-one-common:PAD-TH, F.Cu at (21.9, 73.4)
- added P21: Pad, hellen-one-common:PAD-TH, F.Cu at (-27.5, 121.7)
- added P22: Pad, hellen-one-common:PAD-TH, F.Cu at (10.2, 87.5)
- added P23: Pad, hellen-one-common:PAD-TH, F.Cu at (-33.3, 131.8)
- added P24: Pad, hellen-one-common:PAD-TH, F.Cu at (40.3, 55.6)
- added P25: Pad, hellen-one-common:PAD-TH, F.Cu at (47.6, 47.1)
- added P26: Pad, hellen-one-common:PAD-TH, F.Cu at (163.5, 52.0)
- added P27: Pad, hellen-one-common:PAD-TH, F.Cu at (166.5, 52.0)
- added P28: Pad, hellen-one-common:PAD-TH, F.Cu at (100.0, 52.0)
- added P29: Pad, hellen-one-common:PAD-TH, F.Cu at (87.5, 52.0)
- added P3: Pad, hellen-one-common:PAD-TH, F.Cu at (36.9, 59.4)
- added P30: Pad, hellen-one-common:PAD-TH, F.Cu at (106.0, 52.0)
- added P31: Pad, hellen-one-common:PAD-TH, F.Cu at (103.0, 52.0)
- added P4: Pad, hellen-one-common:PAD-TH, F.Cu at (31.5, 65.0)
- added P5: Pad, hellen-one-common:PAD-TH, F.Cu at (6.46, 88.0)
- added P6: Pad, hellen-one-common:PAD-TH, F.Cu at (-28.8, 125.5)
- added P7: Pad, hellen-one-common:PAD-TH, F.Cu at (-11.5, 105.9)
- added P8: Pad, hellen-one-common:PAD-TH, F.Cu at (-7.71, 105.9)
- added P9: Pad, hellen-one-common:PAD-TH, F.Cu at (1.04, 94.0)
- added Q1: BUK9230-100B, Package_TO_SOT_SMD:TO-252-2, F.Cu at (-1.93, 57.3)
- added Q10: BUK9230-100B, Package_TO_SOT_SMD:TO-252-2, F.Cu at (125.5, 71.6)
- added Q11: BUK9230-100B, Package_TO_SOT_SMD:TO-252-2, F.Cu at (133.0, 73.0)
- added Q12: BUK9230-100B, Package_TO_SOT_SMD:TO-252-2, F.Cu at (148.5, 71.5)
- added Q13: AOD4185, Package_TO_SOT_SMD:TO-252-2, F.Cu at (208.4, 56.5)
- added Q14: VND14NV04TR-E, Package_TO_SOT_SMD:TO-252-2, F.Cu at (188.5, 65.5)
- added Q15: VND14NV04TR-E, Package_TO_SOT_SMD:TO-252-2, F.Cu at (196.0, 65.5)
- added Q2: BUK9230-100B, Package_TO_SOT_SMD:TO-252-2, F.Cu at (172.5, 99.5)
- added Q3: BUK9230-100B, Package_TO_SOT_SMD:TO-252-2, F.Cu at (87.0, 71.5)
- added Q4: BUK9230-100B, Package_TO_SOT_SMD:TO-252-2, F.Cu at (82.5, 60.0)
- added Q5: BUK9230-100B, Package_TO_SOT_SMD:TO-252-2, F.Cu at (118.0, 75.0)
- added Q6: BUK9230-100B, Package_TO_SOT_SMD:TO-252-2, F.Cu at (110.5, 73.0)
- added Q7: BUK9230-100B, Package_TO_SOT_SMD:TO-252-2, F.Cu at (101.0, 62.1)
- added Q8: BUK9230-100B, Package_TO_SOT_SMD:TO-252-2, F.Cu at (103.0, 73.6)
- added Q9: BUK9230-100B, Package_TO_SOT_SMD:TO-252-2, F.Cu at (141.0, 71.5)
- added R1: Jumper-Pad-Pad, hellen-one-common:PAD-0805-PAD, F.Cu at (169.0, 53.5)
- added R10: 10, Resistor_SMD:R_0603_1608Metric, F.Cu at (93.5, 73.5)
- added R11: 10, Resistor_SMD:R_0603_1608Metric, F.Cu at (86.5, 65.2)
- added R12: 0R010, Resistor_SMD:R_1206_3216Metric_Pad1.30x1.75mm_HandSolder, F.Cu at (184.5, 96.2)
- added R13: 10, Resistor_SMD:R_0603_1608Metric, F.Cu at (99.0, 80.0)
- added R14: 10, Resistor_SMD:R_0603_1608Metric, F.Cu at (96.5, 70.0)
- added R15: 10, Resistor_SMD:R_0603_1608Metric, F.Cu at (122.5, 79.0)
- added R16: 10, Resistor_SMD:R_0603_1608Metric, F.Cu at (111.8, 66.5)
- added R17: 10, Resistor_SMD:R_0603_1608Metric, F.Cu at (138.0, 78.8)
- added R18: 10, Resistor_SMD:R_0603_1608Metric, F.Cu at (124.5, 79.0)
- added R19: 10, Resistor_SMD:R_0603_1608Metric, F.Cu at (134.8, 66.5)
- added R2: 10k, Resistor_SMD:R_0402_1005Metric, F.Cu at (203.5, 52.0)
- added R20: 10, Resistor_SMD:R_0603_1608Metric, F.Cu at (145.5, 78.8)
- added R21: 0R010, Resistor_SMD:R_1206_3216Metric_Pad1.30x1.75mm_HandSolder, F.Cu at (107.0, 80.5)
- added R22: 0R010, Resistor_SMD:R_1206_3216Metric_Pad1.30x1.75mm_HandSolder, F.Cu at (143.5, 80.0)
- added R23: 1K, Resistor_SMD:R_0603_1608Metric, F.Cu at (-8.70, 96.5)
- added R24: 10, Resistor_SMD:R_0603_1608Metric, F.Cu at (181.0, 101.0)
- added R25: 1K, Resistor_SMD:R_0603_1608Metric, F.Cu at (-94.1, 133.5)
- added R26: 0R010, Resistor_SMD:R_1206_3216Metric_Pad1.30x1.75mm_HandSolder, F.Cu at (151.0, 80.0)
- added R27: 1K, Resistor_SMD:R_0603_1608Metric, F.Cu at (14.2, 71.8)
- added R28: DNP, Resistor_SMD:R_0402_1005Metric, F.Cu at (-36.8, 132.5)
- added R29: 470K, Resistor_SMD:R_0402_1005Metric, F.Cu at (-25.5, 126.5)
- added R3: 1K, Resistor_SMD:R_0603_1608Metric, F.Cu at (18.7, 70.2)
- added R30: DNP, Resistor_SMD:R_0402_1005Metric, F.Cu at (40.3, 60.4)
- added R31: 470K, Resistor_SMD:R_0402_1005Metric, F.Cu at (20.6, 80.2)
- added R32: DNP, Resistor_SMD:R_0402_1005Metric, F.Cu at (28.7, 72.8)
- added R33: 470K, Resistor_SMD:R_0402_1005Metric, F.Cu at (-21.9, 58.6)
- added R34: 10k, hellen-one-common:R0603, F.Cu at (187.0, 72.0)
- added R35: 10k, hellen-one-common:R0603, F.Cu at (194.5, 72.0)
- added R36: 5.1k, hellen-one-common:R0603, F.Cu at (35.0, 64.2)
- added R37: 1k, Resistor_SMD:R_0402_1005Metric, F.Cu at (227.0, 65.5)
- added R38: 5.1, Resistor_SMD:R_0603_1608Metric, F.Cu at (178.2, 104.0)
- added R39: 1.6k, hellen-one-common:R0603, F.Cu at (-13.1, 112.5)
- added R4: 1K, Resistor_SMD:R_0603_1608Metric, F.Cu at (-1.45, 90.7)
- added R40: 750, hellen-one-common:R0603, F.Cu at (16.4, 83.5)
- added R41: 10, Resistor_SMD:R_0603_1608Metric, F.Cu at (41.0, 49.0)
- added R42: 5.1, Resistor_SMD:R_0603_1608Metric, F.Cu at (126.0, 127.8)
- added R43: 10K, Resistor_SMD:R_0603_1608Metric, F.Cu at (-24.6, 111.8)
- added R44: 10K, Resistor_SMD:R_0603_1608Metric, F.Cu at (9.62, 75.1)
- added R45: 0R010, Resistor_SMD:R_1206_3216Metric_Pad1.30x1.75mm_HandSolder, F.Cu at (103.8, 122.2)
- added R46: 6.8K, Resistor_SMD:R_0603_1608Metric, F.Cu at (-25.1, 114.3)
- added R47: 6.8K, Resistor_SMD:R_0603_1608Metric, F.Cu at (-6.65, 94.0)
- added R48: 6.8K, Resistor_SMD:R_0603_1608Metric, F.Cu at (27.4, 56.8)
- added R49: 6.8K, Resistor_SMD:R_0603_1608Metric, F.Cu at (9.21, 80.1)
- added R5: DNP, Resistor_SMD:R_0402_1005Metric, F.Cu at (-16.7, 116.5)
- added R50: 10K, Resistor_SMD:R_0603_1608Metric, F.Cu at (22.7, 66.8)
- added R51: 10K, Resistor_SMD:R_0603_1608Metric, F.Cu at (19.8, 64.3)
- added R52: 10K, Resistor_SMD:R_0603_1608Metric, F.Cu at (-90.1, 133.5)
- added R53: 10K, Resistor_SMD:R_0603_1608Metric, F.Cu at (-31.4, 121.0)
- added R54: 10K, Resistor_SMD:R_0603_1608Metric, F.Cu at (-45.0, 128.9)
- added R55: 1K, Resistor_SMD:R_0603_1608Metric, F.Cu at (-14.5, 100.1)
- added R56: Jumper-Pad-Pad, hellen-one-common:PAD-0805-PAD, F.Cu at (185.5, 53.5)
- added R57: Jumper-Pad-Pad, hellen-one-common:PAD-0805-PAD, F.Cu at (146.0, 53.5)
- added R58: Jumper-Pad-Pad, hellen-one-common:PAD-0805-PAD, F.Cu at (153.5, 53.5)
- added R59: Jumper-Pad-Pad, hellen-one-common:PAD-0805-PAD, F.Cu at (158.5, 53.5)
- added R6: 470K, Resistor_SMD:R_0402_1005Metric, F.Cu at (34.8, 66.1)
- added R60: Jumper-Pad-Pad, hellen-one-common:PAD-0805-PAD, F.Cu at (183.0, 53.5)
- added R61: Jumper-Pad-Pad, hellen-one-common:PAD-0805-PAD, F.Cu at (143.5, 53.5)
- added R62: Jumper-Pad-Pad, hellen-one-common:PAD-0805-PAD, F.Cu at (148.5, 53.5)
- added R63: Jumper-Pad-Pad, hellen-one-common:PAD-0805-PAD, F.Cu at (156.0, 53.5)
- added R64: Jumper-Pad-Pad, hellen-one-common:PAD-0805-PAD, F.Cu at (161.0, 53.5)
- added R65: Jumper-Pad-Pad, hellen-one-common:PAD-0805-PAD, F.Cu at (171.5, 53.5)
- added R66: Jumper-Pad-Pad, hellen-one-common:PAD-0805-PAD, F.Cu at (174.0, 53.5)
- added R67: Jumper-Pad-Pad, hellen-one-common:PAD-0805-PAD, F.Cu at (151.0, 53.5)
- added R68: Jumper-Pad-Pad, hellen-one-common:PAD-0805-PAD, F.Cu at (189.5, 53.5)
- added R69: Jumper-Pad-Pad, hellen-one-common:PAD-0805-PAD, F.Cu at (195.0, 53.5)
- added R7: 1K, Resistor_SMD:R_0603_1608Metric, F.Cu at (-5.90, 91.2)
- added R70: Jumper-Pad-Pad, hellen-one-common:PAD-0805-PAD, F.Cu at (112.5, 53.5)
- added R71: Jumper-Pad-Pad, hellen-one-common:PAD-0805-PAD, F.Cu at (97.5, 53.5)
- added R72: Jumper-Pad-Pad, hellen-one-common:PAD-0805-PAD, F.Cu at (108.5, 53.5)
- added R73: Jumper-Pad-Pad, hellen-one-common:PAD-0805-PAD, F.Cu at (93.5, 53.5)
- added R74: Jumper-Pad-Pad, hellen-one-common:PAD-0805-PAD, F.Cu at (136.0, 53.5)
- added R75: Jumper-Pad-Pad, hellen-one-common:PAD-0805-PAD, F.Cu at (128.0, 53.5)
- added R76: Jumper-Pad-Pad, hellen-one-common:PAD-0805-PAD, F.Cu at (132.0, 53.5)
- added R77: Jumper-Pad-Pad, hellen-one-common:PAD-0805-PAD, F.Cu at (124.0, 53.5)
- added R78: Jumper-Pad-Pad, hellen-one-common:PAD-0805-PAD, F.Cu at (120.0, 53.5)
- added R79: Jumper-Pad-Pad, hellen-one-common:PAD-0805-PAD, F.Cu at (116.5, 53.5)
- added R8: 1K, Resistor_SMD:R_0603_1608Metric, F.Cu at (5.20, 82.4)
- added R9: 1K, Resistor_SMD:R_0603_1608Metric, F.Cu at (13.6, 74.3)
- added RN1: 10k, Resistor_SMD:R_Array_Convex_4x0603, F.Cu at (-18.6, 101.2)
- added RN2: 10k, Resistor_SMD:R_Array_Convex_4x0603, F.Cu at (-23.5, 105.6)
- added RN3: 10k, Resistor_SMD:R_Array_Convex_4x0603, F.Cu at (5.54, 76.2)
- added TP1: TestPoint, Connector_PinHeader_2.54mm:PinHeader_1x01_P2.54mm_Horizontal, F.Cu at (-57.6, 84.3)
- added TP101: CONN_01X01, Connector_Pin:Pin_D0.7mm_L6.5mm_W1.8mm_FlatFork, F.Cu at (9.13, 83.1)
- added TP102: CONN_01X01, Connector_Pin:Pin_D0.7mm_L6.5mm_W1.8mm_FlatFork, F.Cu at (36.5, 50.0)
- added TP103: CONN_01X01, Connector_Pin:Pin_D0.7mm_L6.5mm_W1.8mm_FlatFork, F.Cu at (-10.6, 102.3)
- added TP104: CONN_01X01, Connector_Pin:Pin_D0.7mm_L6.5mm_W1.8mm_FlatFork, F.Cu at (18.1, 73.2)
- added TP2: TestPoint, Connector_PinHeader_2.54mm:PinHeader_1x01_P2.54mm_Horizontal, F.Cu at (-75.1, 102.0)
- added TP23: CONN_01X01, Connector_Pin:Pin_D0.7mm_L6.5mm_W1.8mm_FlatFork, F.Cu at (33.1, 59.8)
- added TP24: CONN_01X01, Connector_Pin:Pin_D0.7mm_L6.5mm_W1.8mm_FlatFork, F.Cu at (-2.72, 94.2)
- added TP4: CONN_01X01, Connector_Pin:Pin_D0.7mm_L6.5mm_W1.8mm_FlatFork, F.Cu at (-32.6, 124.4)
- added TP5: CONN_01X01, Connector_Pin:Pin_D0.7mm_L6.5mm_W1.8mm_FlatFork, F.Cu at (2.48, 90.4)
- added TP6: CONN_01X01, Connector_Pin:Pin_D0.7mm_L6.5mm_W1.8mm_FlatFork, F.Cu at (41.0, 52.0)
- added TP7: CONN_01X01, Connector_Pin:Pin_D0.7mm_L6.5mm_W1.8mm_FlatFork, F.Cu at (22.6, 69.8)
- added TP8: CONN_01X01, Connector_Pin:Pin_D0.7mm_L6.5mm_W1.8mm_FlatFork, F.Cu at (-15.5, 108.1)
- added U1: MC33816, Package_QFP:LQFP-64-1EP_10x10mm_P0.5mm_EP5x5mm_ThermalVias, F.Cu at (112.2, 112.2)
- added U2: TJA1051T-3, Package_SO:SOIC-8_3.9x4.9mm_P1.27mm, F.Cu at (-18.1, 80.7)
- added U3: LM78M05_TO252, Package_TO_SOT_SMD:TO-252-2, F.Cu at (220.0, 62.5)
- added U4: 74HC14, Package_SO:TSSOP-14_4.4x5mm_P0.65mm, F.Cu at (-6.87, 72.3)
- added U5: XC6206P332MR, Package_TO_SOT_SMD:SOT-23, F.Cu at (220.4, 68.4)
- added U6: MCP6004, Package_SO:TSSOP-14_4.4x5mm_P0.65mm, F.Cu at (-30.1, 91.4)
- added U7: STM32F103C6Tx, Package_QFP:LQFP-48_7x7mm_P0.5mm, F.Cu at (-46.2, 108.5)
- added Y2: 1MHz, Oscillator:Oscillator_SMD_Diodes_FN-4Pin_7.0x5.0mm, F.Cu at (8.12, 57.5)
Connections:
- P1 pad 1: unconnected-(P1-Pad1) -> GND
- P1 pad 114: unconnected-(P1-Pad114) -> /OUT_INJ1_N
- P1 pad 115: unconnected-(P1-Pad115) -> Net-(P1-Pad115)
- P1 pad 116: unconnected-(P1-Pad116) -> Net-(P1-Pad116)
- P1 pad 117: unconnected-(P1-Pad117) -> Net-(P1-Pad117)
- P1 pad 118: unconnected-(P1-Pad118) -> /OUT_INJ1_P
- P1 pad 119: unconnected-(P1-Pad119) -> /OUT_INJ2_N
- P1 pad 120: unconnected-(P1-Pad120) -> Net-(P1-Pad120)
- P1 pad 121: unconnected-(P1-Pad121) -> /OUT_INJ2_P
- P1 pad 2: unconnected-(P1-Pad2) -> GND
- P1 pad 21: unconnected-(P1-Pad21) -> Net-(P1-Pad21)
- P1 pad 22: unconnected-(P1-Pad22) -> Net-(P1-Pad21)
- P1 pad 23: unconnected-(P1-Pad23) -> Net-(P1-Pad23)
- P1 pad 24: unconnected-(P1-Pad24) -> Net-(P1-Pad23)
- P1 pad 4: unconnected-(P1-Pad4) -> Net-(P1-Pad4)
- P1 pad 40: unconnected-(P1-Pad40) -> Net-(P1-Pad40)
- P1 pad 41: unconnected-(P1-Pad41) -> Net-(P1-Pad41)
- P1 pad 44: unconnected-(P1-Pad44) -> Net-(P1-Pad44)
- P1 pad 45: unconnected-(P1-Pad45) -> Net-(P1-Pad45)
- P1 pad 46: unconnected-(P1-Pad46) -> Net-(P1-Pad46)
- P1 pad 47: unconnected-(P1-Pad47) -> Net-(P1-Pad47)
- P1 pad 48: unconnected-(P1-Pad48) -> Net-(P1-Pad48)
- P1 pad 49: unconnected-(P1-Pad49) -> Net-(P1-Pad49)
- P1 pad 51: unconnected-(P1-Pad51) -> Net-(P1-Pad51)
- P1 pad 52: unconnected-(P1-Pad52) -> Net-(P1-Pad52)
- P1 pad 53: unconnected-(P1-Pad53) -> Net-(P1-Pad53)
- P1 pad 6: unconnected-(P1-Pad6) -> Net-(P1-Pad6)
- P1 pad 7: unconnected-(P1-Pad7) -> Net-(P1-Pad7)
- P1 pad 8: unconnected-(P1-Pad8) -> Net-(P1-Pad8)
- P1 pad 82: unconnected-(P1-Pad82) -> /OUT_PUMP_L
- P1 pad 83: unconnected-(P1-Pad83) -> /OUT_PUMP_L
- P1 pad 84: unconnected-(P1-Pad84) -> /OUT_PUMP_H
- P1 pad 85: unconnected-(P1-Pad85) -> /OUT_PUMP_H
- P1 pad 9: unconnected-(P1-Pad9) -> Net-(P1-Pad9)
- P1 pad 90: unconnected-(P1-Pad90) -> /OUT_INJ3_N
- P1 pad 91: unconnected-(P1-Pad91) -> /OUT_INJ3_N
- P1 pad 92: unconnected-(P1-Pad92) -> /OUT_INJ4_N
- P1 pad 93: unconnected-(P1-Pad93) -> /OUT_INJ4_N
- P1 pad 94: unconnected-(P1-Pad94) -> /OUT_INJ3_P
- P1 pad 95: unconnected-(P1-Pad95) -> /OUT_INJ3_P
- P1 pad 96: unconnected-(P1-Pad96) -> /OUT_INJ4_P
- P1 pad 97: unconnected-(P1-Pad97) -> /OUT_INJ4_P

Commit message: Upd PCB
Parts:
- removed D30, D35, D36, D37, D38: 5.7V, Diode_SMD:D_MicroMELF_Handsoldering
- removed J14: CONN_01X03, Connector_PinHeader_2.54mm:PinHeader_1x03_P2.54mm_Vertical
- removed J15: CONN_01X01, Connector_Pin:Pin_D1.4mm_L8.5mm_W2.8mm_FlatFork
- removed Q1: BUK9230-100B, Package_TO_SOT_SMD:TO-252-2
- removed R44: 10K, Resistor_SMD:R_0603_1608Metric
- removed R55: 1K, Resistor_SMD:R_0603_1608Metric
- removed TP1, TP2: TestPoint, Connector_PinHeader_2.54mm:PinHeader_1x01_P2.54mm_Horizontal
- removed TP101, TP102, TP103, TP104, TP23, TP24, TP4, TP5, TP6, TP7, TP8: CONN_01X01, Connector_Pin:Pin_D0.7mm_L6.5mm_W1.8mm_FlatFork
- added J5: Conn_01x04, Connector_PinHeader_2.54mm:PinHeader_1x04_P2.54mm_Vertical, F.Cu at (159.5, 58.7)
- added P36: Pad, hellen-one-common:PAD-TH, F.Cu at (94.5, 90.0)
- C2, C20, C3: footprint Capacitor_SMD:C_0402_1005Metric -> hellen-one-common:C0603
- C66, C69, C70, C72: value 100nF -> 100n; footprint Capacitor_SMD:C_0402_1005Metric -> hellen-one-common:C0603
- R2: footprint Resistor_SMD:R_0402_1005Metric -> hellen-one-common:R0603
- R28, R29, R30, R31, R32, R33, R5, R6: footprint Resistor_SMD:R_0402_1005Metric -> Resistor_SMD:R_0603_1608Metric
- R37: value 1k -> 1K; footprint Resistor_SMD:R_0402_1005Metric -> Resistor_SMD:R_0603_1608Metric
- moved R52 220.3 mm to (128.0, 102.1), turned to -90 degrees
- moved D28 215.1 mm to (166.4, 58.5), turned to 180 degrees
- moved R43 209.6 mm to (181.0, 70.8), turned to -90 degrees
- moved D20 204.9 mm to (104.5, 103.5), turned to 180 degrees
- moved C3 200.3 mm to (174.1, 57.5), turned to 180 degrees
- moved C17 198.5 mm to (203.8, 128.8)
- moved R25 193.5 mm to (98.5, 114.8), turned to -90 degrees
- moved U2 191.3 mm to (172.5, 63.2), turned to 90 degrees
- moved D7 191.1 mm to (106.0, 124.5), turned to -90 degrees
- moved C19 185.8 mm to (100.0, 114.8), turned to -90 degrees
- moved R39 183.4 mm to (163.1, 61.5), turned to 180 degrees
- moved C20 179.7 mm to (176.0, 63.5), turned to -90 degrees
- moved R28 178.6 mm to (138.4, 97.6), turned to 180 degrees
- moved D33 178.6 mm to (166.5, 65.0), turned to 180 degrees
- moved J4 176.8 mm to (96.1, 84.2), turned to -90 degrees
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Connections:
- net Net-(C24-Pad2) renamed /Vdrive_shunt
- net Net-(D34-Pad1) renamed /Vdrive_coil
- net Net-(L1-Pad2) renamed /+Batt_filtered
- C2 pad 1: GND -> /CAN_H
- C2 pad 2: /CAN_H -> GND
- C20 pad 1: +5V -> GND
- C20 pad 2: GND -> +5V
- C3 pad 1: /CAN_L -> GND
- C3 pad 2: GND -> /CAN_L
- C66 pad 1: Net-(C66-Pad1) -> GND
- C66 pad 2: GND -> Net-(D18-Pad3)
- C69 pad 1: Net-(C69-Pad1) -> GND
- C69 pad 2: GND -> Net-(D18-Pad1)
- C70 pad 1: Net-(C70-Pad1) -> GND
- C70 pad 2: GND -> Net-(D18-Pad6)
- C72 pad 1: Net-(C72-Pad1) -> GND
- C72 pad 2: GND -> Net-(D18-Pad4)
- D18 pad 1: Net-(C69-Pad1) -> Net-(D18-Pad1)
- D18 pad 3: Net-(C66-Pad1) -> Net-(D18-Pad3)
- D18 pad 4: Net-(C72-Pad1) -> Net-(D18-Pad4)
- D18 pad 6: Net-(C70-Pad1) -> Net-(D18-Pad6)
- D31 pad 1: Net-(D31-Pad1) -> GND
- D31 pad 2: /5V -> Net-(R43-Pad1)
- R28 pad 1: /IN_A1 -> +5V
- R28 pad 2: +5V -> /IN_A1
- R30 pad 1: /IN_A2 -> +5V
- R30 pad 2: +5V -> /IN_A2
- R32 pad 1: /IN_A3 -> +5V
- R32 pad 2: +5V -> /IN_A3
- R36 pad 2: /Vbat -> +BATT
- R37 pad 1: GND -> Net-(D19-Pad1)
- R37 pad 2: Net-(D19-Pad1) -> GND
- R39 pad 2: /5V -> +5V
- R40 pad 2: /3.3V -> +3V3
- R43 pad 1: Net-(D35-Pad1) -> Net-(R43-Pad1)
- R5 pad 1: /IN_A0 -> +5V
- R5 pad 2: +5V -> /IN_A0
- RN3 pad 5: Net-(C72-Pad1) -> Net-(D18-Pad4)
- RN3 pad 6: Net-(C70-Pad1) -> Net-(D18-Pad6)
- RN3 pad 7: Net-(C69-Pad1) -> Net-(D18-Pad1)
- RN3 pad 8: Net-(C66-Pad1) -> Net-(D18-Pad3)
- U6 pad 10: Net-(C69-Pad1) -> Net-(D18-Pad1)
- U6 pad 12: Net-(C66-Pad1) -> Net-(D18-Pad3)
- U6 pad 3: Net-(C72-Pad1) -> Net-(D18-Pad4)
- U6 pad 5: Net-(C70-Pad1) -> Net-(D18-Pad6)
Routing:
- net +BATT: track 0.00 -> 261.2 mm, vias 0 -> 7
- net Vdrive: track 0.00 -> 151.7 mm, vias 0 -> 7
- net /OUT_PUMP_H: track 0.00 -> 81.3 mm
- net /OUT_INJ3_P: track 0.00 -> 69.0 mm
- net /OUT_INJ4_N: track 0.00 -> 69.0 mm
- net /L1: track 0.00 -> 33.6 mm, vias 0 -> 1
- net +3V3: track 0.00 -> 32.8 mm, vias 0 -> 1
- net /H3: track 0.00 -> 30.7 mm, vias 0 -> 1
- net +5V: track 0.00 -> 28.6 mm
- net /Vdrive_shunt: track 0.00 -> 25.1 mm, vias 0 -> 2
- net /OUT_PUMP_L: track 0.00 -> 23.6 mm
- net Net-(C11-Pad2): track 0.00 -> 23.5 mm
- net Net-(C10-Pad2): track 0.00 -> 23.1 mm, vias 0 -> 3
- net /L5: track 0.00 -> 21.3 mm
- net /OUT_INJ4_P: track 0.00 -> 20.4 mm
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- added copper zone on F.Cu, net +BATT
- added copper zone on F.Cu, net /+Batt_filtered
- added copper zone on F.Cu, net /Vdrive_coil
- added copper zone on F.Cu, net /Vdrive_shunt
- added copper zone on F.Cu, net Vdrive
