File: GDI-4ch/GDI-4ch.kicad_sch (KiCad schematic)
At the start: 165 parts, among them J14 CONN_01X03, J15 CONN_01X01, J3 CONN_02X08, J4 CONN_02X08, J7 CONN_01X03, P1 368255-2, Q1 BUK9230-100B, Q10 BUK9230-100B, Q11 BUK9230-100B, Q12 BUK9230-100B, Q2 BUK9230-100B, Q3 BUK9230-100B, Q4 BUK9230-100B, Q5 BUK9230-100B, Q6 BUK9230-100B, Q7 BUK9230-100B, Q8 BUK9230-100B, Q9 BUK9230-100B, U1 MC33816, Y2 1MHz

Commit message: Upd SCH
Parts:
- added C? (x3): 10u, Capacitor_SMD:C_0603_1608Metric, symbol Device:C
- added C? (x6): 100n, Capacitor_SMD:C_0402_1005Metric, symbol Device:C
- added C? (x2): 47p, Capacitor_SMD:C_0402_1005Metric, symbol Device:C
- added C?: 4.7u, Capacitor_SMD:C_0603_1608Metric, symbol Device:C
- added C?: 10u, Capacitor_SMD:C_1206_3216Metric, symbol Device:C
- added D?: WHITE, LED_SMD:LED_0603_1608Metric, symbol Device:LED
- added D? (x3): ZMM5V6, Diode_SMD:D_MiniMELF, symbol Device:D_Zener
- added D?: SMCJ22CA, Diode_SMD:D_SMC, symbol Device:D_TVS
- added F?: Fuse, Fuse:Fuseholder_Blade_Mini_Keystone_3568, symbol Device:Fuse
- added J?: Conn_02x03_Odd_Even, Connector:Tag-Connect_TC2030-IDC-NL_2x03_P1.27mm_Vertical, symbol Connector_Generic:Conn_02x03_Odd_Even
- added J?: FTSH-107-01-F-DV-K, Connector_PinHeader_1.27mm:PinHeader_2x07_P1.27mm_Vertical_SMD, symbol Connector_Generic:Conn_02x07_Odd_Even
- added J?: Conn_02x02_Odd_Even, Connector_PinHeader_2.54mm:PinHeader_2x02_P2.54mm_Vertical, symbol Connector_Generic:Conn_02x02_Odd_Even
- added Q?: VBA2625, Package_SO:SOIC-8_3.9x4.9mm_P1.27mm, symbol Transistor_FET:IRF7404
- added R?: 1k, Resistor_SMD:R_0402_1005Metric, symbol Device:R
- added R? (x2): 10k, Resistor_SMD:R_0402_1005Metric, symbol Device:R
- added TP? (x2): TestPoint, Connector_PinHeader_2.54mm:PinHeader_1x01_P2.54mm_Horizontal, symbol Connector:TestPoint
- added U?: XC6206P332MR, Package_TO_SOT_SMD:SOT-23, symbol Regulator_Linear:XC6206PxxxMR
- added U?: LM78M05_TO252, Package_TO_SOT_SMD:TO-252-2, symbol Regulator_Linear:LM78M05_TO252
- added U?: TJA1051T-3, Package_SO:SOIC-8_3.9x4.9mm_P1.27mm, symbol Interface_CAN_LIN:TJA1051T-3
- added U?: STM32F103C6Tx, Package_QFP:LQFP-48_7x7mm_P0.5mm, symbol MCU_ST_STM32F1:STM32F103C6Tx
Connections:
- net +5V: now also C?.1, C?.1, C?.1, J?.4 (Pin_4), U?.3 (VCC), U?.3 (VI), U?.3 (VO)
- net +BATT: now also C?.1, D?.1 (K), Q?.1 (S), Q?.2 (S), Q?.3 (S), U?.1 (VI)
- net 3.3V: no longer R45.1
- net GND: now also P1.1, P1.2, C?.1, C?.2, C?.2, C?.2, C?.2, C?.2, C?.2, C?.2, C?.2, C?.2, C?.2, C?.2, C?.2, D?.2 (A2), J?.11 (Pin_11), J?.3 (Pin_3), J?.5 (Pin_5), J?.5 (Pin_5), J?.7 (Pin_7), R?.1, R?.1, R?.1, U?.1 (GND), U?.2 (GND), U?.2 (GND), U?.23 (VSS), U?.35 (VSS), U?.47 (VSS), U?.8 (S), U?.8 (VSSA)
- net IN_INJ1: now reaches P1.43
- net IN_INJ2: now reaches P1.44
- net IN_INJ3: now reaches P1.45
- net IN_INJ4: now reaches P1.46
- net IN_INJ5: now reaches P1.47
- net IN_INJ6: now reaches P1.48
- net CAN_H: now reaches P1.52
- net CAN_H: now also C?.2, U?.7 (CANH)
- net CAN_L: now reaches P1.53
- net CAN_L: now also C?.1, U?.6 (CANL)
- net OUT_INJ3_N: now reaches P1.90
- net OUT_INJ3_N: now also P1.91
- net OUT_INJ4_N: now reaches P1.92
- net OUT_INJ4_N: now also P1.93
- net OUT_INJ3_P: now reaches P1.94
- net OUT_INJ3_P: now also P1.95
- net OUT_INJ4_P: now reaches P1.96
- net OUT_INJ4_P: now also P1.97
- net OUT_INJ1_N: now reaches P1.114
- net OUT_INJ6_N: now reaches P1.115
- net OUT_INJ5_N: now reaches P1.116
- net OUT_INJ5_P: now reaches P1.117
- net OUT_INJ1_P: now reaches P1.118
- net OUT_INJ2_N: now reaches P1.119
- net OUT_INJ6_P: now reaches P1.120
- net OUT_INJ2_P: now reaches P1.121
- net at P1.4: now also F?.2
- new net: D?.1 (K), R?.2
- new net: D?.1 (K), D?.2 (A) (x2)
- new net: D?.2 (A), Q?.4 (G), R?.2
- new net: D?.1 (A1), F?.1, Q?.5 (D), Q?.6 (D), Q?.7 (D), Q?.8 (D)
- new net +3V3: C?.1, C?.1, C?.1, C?.1, C?.1, C?.1, C?.1, D?.2 (A), J?.1 (Pin_1), J?.3 (Pin_3), R45.1, U?.1 (VBAT), U?.2 (VO), U?.24 (VDD), U?.36 (VDD), U?.48 (VDD), U?.5 (VIO), U?.9 (VDDA)
- new net Boot0: R?.2, TP?.1, U?.44 (BOOT0)
- new net CAN_RX: U?.32 (PA11), U?.4 (RXD)
- new net CAN_TX: U?.1 (TXD), U?.33 (PA12)
- new net SWCLK: J?.4 (Pin_4), J?.6 (Pin_6), U?.37 (PA14)
- new net SWDIO: J?.2 (Pin_2), J?.4 (Pin_4), U?.34 (PA13)
- new net SWO: J?.8 (Pin_8), U?.39 (PB3)
- new net UART_RX: J?.13 (Pin_13), J?.2 (Pin_2), U?.31 (PA10)
- new net UART_TX: J?.1 (Pin_1), J?.14 (Pin_14), U?.30 (PA9)
- new net nRESET: J?.12 (Pin_12), J?.3 (Pin_3), TP?.1, U?.7 (NRST)
- no-connect marks 6 -> 103
Other:
- note added: "???"
- note added: "Channels 5 and 6 in next rev"
- note added: "Debug"
- note added: "TODO: check fuse & mosfet"
- note added: "UART / +5 / GND for integration"
- note removed: "TODO: VCCIO"
- moved on the sheet: C1, C10, C11, C12, C13, C14, C15, C16, C17, C19, C21, C22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

Commit message: UPD sch
Parts:
- added C? (x4): 100nF, Capacitor_SMD:C_0402_1005Metric, symbol Device:C
- added C?: 10nF, Capacitor_SMD:C_0603_1608Metric, symbol Device:C
- added D?: BLUE, LED_SMD:LED_0603_1608Metric, symbol Device:LED
- added D?: GREEN, LED_SMD:LED_0603_1608Metric, symbol Device:LED
- added D? (x2): D_Schottky, Diode_SMD:D_SMA, symbol Device:D_Schottky
- added D?: SRV05-4, Package_TO_SOT_SMD:SOT-23-6, symbol Power_Protection:NUP4202
- added J?: Conn_01x06, Connector_PinHeader_2.54mm:PinHeader_1x06_P2.54mm_Vertical, symbol Connector_Generic:Conn_01x06
- added P? (x4): Pad, hellen-one-common:PAD-TH, symbol hellen-one-common:Pad
- added Q? (x2): VND14NV04TR-E, Package_TO_SOT_SMD:TO-252-2, symbol semiconductors:VND14NV04TR-E
- added R? (x4): 470K, Resistor_SMD:R_0402_1005Metric, symbol Device:R
- added R? (x4): DNP, Resistor_SMD:R_0402_1005Metric, symbol Device:R
- added R? (x2): 10k, hellen-one-common:R0603, symbol hellen-one-common:Res
- added R? (x2): 1k, Resistor_SMD:R_0402_1005Metric, symbol Device:R
- added R? (x4): 6.8K, Resistor_SMD:R_0603_1608Metric, symbol Device:R
- added R? (x4): 10K, Resistor_SMD:R_0603_1608Metric, symbol Device:R
- added R?: Jumper-Pad-Pad, hellen-one-common:PAD-0805-PAD, symbol hellen-one-common:Jumper-Pad-Pad
- added RN?: 10k, Resistor_SMD:R_Array_Convex_4x0603, symbol Device:R_Pack04
- added U? (x5): MCP6004, Package_SO:TSSOP-14_4.4x5mm_P0.65mm, symbol Amplifier_Operational:MCP6004
- J?: value Conn_02x03_Odd_Even -> TC2030
Connections:
- net H_PUMP is gone; now on net OUT_PUMP_H: C63.2, C64.1, C65.1, D16.1 (K), Q11.3 (S), U1.51 (S_HS5)
- net L_PUMP is gone; now on net OUT_PUMP_L: C67.1, D17.2 (A), Q12.2 (D), U1.33 (D_LS6)
- net +3V3: now also J?.1 (Pin_1)
- net +5V: now also C?.1, D?.5, R?.2, R?.2, R?.2, R?.2, U?.4 (V+)
- net +BATT: now also D?.1 (K), D?.1 (K), R?.2
- net CSB: now also U?.18 (PB0), P?.1 (Pin_1)
- net GND: now also C?.2, C?.2, C?.2, C?.2, C?.2, D?.2, J?.3 (Pin_3), Q?.3 (S), Q?.3 (S), R?.1, R?.1, R?.1, R?.1, R?.1, R?.1, R?.1, R?.1, R?.2, R?.2, R?.2, R?.2, U?.11 (V-)
- net MISO: now also U?.16 (PA6), P?.1 (Pin_1)
- net MOSI: now also U?.17 (PA7), P?.1 (Pin_1)
- net SCLK: now also U?.15 (PA5), P?.1 (Pin_1)
- net SWCLK: now also J?.2 (Pin_2)
- net SWDIO: now also J?.4 (Pin_4)
- net nRESET: now also J?.5 (Pin_5)
- net OUT_LS1: now reaches P1.21
- net OUT_LS1: now also P1.22, D?.2 (A), Q?.2 (D)
- net OUT_LS2: now reaches P1.23
- net OUT_LS2: now also P1.24, D?.2 (A), Q?.2 (D)
- net IN_PUMP: now reaches P1.40
- net at P1.51: now also R?.1
- net IN_A0: now reaches P1.6
- net IN_A0: now also R?.1, R?.1, RN?.1 (R1.1)
- net IN_A1: now reaches P1.7
- net IN_A1: now also R?.1, R?.1, RN?.2 (R2.1)
- net IN_A2: now reaches P1.8
- net IN_A2: now also R?.1, R?.1, RN?.3 (R3.1)
- net OUT_PUMP_L: now reaches P1.82
- net OUT_PUMP_L: now also P1.83
- net OUT_PUMP_H: now reaches P1.84
- net OUT_PUMP_H: now also P1.85
- net IN_A3: now reaches P1.9
- net IN_A3: now also R?.1, R?.1, RN?.4 (R4.1)
- net A0: now reaches U?.10 (PA0)
- net A0: now also R?.1, R?.2
- net LS1: now reaches U?.11 (PA1)
- net LS1: now also Q?.1 (G), R?.2
- net A1: now reaches U?.12 (PA2)
- net A1: now also R?.1, R?.2
- net A2: now reaches U?.13 (PA3)
- net A2: now also R?.1, R?.2
- net A3: now reaches U?.14 (PA4)
- net A3: now also R?.1, R?.2
- net LED_BLUE: now reaches U?.26 (PB13)
- net LED_BLUE: now also D?.2 (A)
- net LED_GREEN: now reaches U?.29 (PA8)
- net LED_GREEN: now also D?.2 (A)
- net LS2: now reaches U?.42 (PB6)
- net LS2: now also Q?.1 (G), R?.2
- net IN_INJ5: no longer names the net of P1.47
- net IN_INJ6: no longer names the net of P1.48
- net OUT_INJ5_N: no longer names the net of P1.116
- net OUT_INJ5_P: no longer names the net of P1.117
- net OUT_INJ6_N: no longer names the net of P1.115
- net OUT_INJ6_P: no longer names the net of P1.120
- new net: R?.2, U?.1, U?.2 (-)
- new net: C?.1, D?.4, RN?.5 (R4.2), U?.3 (+)
- new net: D?.1 (K), R?.2 (x2)
- new net: C?.1, D?.3, RN?.8 (R1.2), U?.12 (+)
- new net: R?.2, U?.13 (-), U?.14
- new net: C?.1, D?.6, RN?.6 (R3.2), U?.5 (+)
- new net: R?.2, U?.6 (-), U?.7
- new net: R?.2, U?.8, U?.9 (-)
- new net: C?.1, D?.1, RN?.7 (R2.2), U?.10 (+)
- no-connect marks 103 -> 91
Other:
- note removed: "???"
- moved on the sheet: J7

Commit message: UPD sch
Parts:
- removed C1: 100nF, Capacitor_SMD:C_0603_1608Metric, symbol Device:C
- removed C10, C11, C13, C8: 0.1uF, rusefi_lib:C_0805, symbol Device:C
- removed C12: 4.7uF, rusefi_lib:C_0805, symbol Device:C
- removed C23, C24, C28, C59, C60, C73: 330pF, rusefi_lib:C_0805, symbol Device:C
- removed C26: 470pF, rusefi_lib:C_0805, symbol Device:C
- removed C43, C44, C45, C46, C47, C48, C49, C50, C65, C67: 4700pF, rusefi_lib:C_0805, symbol Device:C
- removed C9: 1uF, rusefi_lib:C_0805, symbol Device:C
- removed C? (x3): 10u, Capacitor_SMD:C_0603_1608Metric, symbol Device:C
- removed C? (x5): 100n, Capacitor_SMD:C_0402_1005Metric, symbol Device:C
- removed C?: 4.7u, Capacitor_SMD:C_0603_1608Metric, symbol Device:C
- removed C?: 10nF, Capacitor_SMD:C_0603_1608Metric, symbol Device:C
- removed C?: 10u, Capacitor_SMD:C_1206_3216Metric, symbol Device:C
- removed D1, D18, D19, D2, D20, D21, D22, D23, D24, D25, D26, D27, D29, D3, D4, D5, D6, D7, D8: LED_Small, LED_SMD:LED_0805_2012Metric, symbol Device:LED_Small
- removed D9: FFD10UP20S, Package_TO_SOT_SMD:TO-252-2, symbol Device:D_Schottky_KKA
- removed J3, J4: CONN_02X08, Pin_Headers:Pin_Header_Straight_2x08_Pitch2.54mm, symbol Connector_Generic:Conn_02x08_Odd_Even
- removed J7: CONN_01X03, Pin_Headers:Pin_Header_Straight_1x03_Pitch2.54mm, symbol Connector_Generic:Conn_01x03
- removed R1, R2, R28, R29, R30, R31, R32, R33, R34, R35, R36, R37, R39, R40, R5, R6: 1k, rusefi_lib:R_0805, symbol Device:R
- removed R? (x2): 1k, Resistor_SMD:R_0402_1005Metric, symbol Device:R
- removed R?: 10k, Resistor_SMD:R_0402_1005Metric, symbol Device:R
- removed TP3: CONN_01X01, Connector_Pin:Pin_D0.7mm_L6.5mm_W1.8mm_FlatFork, symbol Connector_Generic:Conn_01x01
- added C1, C23, C28, C32, C34, C59, C75, C76, C77, C78, C79, C8: 100n, hellen-one-common:C0603, symbol hellen-one-common:Cap
- added C10, C11, C13, C24, C60, C73: 330p, hellen-one-common:C0603, symbol hellen-one-common:Cap
- added C12, C26: 4.7u, hellen-one-common:C0603, symbol hellen-one-common:Cap
- added C18, C29, C30, C5, C51, C52, C53, C54, C6, C61, C62, C7: 1000pF, Capacitor_SMD:C_0603_1608Metric, symbol Device:C
- added C31, C33, C4, C68: 10u, Capacitor_SMD:C_0805_2012Metric, symbol hellen-one-common:Cap
- added C43, C44, C45, C46, C47, C48, C49, C50, C65, C67: 4700p, hellen-one-common:C0603, symbol hellen-one-common:Cap
- added C74: 470p, hellen-one-common:C0603, symbol hellen-one-common:Cap
- added C9: 1u, hellen-one-common:C0603, symbol hellen-one-common:Cap
- added D7, D8: SRV05-4, Package_TO_SOT_SMD:SOT-23-6, symbol Power_Protection:NUP4202
- added P10, P11, P12, P13, P14, P15, P16, P17, P21, P22, P23, P24, P25, P26, P27, P28, P29, P3, P30, P31, P4, P5, P6, P7, P8, P9: Pad, hellen-one-common:PAD-TH, symbol hellen-one-common:Pad
- added R36: 5.1k, hellen-one-common:R0603, symbol hellen-one-common:Res
- added R39: 1.6k, hellen-one-common:R0603, symbol hellen-one-common:Res
- added R40: 750, hellen-one-common:R0603, symbol hellen-one-common:Res
- added R54: 10K, Resistor_SMD:R_0603_1608Metric, symbol Device:R
- added R55: 1K, Resistor_SMD:R_0603_1608Metric, symbol Device:R
- added R57, R58, R59, R60, R61, R62, R63, R64, R65, R66, R67, R68, R69, R70, R71, R72, R73, R74, R75, R76, R77, R78, R79: Jumper-Pad-Pad, hellen-one-common:PAD-0805-PAD, symbol hellen-one-common:Jumper-Pad-Pad
- added RN1, RN2: 10k, Resistor_SMD:R_Array_Convex_4x0603, symbol Device:R_Pack04
- added U4: 74HC14, symbol 74xx:74HC14
- C19, C35, C36, C37, C38, C55, C56, C57, C58, C63, C71: footprint rusefi_lib:C_0805 -> Capacitor_SMD:C_0603_1608Metric; LCSC C46653 -> C106247; MFG,MFG# avx,08051C102KAT2A -> (none); VEND1,VEND1# DIGI,478-1352-1-ND -> (none); VEND2,VEND2# JLCPCB,C209838 -> (none)
- C39, C40, C41, C42, C64: footprint rusefi_lib:C_0805 -> Capacitor_SMD:C_0603_1608Metric; LCSC C1740 -> C1615; MFG,MFG# Yageo,CC0805KKX7R8BB334 -> (none); VEND1,VEND1# DIGI,311-3385-1-ND -> (none); VEND2,VEND2# JLCPCB,C1740 -> (none)
- R10: value 5.1R -> 10; footprint rusefi_lib:R_0805 -> Resistor_SMD:R_0603_1608Metric; LCSC C247080 -> C22859; MFG,MFG# Stackpole,RMCF0805JT5R10 -> (none); VEND1,VEND1# DIGI,RMCF0805JT5R10CT-ND -> (none); VEND2,VEND2# JLCPCB,C247080 -> (none)
- R11, R13, R14, R15, R16, R17, R18, R19, R20, R24: value 10R -> 10; footprint rusefi_lib:R_0805 -> Resistor_SMD:R_0603_1608Metric; LCSC C17415 -> C22859; MFG,MFG# Stackpole,RMCF0805JG10R0 -> (none); VEND1,VEND1# DIGI,RMCF0805JG10R0CT-ND -> (none); VEND2,VEND2# JLCPCB,C17403 -> (none)
- R12, R21, R22, R26: footprint Resistors_SMD:R_1206_HandSoldering -> Resistor_SMD:R_1206_3216Metric_Pad1.30x1.75mm_HandSolder
- R23: value 10R -> 1K; footprint rusefi_lib:R_0805 -> Resistor_SMD:R_0603_1608Metric; LCSC C17415 -> C21190; MFG,MFG# Stackpole,RMCF0805JG10R0 -> (none); VEND1,VEND1# DIGI,RMCF0805JG10R0CT-ND -> (none); VEND2,VEND2# JLCPCB,C17403 -> (none)
- R25, R27, R3, R4, R7, R8: value 1k -> 1K; footprint rusefi_lib:R_0805 -> Resistor_SMD:R_0603_1608Metric; LCSC C17513 -> C21190; MFG,MFG# , -> (none); VEND1,VEND1# , -> (none); VEND2,VEND2# , -> (none)
- R38: value 10k -> 5.1; LCSC C17513 -> C25197; MFG,MFG# , -> (none); VEND1,VEND1# , -> (none); VEND2,VEND2# , -> (none)
- R42: value 1k -> 5.1; footprint Resistor_SMD:R_0805_2012Metric -> Resistor_SMD:R_0603_1608Metric; LCSC C17513 -> C25197; MFG,MFG# , -> (none); VEND1,VEND1# , -> (none); VEND2,VEND2# , -> (none)
- R43: value 0R010 -> 10K; footprint Resistor_SMD:R_1206_3216Metric_Pad1.42x1.75mm_HandSolder -> Resistor_SMD:R_0603_1608Metric; LCSC C76294 -> C25804; MFG,MFG# Ohmite,MCS1632R010FER -> (none); Manufacturer (none) -> StackPole; Part # (none) -> RMCF0603JT10K0; VEND (none) -> DIGI; VEND# (none) -> RMCF0603JT10K0CT-ND; VEND1,VEND1# DIGI,MCS1632R010FERCT-ND -> (none); VEND2,VEND2# , -> (none)
- R44: value 10k -> 10K; LCSC C17513 -> C25804; MFG,MFG# , -> (none); Manufacturer (none) -> StackPole; Part # (none) -> RMCF0603JT10K0; VEND (none) -> DIGI; VEND# (none) -> RMCF0603JT10K0CT-ND; VEND1,VEND1# , -> (none); VEND2,VEND2# , -> (none)
- R45: footprint Resistor_SMD:R_1206_3216Metric_Pad1.42x1.75mm_HandSolder -> Resistor_SMD:R_1206_3216Metric_Pad1.30x1.75mm_HandSolder
- R9: value 5.1R -> 1K; footprint rusefi_lib:R_0805 -> Resistor_SMD:R_0603_1608Metric; LCSC C247080 -> C21190; MFG,MFG# Stackpole,RMCF0805JT5R10 -> (none); VEND1,VEND1# DIGI,RMCF0805JT5R10CT-ND -> (none); VEND2,VEND2# JLCPCB,C247080 -> (none)
- gave numbers to parts that had none: 58
Connections:
- net +3V3: now also R25.1, R27.1, R3.1, R4.1, R7.1, R8.1, C1.2, C12.2, C68.2, C75.2, C76.2, C77.2, C78.2, C79.2, D7.5, D8.5, U4.14 (VCC)
- net +5V: now also C31.2, C33.2, C34.2, C8.2
- net +BATT: now also C23.2, C4.2
- net 3.3V: now also C71.2, R40.2; no longer C19.1
- net 5V: now also R39.2
- net Boot0: now also R54.1
- net CAN_H: now also R65.2; no longer P1.52
- net CAN_L: now also R66.2; no longer P1.53
- net CSB: now also U7.20 (PB2); no longer R25.2, U7.18 (PB0)
- net DRVEN: now also U7.40 (PB4), P3.1 (Pin_1); no longer R8.2
- net FLAG_0: now also U7.43 (PB7), P5.1 (Pin_1)
- net GND: now also C19.1, C35.1, C36.1, C37.1, C38.1, C71.1, R23.1, R44.2, R9.2, C1.1, C10.1, C11.1, C12.1, C13.1, C18.1, C23.1, C24.1, C26.1, C28.1, C29.1, C30.1, C31.1, C32.1, C33.1, C34.1, C4.1, C43.1, C44.1, C45.1, C46.1, C47.1, C48.1, C49.1, C5.1, C50.1, C51.1, C59.1, C6.1, C65.1, C67.1, C68.1, C7.1, C75.1, C76.1, C77.1, C78.1, C79.1, C8.1, C9.1, D7.2, D8.2, R54.2, U4.7 (GND); no longer C19.2, J14.1 (Pin_1), R44.1
- net H1: now also C41.2, C43.2, C44.2, C53.1, R71.2, R73.2; no longer C36.2, C40.1
- net H3: now also C42.2, C57.1, C47.2, C48.2, R78.2, R79.2; no longer C38.2, C42.1
- net IN_A0: now also R57.2; no longer P1.6
- net IN_A1: now also R67.2; no longer P1.7
- net IN_A2: now also R58.2; no longer P1.8
- net IN_A3: now also R59.2; no longer P1.9
- net IN_INJ1: now also R3.2, C5.2, R61.2, RN1.1 (R1.1); no longer P1.43
- net IN_INJ2: now also R4.2, C6.2, R62.2, RN1.2 (R2.1); no longer P1.44
- net IN_INJ3: now also R7.2, R8.2, C18.2, C7.2, R63.2, RN1.3 (R3.1), RN2.3 (R3.1); no longer P1.45
- net IN_INJ4: now also C19.2, R25.2, R27.2, C29.2, R64.2, RN1.4 (R4.1), RN2.4 (R4.1); no longer P1.46
- net IN_PUMP: now also R60.2; no longer P1.40
- net L1: now also C45.2, R70.2
- net L2: now also C46.2, R72.2
- net L3: now also C49.2, R76.2
- net L4: now also C50.2, R77.2
- net OA_1: now also U7.18 (PB0); no longer R27.2
- net OA_2: now also U7.19 (PB1)
- net OUT_INJ1_N: now also R70.1
- net OUT_INJ1_P: now also R71.1
- net OUT_INJ2_N: now also R72.1
- net OUT_INJ2_P: now also R73.1
- net OUT_INJ3_N: now also R76.1
- net OUT_INJ3_P: now also R78.1
- net OUT_INJ4_N: now also R77.1
- net OUT_INJ4_P: now also R79.1
- net OUT_LS1: now also R68.2; no longer P1.21, P1.22
- net OUT_LS2: now also R69.2; no longer P1.23, P1.24
- net OUT_PUMP_H: now also R75.1; no longer C63.2, C64.1, D16.1 (K), Q11.3 (S), U1.51 (S_HS5)
- net OUT_PUMP_L: now also R74.1; no longer D17.2 (A), Q12.2 (D), U1.33 (D_LS6)
- net RESETB: now also U7.41 (PB5), P4.1 (Pin_1); no longer R7.2
- net START1: now also U4.2
- net START2: now also U4.4
- net START3: now also U4.6; no longer R4.2
- net START4: now also U4.8; no longer R3.2
- net START5: now also U4.10
- net START6: now also U4.12
- net VCCP: now also C26.2, C28.2
- net Vbat: now also R36.2
- net Vdrive: now also D34.2 (K), R42.2, R43.2; no longer R10.1, R38.2
- net at Q10.3 (S), Q9.3 (S), R22.1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: now also C58.1, C11.2, C61.1; no longer C57.2, C58.2
- net at Q6.1 (G), R16.2: now also C57.2; no longer C38.1
- net at D11.3 (A), Q5.3 (S), U1.57 (S_HS3): now also C40.2, C56.1; no longer C37.2, C41.1
- net at R15.2: now also C56.2, Q5.1 (G); no longer U1.56 (G_HS3)
- net at U1.45 (G_LS3): now also R17.1; no longer R19.1
- net at R20.1: now also U1.42 (G_LS6); no longer U1.44 (G_LS4)
- net at L2.2, Q2.2 (D): now also D34.1 (A), D34.3 (A), R38.2; no longer R9.1
- net at Q2.1 (G): now also R24.1, C74.2; no longer R11.1
- net at Q2.3 (S): now also C21.2, C22.2, C25.2, C27.2, R12.1, TP23.1 (Pin_1), U1.32 (VSENSEP4), C24.2, C60.1, C73.1, C74.1
- net at R11.2: now also Q4.1 (G), C53.2; no longer U1.41 (G_LS7)
- net at R10.2: now also Q3.1 (G), C52.2
- net at U1.50 (G_HS5): now also R19.1; no longer R23.2
- net at Q12.3 (S), R26.1, U1.30 (VSENSEP3): now also C63.1, C13.2; no longer C71.2
- net at R24.2: now also U1.41 (G_LS7); no longer U1.42 (G_LS6)
- net at R45.2, U1.17 (VCCIO): now also C59.2
- net at U1.20 (VCC2P5): now also C32.2, C9.2
- net at U1.55 (B_HS3): now also C40.1; no longer C41.2
- net at U1.49 (B_HS5): now also C64.1; no longer C64.2
- net at U1.18 (DBG): now also P24.1 (Pin_1)
- net at C55.1, Q7.3 (S), Q8.3 (S)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: now also C10.2, C54.1; no longer C56.2
- net at C39.2, D10.3 (A), Q3.3 (S)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: now also C52.1; no longer C35.2
- net at R14.2: now also C55.2, Q7.1 (G); no longer U1.59 (G_HS2)
- net at R13.2: now also Q8.1 (G), C54.2; no longer U1.62 (G_HS1)
- net at R18.2: now also Q10.1 (G), C61.2; no longer U1.47 (G_LS1)
- net at R17.2: now also C58.2, Q9.1 (G); no longer U1.46 (G_LS2)
- net at U1.58 (B_HS2): now also C41.1; no longer C40.2
- net at U1.52 (B_HS4): now also C42.1; no longer C42.2
- net at D32.2 (A): now also R39.1
- net at D28.2 (A): now also R36.1
- net at D33.2 (A): now also R40.1
- net at Q1.2 (D): now also R55.2; no longer R42.1
- net at D31.1 (K): now also R55.1; no longer R42.2
- net at D30.1 (K), Q1.1 (G): now also D38.2 (A), R44.1; no longer R43.2, R44.2
- net at R43.1: now also D35.1 (K); no longer D38.2 (A)
- net at R38.1: now also C60.2; no longer D35.1 (K)
- net at P1.47: now also R64.1
- net at P1.48: now also P26.1 (Pin_1)
- net at P1.49: now also P27.1 (Pin_1)
- net at D21.1 (K): now also R23.2
- net at P1.115: now also P28.1 (Pin_1)
- net at P1.116: now also P29.1 (Pin_1)
- net at P1.117: now also P30.1 (Pin_1)
- net at P1.120: now also P31.1 (Pin_1)
- net at D20.1 (K): now also R9.1
- net at U7.2 (PC13): now also P8.1 (Pin_1)
- net at U7.21 (PB10): now also P13.1 (Pin_1)
- net at U7.22 (PB11): now also P14.1 (Pin_1)
- net at U7.25 (PB12): now also P15.1 (Pin_1)
- net at U7.27 (PB14): now also P16.1 (Pin_1)
- net at U7.28 (PB15): now also P17.1 (Pin_1)
- net at U7.3 (PC14): now also P9.1 (Pin_1)
- net at U7.38 (PA15): now also P25.1 (Pin_1)
- net at U7.4 (PC15): now also P10.1 (Pin_1)
- net at U7.45 (PB8): now also P11.1 (Pin_1)
- net at U7.46 (PB9): now also P12.1 (Pin_1)
- net at U7.5 (PD0): now also P6.1 (Pin_1)
- net at U7.6 (PD1): now also P7.1 (Pin_1)
- net FLAG_1: no longer names the net of U1.11 (FLAG1)
- net FLAG_1: now also P22.1 (Pin_1)
- net FLAG_2: no longer names the net of U1.12 (FLAG2)
- net FLAG_2: now also P23.1 (Pin_1)
- net IRQB: no longer names the net of U1.64 (IRQ)
- net IRQB: now also P21.1 (Pin_1)
- net LED_BLUE: no longer names the net of D20.2 (A), U7.26 (PB13)
- new net: C62.2, Q11.1 (G), R19.2
- new net: C63.2, Q12.1 (G), R20.2
- new net: P1.7, R67.1
- new net: C51.2, D8.4, RN2.5 (R4.2), U4.13
- new net: C73.2, R42.1
- new net: P1.53, R66.1
- new net: P1.44, R61.1
- new net: P1.21, P1.22, R68.1
- new net: P1.23, P1.24, R69.1
- new net: P1.40, R60.1
- new net: P1.45, R62.1
- new net: P1.46, R63.1
- new net: P1.52, R65.1
- new net: P1.6, R57.1
- new net: P1.8, R58.1
- new net: P1.9, R59.1
- new net: C35.2, D7.1, RN1.7 (R2.2), U4.3
- new net: C30.2, D7.3, RN1.8 (R1.2), U4.1
- new net: C38.2, D7.4, RN1.5 (R4.2), U4.9
- new net: C36.2, D7.6, RN1.6 (R3.2), U4.5
- new net: C37.2, D8.6, RN2.6 (R3.2), U4.11
- new net: R14.1, U1.46 (G_LS2)
- new net: R11.1, U1.59 (G_HS2)
- new net: R10.1, U1.62 (G_HS1)
- new net: R18.1, U1.44 (G_LS4)
- new net: R13.1, U1.47 (G_LS1)
- new net: R15.1, U1.56 (G_HS3)
- new net GNDD: J14.1 (Pin_1)
- new net H5: C62.1, C64.2, C65.2, D16.1 (K), Q11.3 (S), R75.2, U1.51 (S_HS5)
- new net L5: C67.2, D17.2 (A), Q12.2 (D), R74.2, U1.33 (D_LS6)
- no-connect marks 91 -> 94
Other:
- note removed: "Channels 5 and 6 in next rev"
- note removed: "IF REQURIED, R43 COULD BE A VOLT DIVIDER."
- note removed: "INJECTOR BOOSTED VOLTAGE"
- moved on the sheet: C14, C15, C16, C17, C2, C20, C21, C22, C25, C27, C3, C39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

Commit message: Upd PCB
Parts:
- removed C14, C15: 1000uF, Capacitors_ThroughHole:CP_Radial_D22.0mm_P10.00mm_SnapIn, symbol Device:CP1
- removed C16: 220nF, rusefi_lib:C_0805, symbol Device:C
- removed C21, C22: 390uF, Capacitors_ThroughHole:CP_Radial_D16.0mm_P7.50mm, symbol Device:CP1
- removed C25, C27: 0.22uF, rusefi_lib:C_0805, symbol Device:C
- removed D10, D11: SBR10200CTL, Package_TO_SOT_SMD:TO-252-2, symbol Device:D_Schottky_x2_KCom_AKA
- removed D12, D13, D14, D15, D16, D17: STPS2H100UY, Diodes_SMD:D_SMB, symbol Device:D_Small_ALT
- removed F1: Fuse, Fuse:Fuseholder_Blade_Mini_Keystone_3568, symbol Device:Fuse
- removed Q13: VBA2625, Package_SO:SOIC-8_3.9x4.9mm_P1.27mm, symbol Transistor_FET:IRF7404
- added C14, C15, C16, C21, C22, C25, C27, C83: 390uF, Capacitor_SMD:CP_Elec_16x17.5, symbol Device:C_Polarized_US
- added C80, C81, C82: 0.22uF, Capacitor_SMD:C_0805_2012Metric, symbol Device:C
- added D10, D11: SBR10200CTL, Package_TO_SOT_SMD:TO-252-2, symbol Device:D_Schottky_Dual_CommonCathode_AKA
- added D12, D13, D14, D15, D16, D9: STPS2H100UY, Diode_SMD:D_SMB, symbol Device:D_Schottky_Small
- added F1: Fuse-Pad-Pad, hellen-one-common:PAD-1206-PAD, symbol hellen-one-common:Fuse-Pad-Pad
- added Q13: AOD4185, Package_TO_SOT_SMD:TO-252-2, symbol Transistor_FET:QM6015D
- added R56: Jumper-Pad-Pad, hellen-one-common:PAD-0805-PAD, symbol hellen-one-common:Jumper-Pad-Pad
- C17: value 220nF -> 0.22uF; footprint rusefi_lib:C_0805 -> Capacitor_SMD:C_0805_2012Metric; LCSC C5378 -> C342873; MFG,MFG# KEMET,C0805C224M1RACTU -> (none); VEND1,VEND1# DIGI,399-9205-1-ND -> (none); VEND2,VEND2# , -> (none)
- J14: footprint Pin_Headers:Pin_Header_Straight_1x03_Pitch2.54mm -> Connector_PinHeader_2.54mm:PinHeader_1x03_P2.54mm_Vertical
- L1: value 6uH -> 6.8uH; footprint rusefi_lib:744710610-Inductor -> Inductor_SMD:L_Wuerth_HCI-1350; LCSC (none) -> C380073; MFG,MFG# Würth Elektronik,744710610 -> (none); VEND1,VEND1# DIGI,732-3255-ND -> (none); VEND2,VEND2# , -> (none)
- L2: footprint rusefi_lib:IHLP6767GZER100M01 -> Inductor_SMD:L_Vishay_IHLP-6767; LCSC (none) -> C237980; MFG,MFG# Vishay,IHLP6767GZER100M01 -> (none); VEND1,VEND1# DIGI,541-1259-1-ND -> (none); VEND2,VEND2# , -> (none)
- R41: value 10R -> 10; footprint rusefi_lib:R_0805 -> Resistor_SMD:R_0603_1608Metric; LCSC C17415 -> C22859; MFG,MFG# Stackpole,RMCF0805JG10R0 -> (none); VEND1,VEND1# DIGI,RMCF0805JG10R0CT-ND -> (none); VEND2,VEND2# JLCPCB,C17403 -> (none)
- U4: footprint (none) -> Package_SO:TSSOP-14_4.4x5mm_P0.65mm
- U4: footprint (none) -> Package_SO:TSSOP-14_4.4x5mm_P0.65mm; LCSC (none) -> C6821
- U7: LCSC (none) -> C8303
Connections:
- net +BATT: now also C17.1, C14.1, C15.1, C16.1, D16.1 (K), Q13.3 (S)
- net GND: now also R41.2, C14.2, C15.2, C16.2, C21.2, C22.2, C25.2, C80.2, D10.1 (A), D11.1 (A), D15.2 (A); no longer R41.1
- net H1: now also D10.2 (K)
- net H3: now also D11.2 (K)
- net H5: now also D15.1 (K)
- net IN_INJ3: no longer C18.2, R8.2, RN2.3 (R3.1)
- net IN_INJ4: no longer C29.2, R27.2, RN2.4 (R4.1)
- net L1: now also D9.2 (A)
- net L2: now also D12.2 (A)
- net L3: now also D13.2 (A)
- net L4: now also D14.2 (A)
- net L5: now also D16.2 (A)
- net Vdrive: now also C27.1, C81.1, C82.1, C83.1, D12.1 (K), D13.1 (K), D14.1 (K), D9.1 (K)
- net at C40.2, C56.1, Q5.3 (S)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: now also D11.3 (A)
- net at L1.2, L2.1: now also C21.1, C22.1, C25.1, C80.1; no longer C17.1
- net at C24.2, C60.1, C73.1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: now also C27.2, C81.2, C82.2, C83.2
- net at C39.2, C52.1, Q3.3 (S)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: now also D10.3 (A)
- net at Y2.1 (Vctrl): now also R41.1; no longer R41.2
- net at D4.2 (A), R2.2: now also Q13.1 (G)
- net at P1.41: now also R56.1
- net at D1.1 (A1): now also F1.2, Q13.2 (D)
- net at P1.4: now also F1.1
- net IN_PUMP renamed IN_PUMP2
- net IN_PUMP2: now also C29.2, R27.2, RN2.4 (R4.1)
- new net IN_PUMP1: C18.2, R56.2, R8.2, RN2.3 (R3.1)
- no-connect marks 94 -> 93
Other:
- note added: "Cap height 17mm"
- note added: "Non-JLC: EEE-TP1K391V"
- note removed: "TODO: check fuse & mosfet"
- moved on the sheet: C31, C33, C4, C60, C68, C73, C74, D1, D19, D2, D28, D3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

Commit message: Upd PCB
Parts:
- removed C2, C3: 47p, Capacitor_SMD:C_0402_1005Metric, symbol Device:C
- removed C20: 100n, Capacitor_SMD:C_0402_1005Metric, symbol Device:C
- removed C66, C69, C70, C72: 100nF, Capacitor_SMD:C_0402_1005Metric, symbol Device:C
- removed D30, D35, D36, D37, D38: 5.7V, Diode_SMD:D_MicroMELF_Handsoldering, symbol Device:D_Zener_Small
- removed J14: CONN_01X03, Connector_PinHeader_2.54mm:PinHeader_1x03_P2.54mm_Vertical, symbol Connector_Generic:Conn_01x03
- removed J15: CONN_01X01, Connector_Pin:Pin_D1.4mm_L8.5mm_W2.8mm_FlatFork, symbol Connector_Generic:Conn_01x01
- removed Q1: BUK9230-100B, Package_TO_SOT_SMD:TO-252-2, symbol Device:Q_NMOS_GDS
- removed R2: 10k, Resistor_SMD:R_0402_1005Metric, symbol Device:R
- removed R44: 10K, Resistor_SMD:R_0603_1608Metric, symbol Device:R
- removed R55: 1K, Resistor_SMD:R_0603_1608Metric, symbol Device:R
- removed TP1, TP2: TestPoint, Connector_PinHeader_2.54mm:PinHeader_1x01_P2.54mm_Horizontal, symbol Connector:TestPoint
- removed TP101, TP102, TP103, TP104, TP23, TP24, TP4, TP5, TP6, TP7, TP8: CONN_01X01, Connector_Pin:Pin_D0.7mm_L6.5mm_W1.8mm_FlatFork, symbol Connector_Generic:Conn_01x01
- added C2, C3: 47p, hellen-one-common:C0603, symbol hellen-one-common:Cap
- added C20, C66, C69, C70, C72: 100n, hellen-one-common:C0603, symbol hellen-one-common:Cap
- added J5: Conn_01x04, Connector_PinHeader_2.54mm:PinHeader_1x04_P2.54mm_Vertical, symbol Connector_Generic:Conn_01x04
- added P36: Pad, hellen-one-common:PAD-TH, symbol hellen-one-common:Pad
- added R2: 10k, hellen-one-common:R0603, symbol hellen-one-common:Res
- R28, R30, R32, R5: footprint Resistor_SMD:R_0402_1005Metric -> Resistor_SMD:R_0603_1608Metric
- R29, R31, R33, R6: footprint Resistor_SMD:R_0402_1005Metric -> Resistor_SMD:R_0603_1608Metric; LCSC C25790 -> C23178
- R37: value 1k -> 1K; footprint Resistor_SMD:R_0402_1005Metric -> Resistor_SMD:R_0603_1608Metric; LCSC C11702 -> C21190
Connections:
- net Vbat is gone; now on net +BATT: R36.2
- net +3V3: now also R40.2, J5.3 (Pin_3)
- net +5V: now also R28.1, R30.1, R32.1, R39.2, R5.1, C20.2, J5.2 (Pin_2); no longer R28.2, R30.2, R32.2, R5.2
- net +BATT: now also J5.1 (Pin_1)
- net 3.3V: no longer R40.2
- net Boot0: now also P36.1 (Pin_1)
- net CAN_H: now also C2.1
- net CAN_L: now also C3.2
- net GND: now also D31.1 (K), R37.2, C2.2, C20.1, C3.1, C66.1, C69.1, C70.1, C72.1, J5.4 (Pin_4), R2.1; no longer R37.1
- net IN_A0: now also R5.2; no longer R5.1
- net IN_A1: now also R28.2; no longer R28.1
- net IN_A2: now also R30.2; no longer R30.1
- net IN_A3: now also R32.2; no longer R32.1
- net +Batt_filtered: now reaches C21.1, C22.1, C25.1, C80.1, L1.2, L2.1
- net Vdrive_coil: now reaches D34.1 (A), D34.3 (A), L2.2, Q2.2 (D), R38.2
- net Vdrive_shunt: now reaches C24.2, C27.2, C60.1, C73.1, C74.1, C81.2, C82.2, C83.2, Q2.3 (S), R12.1, U1.32 (VSENSEP4)
- net at R43.1: now also D31.2 (A)
- net at D18.4, RN3.5 (R4.2), U6.3 (+): now also C72.2
- net at D19.1 (K): now also R37.1; no longer R37.2
- net at D4.2 (A), Q13.1 (G): now also R2.2
- net at D18.3, RN3.8 (R1.2), U6.12 (+): now also C66.2
- net at D18.6, RN3.6 (R3.2), U6.5 (+): now also C70.2
- net at D18.1, RN3.7 (R2.2), U6.10 (+): now also C69.2
- removed net 5V: D31.2 (A), R39.2
Other:
- moved on the sheet: D31

Commit message: PCB preview
Parts:
- removed R12, R21, R22, R26: 0R010, Resistor_SMD:R_1206_3216Metric_Pad1.30x1.75mm_HandSolder, symbol Device:R
- added G1: RUSEFI_LOGO, kicad6-libraries:rusefi_logo, symbol rusefi_logo:RUSEFI_LOGO
- added R12, R21, R22, R26: 0.01, kicad6-libraries:Shunt_1206, symbol Device:R_Shunt
Connections:
- net 3.3V is gone; now on net +3V3: C71.2, Y2.4 (VDD)
- net GND: now also R12.4, R21.4, R22.4, R26.4; no longer C10.1, C11.1, C13.1, C24.1, U1.25 (VSENSEN1), U1.27 (VSENSEN2), U1.29 (VSENSEN3), U1.31 (VSENSEN4)
- net Vdrive_shunt: now also R12.1; no longer C24.2, U1.32 (VSENSEP4)
- net at C58.1, C61.1, Q10.3 (S)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: now also R22.1; no longer C11.2, U1.28 (VSENSEP2)
- net at C63.1, Q12.3 (S): now also R26.1; no longer C13.2, U1.30 (VSENSEP3)
- net at C54.1, C55.1, Q7.3 (S)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: now also R21.1; no longer C10.2, U1.26 (VSENSEP1)
- new net: C10.2, R21.2, U1.26 (VSENSEP1)
- new net: C10.1, R21.3, U1.25 (VSENSEN1)
- new net: C13.1, R26.3, U1.29 (VSENSEN3)
- new net: C13.2, R26.2, U1.30 (VSENSEP3)
- new net: C24.1, R12.3, U1.31 (VSENSEN4)
- new net: C24.2, R12.2, U1.32 (VSENSEP4)
- new net: C11.1, R22.3, U1.27 (VSENSEN2)
- new net: C11.2, R22.2, U1.28 (VSENSEP2)
