File: GDI-4ch/GDI-4ch.kicad_sch (KiCad schematic)
At the start: 251 parts, among them J1 Conn_02x02_Odd_Even, J2 FTSH-107-01-F-DV-K, J3 TC2030, J4 Conn_01x06, J5 Conn_01x04, P1 368255-2, P10 Pad, P11 Pad, P12 Pad, P13 Pad, P14 Pad, P15 Pad, P16 Pad, P17 Pad, P18 Pad, P19 Pad, P2 Pad, P20 Pad, P21 Pad, P22 Pad, P23 Pad, P24 Pad, P25 Pad, P26 Pad, P27 Pad, P28 Pad, P29 Pad, P3 Pad, P30 Pad, P31 Pad, P36 Pad, P4 Pad, P5 Pad, P6 Pad, P7 Pad, P8 Pad, P9 Pad, Q10 BUK9230-100B, Q11 BUK9230-100B, Q12 BUK9230-100B, Q13 AOD4185, Q14 VND14NV04TR-E, Q15 VND14NV04TR-E, Q2 BUK9230-100B, Q3 BUK9230-100B, Q4 BUK9230-100B, Q5 BUK9230-100B, Q6 BUK9230-100B, Q7 BUK9230-100B, Q8 BUK9230-100B, Q9 BUK9230-100B, U1 MC33816, U2 TJA1051T-3, U3 LM78M05_TO252, U4 74HC14, U5 XC6206P332MR, U6 MCP6004, U7 STM32F103C6Tx, Y2 1MHz

Commit message: Fab preview
Parts:
- D12, D13, D14, D15, D16, D9: LCSC C157420 -> C163541
- Q10, Q11, Q12, Q2, Q3, Q4, Q5, Q6, Q7, Q8, Q9: LCSC C67277 -> C194346
- Q13: LCSC TO-252-2 -> C400894
Changed lines of the file:
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@@
     )
     (property "Value" "BUK9230-100B" (id 1) (at 327.66 289.56 0)
-      (effects (font (size 1.524 1.524)) (justify right))
+      (effects (font (size 1.524 1.524)) (justify right) hide)
     )
     (property "Footprint" "Package_TO_SOT_SMD:TO-252-2" (id 2) (at 503.428 271.78 90)
@@
       (effects (font (size 1.524 1.524)) hide)
     )
-    (property "LCSC" "C67277 " (id 7) (at 328.93 293.37 0)
+    (property "LCSC" "C194346" (id 7) (at 328.93 293.37 0)
       (effects (font (size 1.27 1.27)) hide)
     )
@@
     )
     (property "Value" "BUK9230-100B" (id 1) (at 327.66 274.32 0)
-      (effects (font (size 1.524 1.524)) (justify right))
+      (effects (font (size 1.524 1.524)) (justify right) hide)
     )
     (property "Footprint" "Package_TO_SOT_SMD:TO-252-2" (id 2) (at 536.448 243.205 90)
@@
       (effects (font (size 1.524 1.524)) hide)
     )
-    (property "LCSC" "C67277 " (id 7) (at 328.93 278.13 0)
+    (property "LCSC" "C194346" (id 7) (at 328.93 278.13 0)
       (effects (font (size 1.27 1.27)) hide)
     )
@@
     )
     (property "Value" "BUK9230-100B" (id 1) (at 327.66 304.8 0)
-      (effects (font (size 1.524 1.524)) (justify right))
+      (effects (font (size 1.524 1.524)) (justify right) hide)
     )
     (property "Footprint" "Package_TO_SOT_SMD:TO-252-2" (id 2) (at 503.428 317.5 90)
@@
       (effects (font (size 1.524 1.524)) hide)
     )
-    (property "LCSC" "C67277 " (id 7) (at 328.93 308.61 0)
+    (property "LCSC" "C194346" (id 7) (at 328.93 308.61 0)
       (effects (font (size 1.27 1.27)) hide)
     )
@@
     )
     (property "Value" "BUK9230-100B" (id 1) (at 327.66 320.04 0)
-      (effects (font (size 1.524 1.524)) (justify right))
+      (effects (font (size 1.524 1.524)) (justify right) hide)
     )
     (property "Footprint" "Package_TO_SOT_SMD:TO-252-2" (id 2) (at 536.448 346.71 90)
@@
       (effects (font (size 1.524 1.524)) hide)
     )
-    (property "LCSC" "C67277 " (id 7) (at 328.93 323.85 0)
+    (property "LCSC" "C194346" (id 7) (at 328.93 323.85 0)
       (effects (font (size 1.27 1.27)) hide)
     )
@@
     )
     (property "Value" "BUK9230-100B" (id 1) (at 327.66 347.98 0)
-      (effects (font (size 1.524 1.524)) (justify right))
+      (effects (font (size 1.524 1.524)) (justify right) hide)
     )
     (property "Footprint" "Package_TO_SOT_SMD:TO-252-2" (id 2) (at 384.048 403.86 90)
@@
       (effects (font (size 1.524 1.524)) hide)
     )
-    (property "LCSC" "C67277 " (id 7) (at 328.93 351.79 0)
+    (property "LCSC" "C194346" (id 7) (at 328.93 351.79 0)
       (effects (font (size 1.27 1.27)) hide)
     )
@@
       (effects (font (size 1.524 1.524)) hide)
     )
-    (property "LCSC" "C67277 " (id 7) (at 486.41 325.12 0)
+    (property "LCSC" "C194346" (id 7) (at 486.41 325.12 0)
       (effects (font (size 1.27 1.27)) hide)
     )
@@
     )
     (property "Value" "BUK9230-100B" (id 1) (at 327.66 378.46 0)
-      (effects (font (size 1.524 1.524)) (justify right))
+      (effects (font (size 1.524 1.524)) (justify right) hide)
     )
     (property "Footprint" "Package_TO_SOT_SMD:TO-252-2" (id 2) (at 384.048 459.74 90)
@@
       (effects (font (size 1.524 1.524)) hide)
     )
-    (property "LCSC" "C67277 " (id 7) (at 328.93 382.27 0)
+    (property "LCSC" "C194346" (id 7) (at 328.93 382.27 0)
       (effects (font (size 1.27 1.27)) hide)
     )
@@
     )
     (property "Value" "BUK9230-100B" (id 1) (at 328.93 215.9 0)
-      (effects (font (size 1.524 1.524)) (justify right))
+      (effects (font (size 1.524 1.524)) (justify right) hide)
     )
     (property "Footprint" "Package_TO_SOT_SMD:TO-252-2" (id 2) (at 381.508 198.12 90)
@@
       (effects (font (size 1.524 1.524)) hide)
     )
-    (property "LCSC" "C67277 " (id 7) (at 328.93 219.71 0)
+    (property "LCSC" "C194346" (id 7) (at 328.93 219.71 0)
       (effects (font (size 1.27 1.27)) hide)
     )
@@
     )
     (property "Value" "BUK9230-100B" (id 1) (at 327.66 200.66 0)
-      (effects (font (size 1.524 1.524)) (justify right))
+      (effects (font (size 1.524 1.524)) (justify right) hide)
     )
     (property "Footprint" "Package_TO_SOT_SMD:TO-252-2" (id 2) (at 348.488 169.545 90)
@@
       (effects (font (size 1.524 1.524)) hide)
     )
-    (property "LCSC" "C67277 " (id 7) (at 328.93 204.47 0)
+    (property "LCSC" "C194346" (id 7) (at 328.93 204.47 0)
       (effects (font (size 1.27 1.27)) hide)
     )
@@
     )
     (property "Value" "BUK9230-100B" (id 1) (at 327.66 231.14 0)
-      (effects (font (size 1.524 1.524)) (justify right))
+      (effects (font (size 1.524 1.524)) (justify right) hide)
     )
     (property "Footprint" "Package_TO_SOT_SMD:TO-252-2" (id 2) (at 381.508 243.84 90)
@@
       (effects (font (size 1.524 1.524)) hide)
     )
-    (property "LCSC" "C67277 " (id 7) (at 328.93 234.95 0)
+    (property "LCSC" "C194346" (id 7) (at 328.93 234.95 0)
       (effects (font (size 1.27 1.27)) hide)
     )
@@
     )
     (property "Value" "BUK9230-100B" (id 1) (at 327.66 246.38 0)
-      (effects (font (size 1.524 1.524)) (justify right))
+      (effects (font (size 1.524 1.524)) (justify right) hide)
     )
     (property "Footprint" "Package_TO_SOT_SMD:TO-252-2" (id 2) (at 348.488 273.05 90)
@@
       (effects (font (size 1.524 1.524)) hide)
     )
-    (property "LCSC" "C67277 " (id 7) (at 328.93 250.19 0)
+    (property "LCSC" "C194346" (id 7) (at 328.93 250.19 0)
       (effects (font (size 1.27 1.27)) hide)
     )
@@
       (effects (font (size 1.27 1.27)) hide)
     )
-    (property "LCSC" "C157420" (id 4) (at 308.61 377.19 0)
+    (property "LCSC" "C163541" (id 4) (at 308.61 377.19 0)
       (effects (font (size 1.524 1.524)) hide)
     )
@@
       (effects (font (size 1.27 1.27)) hide)
     )
-    (property "LCSC" "C157420" (id 4) (at 308.61 303.53 0)
+    (property "LCSC" "C163541" (id 4) (at 308.61 303.53 0)
       (effects (font (size 1.524 1.524)) hide)
     )
@@
       (effects (font (size 1.27 1.27)) hide)
     )
-    (property "LCSC" "C157420" (id 4) (at 308.61 359.41 0)
+    (property "LCSC" "C163541" (id 4) (at 308.61 359.41 0)
       (effects (font (size 1.524 1.524)) hide)
     )
@@
       (effects (font (size 1.27 1.27)) (justify left) hide)
     )
-    (property "LCSC" "TO-252-2" (id 4) (at 85.09 26.67 0)
+    (property "LCSC" "C400894" (id 4) (at 85.09 26.67 0)
       (effects (font (size 1.524 1.524)) hide)
     )
@@
       (effects (font (size 1.27 1.27)) hide)
     )
-    (property "LCSC" "C157420" (id 4) (at 308.61 245.11 0)
+    (property "LCSC" "C163541" (id 4) (at 308.61 245.11 0)
       (effects (font (size 1.524 1.524)) hide)
     )
@@
       (effects (font (size 1.27 1.27)) hide)
     )
-    (property "LCSC" "C157420" (id 4) (at 308.61 318.77 0)
+    (property "LCSC" "C163541" (id 4) (at 308.61 318.77 0)
       (effects (font (size 1.524 1.524)) hide)
     )
@@
       (effects (font (size 1.27 1.27)) hide)
     )
-    (property "LCSC" "C157420" (id 4) (at 308.61 229.87 0)
+    (property "LCSC" "C163541" (id 4) (at 308.61 229.87 0)
       (effects (font (size 1.524 1.524)) hide)
     )

Commit message: Fab preview 2
Parts:
- removed P12, P13, P14, P15, P16, P17, P21, P22, P23, P24: Pad, hellen-one-common:PAD-TH, symbol hellen-one-common:Pad
- added P32: Pad, hellen-one-common:PAD-TH, symbol hellen-one-common:Pad
- added R44, R55, R80, R81, R82, R83: Jumper-Pad-Pad, hellen-one-common:PAD-0805-PAD, symbol hellen-one-common:Jumper-Pad-Pad
- U7: value STM32F103C6Tx -> STM32F103C8Tx; LCSC C8303 -> C8734
- renumbered R60 to R56, R56 to R60
Connections:
- net +5V: now also P1.11, P1.30
- net IN_PUMP1: now also R56.2, R55.1; no longer R60.2
- net IN_PUMP2: now also R60.2, R44.1; no longer R56.2
- net Vdrive: now also P32.1 (Pin_1)
- net at P1.40: now also R60.1; no longer R56.1
- net at P1.41: now also R56.1; no longer R60.1
- net at U1.64 (IRQ): now also R80.1
- net FLAG_1: now reaches U7.21 (PB10)
- net FLAG_1: now also R81.2
- net at U1.11 (FLAG1): now also R81.1
- net at U1.12 (FLAG2): now also R82.1
- net at U1.18 (DBG): now also R83.1
- net IRQ: now reaches U7.46 (PB9)
- net IRQ: now also R80.2
- net FLAG_2: now reaches U7.22 (PB11)
- net FLAG_2: now also R82.2
- net DBG: now reaches U7.25 (PB12)
- net DBG: now also R83.2
- net at U7.27 (PB14): now also R44.2
- net at U7.28 (PB15): now also R55.2
- net OUT_PUMP_H renamed OUT_PUMP_P
- net OUT_PUMP_L renamed OUT_PUMP_N
- no-connect marks 93 -> 91
Other:
- moved on the sheet: R56, R60
