File: GDI-4ch/GDI-4ch.kicad_sch (KiCad schematic)
At the start: 274 parts, among them J1 Conn_02x02_Odd_Even, J2 FTSH-107-01-F-DV-K, J3 TC2030, J4 Conn_01x06, J5 Conn_01x04, P1 368255-2, P10 Pad, P18 Pad, P19 Pad, P2 Pad, P20 Pad, P25 Pad, P3 Pad, P32 Pad, P36 Pad, P4 Pad, P5 Pad, P8 Pad, P9 Pad, Q1 BUK9230-100B, Q10 BUK9230-100B, Q11 BUK9230-100B, Q12 BUK9230-100B, Q13 AOD4185, Q14 VND14NV04TR-E, Q15 VND14NV04TR-E, Q16 BUK9230-100B, Q2 BUK9230-100B, Q3 BUK9230-100B, Q4 BUK9230-100B, Q5 BUK9230-100B, Q6 BUK9230-100B, Q7 BUK9230-100B, Q8 BUK9230-100B, Q9 BUK9230-100B, U1 MC33816, U2 TJA1051T-3, U3 LM78M05_TO252, U4 74HC14, U5 XC6206P332MR, U6 MCP6004, U7 GD32F103CBT6, Y1 8MHz, Y2 1MHz

Commit message: #125
Parts:
- removed P10, P25, P8, P9: Pad, hellen-one-common:PAD-TH, symbol hellen-one-common:Pad
- added C100, C101, C93, C94, C95, C96, C98, C99: 1000pF, Capacitor_SMD:C_0603_1608Metric, symbol Device:C
- added C97: 100n, hellen-one-common:C0603, symbol hellen-one-common:Cap
- added D22: SRV05-4, Package_TO_SOT_SMD:SOT-23-6, symbol Power_Protection:NUP4202
- added R101, R102, R103, R104: 1K, Resistor_SMD:R_0603_1608Metric, symbol Device:R
- added R105, R106, R107, R108: 10k, hellen-one-common:R0603, symbol hellen-one-common:Res
- added R109, R110, R111, R112: Jumper-Pad-Pad, hellen-one-common:PAD-0805-PAD, symbol hellen-one-common:Jumper-Pad-Pad
- added R113, R114, R115, R116: 0, Resistor_SMD:R_0603_1608Metric, symbol Device:R
- added R117, R118, R119, R120: DNP, Resistor_SMD:R_0603_1608Metric, symbol Device:R
- added U8: 74HC14, Package_SO:TSSOP-14_4.4x5mm_P0.65mm, symbol 74xx:74HC14
Connections:
- net +3V3: now also C97.2, D22.5, R101.1, R102.1, R103.1, R104.1, U8.14 (VCC)
- net GND: now also C100.1, C101.1, C93.1, C94.1, C95.1, C96.1, C97.1, C98.1, C99.1, D22.2, R117.1, R118.1, R119.1, R120.1, U8.11, U8.13, U8.7 (GND)
- net at U7.38 (PA15): now also R116.2
- net at P1.17: now also R109.1
- net at P1.18: now also R110.1
- net at P1.36: now also R111.1
- net at P1.37: now also R112.1
- net at U7.2 (PC13): now also R113.1
- net at U7.3 (PC14): now also R114.1
- net at U7.4 (PC15): now also R115.1
- new net: C98.2, D22.3, R105.1, U8.1
- new net: C99.2, D22.1, R106.1, U8.3
- new net: C101.2, D22.4, R108.1, U8.9
- new net: C100.2, D22.6, R107.1, U8.5
- new net DIN1: R113.2, U8.2
- new net DIN2: R114.2, U8.4
- new net DIN3: R115.2, U8.6
- new net DIN4: R116.1, U8.8
- new net IN_DIN1: C93.2, R101.2, R105.2, R109.2, R117.2
- new net IN_DIN2: C94.2, R102.2, R106.2, R110.2, R118.2
- new net IN_DIN3: C95.2, R103.2, R107.2, R111.2, R119.2
- new net IN_DIN4: C96.2, R104.2, R108.2, R112.2, R120.2
- no-connect marks 88 -> 86
Other:
- moved on the sheet: C1, C18, C19, C2, C20, C29, C3, C30, C35, C36, C37, C38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

Commit message: #125 part 2
Parts:
- added R121: DNP, hellen-one-common:PAD-0805-PAD, symbol hellen-one-common:Jumper-Pad-Pad
- added R122: Jumper-Pad-Pad, hellen-one-common:PAD-0805-PAD, symbol hellen-one-common:Jumper-Pad-Pad
Connections:
- net A0: now also R121.2; no longer U7.10 (PA0)
- net DIN1: now also R122.2
- net LS2: now also U7.38 (PA15); no longer U7.42 (PB6)
- net VCC2P5: now also U7.10 (PA0); no longer U7.11 (PA1)
- net at R116.2: now also U7.42 (PB6); no longer U7.38 (PA15)
- new net: R121.1, R122.1, U7.11 (PA1)
Other:
- moved on the sheet: R116
Changed lines of the file:
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@@
   (title_block
     (title "GDI 4ch")
-    (date "2022-07-18")
+    (date "2022-07-22")
     (rev "rev. c")
     (company "rusEFI.com")
@@
   (junction (at 502.92 248.92) (diameter 0) (color 0 0 0 0)
   )
+  (junction (at 415.29 73.66) (diameter 0) (color 0 0 0 0)
+  )
   (junction (at 183.515 156.845) (diameter 0) (color 0 0 0 0)
   )
@@
     (stroke (width 0) (type default) (color 0 0 0 0))
   )
-  (wire (pts (xy 398.78 73.66) (xy 411.48 73.66))
+  (wire (pts (xy 398.78 71.12) (xy 411.48 71.12))
     (stroke (width 0) (type default) (color 0 0 0 0))
   )
@@
     (stroke (width 0) (type default) (color 0 0 0 0))
   )
-  (wire (pts (xy 365.76 86.36) (xy 353.06 86.36))
+  (wire (pts (xy 340.995 86.36) (xy 365.76 86.36))
     (stroke (width 0) (type default) (color 0 0 0 0))
   )
@@
     (stroke (width 0) (type default) (color 0 0 0 0))
   )
+  (wire (pts (xy 429.26 76.2) (xy 437.515 76.2))
+    (stroke (width 0) (type default) (color 0 0 0 0))
+  )
   (wire (pts (xy 231.775 123.825) (xy 224.155 123.825))
     (stroke (width 0) (type default) (color 0 0 0 0))
@@
     (stroke (width 0) (type default) (color 0 0 0 0))
   )
+  (wire (pts (xy 419.1 76.2) (xy 415.29 76.2))
+    (stroke (width 0) (type default) (color 0 0 0 0))
+  )
   (wire (pts (xy 54.61 172.72) (xy 67.31 172.72))
     (stroke (width 0) (type default) (color 0 0 0 0))
@@
     (stroke (width 0) (type default) (color 0 0 0 0))
   )
-  (wire (pts (xy 398.78 71.12) (xy 411.48 71.12))
+  (wire (pts (xy 398.78 73.66) (xy 415.29 73.66))
     (stroke (width 0) (type default) (color 0 0 0 0))
   )
@@
     (stroke (width 0) (type default) (color 0 0 0 0))
   )
+  (wire (pts (xy 429.26 73.66) (xy 437.515 73.66))
+    (stroke (width 0) (type default) (color 0 0 0 0))
+  )
   (wire (pts (xy 330.2 313.69) (xy 345.44 313.69))
     (stroke (width 0) (type default) (color 0 0 0 0))
@@
     (stroke (width 0) (type default) (color 0 0 0 0))
   )
+  (wire (pts (xy 415.29 76.2) (xy 415.29 73.66))
+    (stroke (width 0) (type default) (color 0 0 0 0))
+  )
   (wire (pts (xy 355.6 344.17) (xy 359.41 344.17))
     (stroke (width 0) (type default) (color 0 0 0 0))
@@
     (stroke (width 0) (type default) (color 0 0 0 0))
   )
-  (wire (pts (xy 416.56 109.22) (xy 409.575 109.22))
+  (wire (pts (xy 326.39 86.36) (xy 333.375 86.36))
+    (stroke (width 0) (type default) (color 0 0 0 0))
+  )
+  (wire (pts (xy 415.29 73.66) (xy 419.1 73.66))
     (stroke (width 0) (type default) (color 0 0 0 0))
   )
@@
     (stroke (width 0) (type default) (color 0 0 0 0))
   )
-  (wire (pts (xy 401.955 109.22) (xy 398.78 109.22))
+  (wire (pts (xy 411.48 109.22) (xy 398.78 109.22))
     (stroke (width 0) (type default) (color 0 0 0 0))
   )
@@
     (effects (font (size 1.524 1.524)) (justify left bottom))
   )
-  (label "A0" (at 411.48 71.12 180)
+  (label "A0" (at 437.515 73.66 180)
     (effects (font (size 1.524 1.524)) (justify right bottom))
   )
@@
     (effects (font (size 1.524 1.524)) (justify left bottom))
   )
-  (label "DIN4" (at 416.56 109.22 180)
-    (effects (font (size 1.524 1.524)) (justify right bottom))
+  (label "DIN4" (at 326.39 86.36 0)
+    (effects (font (size 1.524 1.524)) (justify left bottom))
   )
   (label "START4" (at 257.175 123.825 180)
@@
     (effects (font (size 1.27 1.27)) (justify left bottom))
   )
+  (label "DIN1" (at 437.515 76.2 180)
+    (effects (font (size 1.524 1.524)) (justify right bottom))
+  )
   (label "L4" (at 295.91 265.43 0)
     (effects (font (size 1.524 1.524)) (justify left bottom))
@@
     (effects (font (size 1.524 1.524)) (justify left bottom))
   )
-  (label "LS2" (at 353.06 86.36 0)
-    (effects (font (size 1.524 1.524)) (justify left bottom))
+  (label "LS2" (at 411.48 109.22 180)
+    (effects (font (size 1.524 1.524)) (justify right bottom))
   )
   (label "A3" (at 411.48 81.28 180)
@@
     (effects (font (size 1.27 1.27)) (justify right bottom))
   )
-  (label "VCC2P5" (at 411.48 73.66 180)
+  (label "VCC2P5" (at 411.48 71.12 180)
     (effects (font (size 1.524 1.524)) (justify right bottom))
   )
@@
     (pin "1")
   )
+  (symbol (lib_id "hellen-one-common:Jumper-Pad-Pad") (at 424.18 76.2 0) (unit 1)
+    (in_bom yes) (on_board yes)
+    (property "Reference" "R122" (id 0) (at 429.26 74.93 0)
+      (effects (font (size 1.016 1.016)))
+    )
+    (property "Value" "Jumper-Pad-Pad" (id 1) (at 424.18 77.978 0)
+      (effects (font (size 1.016 1.016)) hide)
+    )
+    (property "Footprint" "hellen-one-common:PAD-0805-PAD" (id 2) (at 424.18 80.01 0)
+      (effects (font (size 1.524 1.524)) hide)
+    )
+    (property "Datasheet" "" (id 3) (at 424.18 76.2 0)
+      (effects (font (size 1.524 1.524)) hide)
+    )
+    (property "LCSC" "C17477" (id 4) (at 424.18 80.01 0)
+      (effects (font (size 1.27 1.27)) hide)
+    )
+    (pin "1")
+    (pin "2")
+  )
   (symbol (lib_id "power:GND") (at 192.405 236.855 0) (unit 1)
     (in_bom yes) (on_board yes)
@@
     (pin "1")
   )
-  (symbol (lib_id "Device:R") (at 405.765 109.22 270) (unit 1)
+  (symbol (lib_id "Device:R") (at 337.185 86.36 90) (mirror x) (unit 1)
     (in_bom yes) (on_board yes)
-    (property "Reference" "R116" (id 0) (at 400.05 108.585 90)
+    (property "Reference" "R116" (id 0) (at 342.9 85.725 90)
       (effects (font (size 1.016 1.016)))
     )
-    (property "Value" "0" (id 1) (at 405.7904 109.3978 90)
+    (property "Value" "0" (id 1) (at 337.1596 86.5378 90)
       (effects (font (size 1.016 1.016)))
     )
-    (property "Footprint" "Resistor_SMD:R_0603_1608Metric" (id 2) (at 385.445 155.067 90)
+    (property "Footprint" "Resistor_SMD:R_0603_1608Metric" (id 2) (at 357.505 132.207 90)
       (effects (font (size 1.524 1.524)) hide)
     )
-    (property "Datasheet" "" (id 3) (at 386.08 244.475 0)
+    (property "Datasheet" "" (id 3) (at 356.87 221.615 0)
       (effects (font (size 1.524 1.524)) hide)
     )
-    (property "LCSC" "C21189" (id 4) (at 405.765 109.22 0)
+    (property "LCSC" "C21189" (id 4) (at 337.185 86.36 0)
       (effects (font (size 1.27 1.27)) hide)
     )
@@
     (pin "1")
   )
+  (symbol (lib_id "hellen-one-common:Jumper-Pad-Pad") (at 424.18 73.66 0) (unit 1)
+    (in_bom yes) (on_board yes)
+    (property "Reference" "R121" (id 0) (at 429.26 72.39 0)
+      (effects (font (size 1.016 1.016)))
+    )
+    (property "Value" "DNP" (id 1) (at 424.18 73.66 0)
+      (effects (font (size 1.016 1.016)))
+    )
+    (property "Footprint" "hellen-one-common:PAD-0805-PAD" (id 2) (at 424.18 77.47 0)
+      (effects (font (size 1.524 1.524)) hide)
+    )
+    (property "Datasheet" "" (id 3) (at 424.18 73.66 0)
+      (effects (font (size 1.524 1.524)) hide)
+    )
+    (property "LCSC" "" (id 4) (at 424.18 77.47 0)
+      (effects (font (size 1.27 1.27)) hide)
+    )
+    (pin "1")
+    (pin "2")
+  )
   (symbol (lib_id "power:+3.3V") (at 125.73 52.07 180) (unit 1)
     (in_bom yes) (on_board yes)
@@
       (reference "R120") (unit 1) (value "DNP") (footprint "Resistor_SMD:R_0603_1608Metric")
     )
+    (path "/e2674f39-2445-4e92-86ee-82a58b1d5f68"
+      (reference "R121") (unit 1) (value "DNP") (footprint "hellen-one-common:PAD-0805-PAD")
+    )
+    (path "/d1170cb1-0024-4094-9958-5d3f50eb2921"
+      (reference "R122") (unit 1) (value "Jumper-Pad-Pad") (footprint "hellen-one-common:PAD-0805-PAD")
+    )
     (path "/39c4e0a0-bf4a-4a70-8602-0df444eb3d47"

Commit message: Upd SCH, PCB
Parts:
- removed C22, C25, C27, C83: 390uF, Capacitor_SMD:CP_Elec_16x17.5, symbol Device:C_Polarized_US
- added R123, R124, R125: 1K, Resistor_SMD:R_0603_1608Metric, symbol Device:R
- added R126, R127: 2K, Resistor_SMD:R_1206_3216Metric, symbol Device:R
- added R128, R129, R130, R131, R132, R133, R134, R135, R136: 56k, Resistor_SMD:R_0805_2012Metric, symbol Device:R
- C14, C15: value 390uF -> 1200uF; footprint Capacitor_SMD:CP_Elec_16x17.5 -> Capacitor_THT:C_Radial_D16.0mm_H25.0mm_P7.50mm; LCSC C487421 -> C5111952
- C16, C21: value 390uF -> 470uF; footprint Capacitor_SMD:CP_Elec_16x17.5 -> Capacitor_THT:C_Radial_D16.0mm_H25.0mm_P7.50mm; LCSC C487421 -> C5110766
- J1: LCSC (none) -> C66690
- J4: LCSC (none) -> C5156615
- R38: value 5.1 -> 220; LCSC C25197 -> C22962
Connections:
- net +BATT: no longer C15.1, C16.1
- net +Batt_filtered: now also C15.1, R126.1, R127.1; no longer C21.1
- net DRVEN: now also R123.1
- net FLAG_0: now also R125.1
- net GND: now also R123.2, R124.2, R125.2, R126.2, R127.2; no longer C16.2, C21.2
- net RESETB: now also R124.1
- net Vdrive: now also C16.1, C21.1, R128.1, R129.1, R130.1, R131.1, R132.1, R133.1, R134.1, R135.1, R136.1
- net Vdrive_shunt: now also C16.2, C21.2, R128.2, R129.2, R130.2, R131.2, R132.2, R133.2, R134.2, R135.2, R136.2
Other:
- note added: "22V MAX"
- note added: "Discharge circuit"
- note added: "OUT"
- note removed: "Cap height 17mm"
- note removed: "Non-JLC: EEE-TP1K391V"
- moved on the sheet: C14, C71, Y2

Commit message: 4ch+1
Parts:
- removed R90: DNP, hellen-one-common:PAD-0805-PAD, symbol hellen-one-common:Jumper-Pad-Pad
- R37, R87, R89: value DNP -> Jumper-Pad-Pad; LCSC (none) -> C17477
- R41, R88: value Jumper-Pad-Pad -> DNP; LCSC C17477 -> (none)
- U5: footprint Package_TO_SOT_SMD:SOT-23 -> Package_TO_SOT_SMD:SOT-23-3
Connections:
- net +3V3 renamed +3.3V
- net IN_PUMP1 renamed IN_PUMP
- net IN_PUMP2: no longer names the net of P1.40
- no-connect marks 86 -> 87
Other:
- note added: "4ch+1 6ch R87 + DNP R37 + DNP R41 DNP + R88 DNP + R89 + DNP"
- note added: "This board could either drive 4 injectors and one SCV/PUMP, or 6 injectors. In 6 injectors mode we are limited at 120 degrees injection angle"
- moved on the sheet: R91
