File: GDI-4ch/GDI-4ch.kicad_sch (KiCad schematic)
At the start: 312 parts, among them J1 Conn_02x02_Odd_Even, J2 FTSH-107-01-F-DV-K, J3 TC2030, J4 Conn_01x06, J5 Conn_01x04, P1 368255-2, P18 Pad, P19 Pad, P2 Pad, P20 Pad, P3 Pad, P32 Pad, P36 Pad, P4 Pad, P5 Pad, Q1 BUK9230-100B, Q10 BUK9230-100B, Q11 BUK9230-100B, Q12 BUK9230-100B, Q13 AOD4185, Q14 VND14NV04TR-E, Q15 VND14NV04TR-E, Q16 BUK9230-100B, Q2 BUK9230-100B, Q3 BUK9230-100B, Q4 BUK9230-100B, Q5 BUK9230-100B, Q6 BUK9230-100B, Q7 BUK9230-100B, Q8 BUK9230-100B, Q9 BUK9230-100B, U1 MC33816, U2 TJA1051T-3, U3 LM78M05_TO252, U4 74HC14, U5 XC6206P332MR, U6 MCP6004, U7 GD32F103CBT6, U8 74HC14, Y1 8MHz, Y2 1MHz

Commit message: GDI-4ch-d export
Parts:
- C74: LCSC C326973 -> C525649
- R121: value DNP -> Jumper-Pad-Pad; LCSC (none) -> C17477
- R122: value Jumper-Pad-Pad -> DNP; LCSC C17477 -> (none)
- U4: value 74HC14 -> 74HC14PW,118; LCSC (none) -> C5606
- U4, U8: value 74HC14 -> 74HC14PW,118
- U8: value 74HC14 -> 74HC14PW,118; LCSC C5606 -> (none)
- Y2: LCSC C70608 -> C2901463
Other:
- note added: "Use R122 option without R113, R121 for SENT"
Changed lines of the file:
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@@
     (effects (font (size 1.524 1.524)) (justify right bottom))
   )
+  (text "Use R122 option without R113, R121 for SENT" (at 469.9 80.645 0)
+    (effects (font (size 1.524 1.524)) (justify right bottom))
+  )
   (text "rev. a: STTH802G-TR" (at 518.16 275.59 0)
     (effects (font (size 1.27 1.27)) (justify left bottom))
@@
       (effects (font (size 1.524 1.524)) hide)
     )
-    (property "LCSC" "C70608" (at 499.11 143.51 0)
+    (property "LCSC" "C2901463" (at 499.11 143.51 0)
       (effects (font (size 1.27 1.27)) hide)
     )
@@
       (effects (font (size 1.27 1.27)))
     )
-    (property "Value" "74HC14" (at 245.745 136.525 0)
+    (property "Value" "74HC14PW,118" (at 247.015 136.525 0)
       (effects (font (size 1.27 1.27)))
     )
@@
       (effects (font (size 1.27 1.27)) hide)
     )
+    (property "LCSC" "C5606" (at 239.395 139.065 0)
+      (effects (font (size 1.524 1.524)) hide)
+    )
     (pin "1")
     (pin "2")
@@
       (effects (font (size 1.27 1.27)))
     )
-    (property "Value" "74HC14" (at 224.155 240.665 0)
+    (property "Value" "74HC14PW,118" (at 226.06 240.665 0)
       (effects (font (size 1.27 1.27)))
     )
@@
       (effects (font (size 1.27 1.27)))
     )
-    (property "Value" "74HC14" (at 224.155 225.425 0)
+    (property "Value" "74HC14PW,118" (at 226.06 225.425 0)
       (effects (font (size 1.27 1.27)))
     )
@@
       (effects (font (size 1.27 1.27)))
     )
-    (property "Value" "74HC14" (at 245.745 106.045 0)
+    (property "Value" "74HC14PW,118" (at 247.015 106.045 0)
       (effects (font (size 1.27 1.27)))
     )
@@
       (effects (font (size 1.27 1.27)) hide)
     )
+    (property "LCSC" "C5606" (at 239.395 108.585 0)
+      (effects (font (size 1.524 1.524)) hide)
+    )
     (pin "1")
     (pin "2")
@@
     )
   )
+  (symbol (lib_id "hellen-one-common:Jumper-Pad-Pad") (at 424.18 73.66 0) (unit 1)
+    (in_bom yes) (on_board yes) (dnp no)
+    (property "Reference" "R121" (at 429.26 72.39 0)
+      (effects (font (size 1.016 1.016)))
+    )
+    (property "Value" "Jumper-Pad-Pad" (at 424.18 75.438 0)
+      (effects (font (size 1.016 1.016)) hide)
+    )
+    (property "Footprint" "hellen-one-common:PAD-0805-PAD" (at 424.18 77.47 0)
+      (effects (font (size 1.524 1.524)) hide)
+    )
+    (property "Datasheet" "" (at 424.18 73.66 0)
+      (effects (font (size 1.524 1.524)) hide)
+    )
+    (property "LCSC" "C17477" (at 424.18 77.47 0)
+      (effects (font (size 1.27 1.27)) hide)
+    )
+    (pin "1")
+    (pin "2")
+    (instances
+      (project "GDI-4ch"
+        (path "/03caada9-9e22-4e2d-9035-b15433dfbb17"
+          (reference "R121") (unit 1)
+        )
+      )
+    )
+  )
   (symbol (lib_id "power:GND") (at 469.9 179.07 0) (unit 1)
     (in_bom yes) (on_board yes) (dnp no)
@@
       (effects (font (size 1.27 1.27)))
     )
-    (property "Value" "74HC14" (at 224.155 210.185 0)
+    (property "Value" "74HC14PW,118" (at 226.06 210.185 0)
       (effects (font (size 1.27 1.27)))
     )
@@
       (effects (font (size 1.27 1.27)) (justify left))
     )
-    (property "Value" "74HC14" (at 184.7849 192.405 0)
+    (property "Value" "74HC14PW,118" (at 184.7849 192.405 0)
       (effects (font (size 1.27 1.27)) (justify left))
     )
@@
       (effects (font (size 1.27 1.27)))
     )
-    (property "Value" "74HC14" (at 224.155 217.805 0)
+    (property "Value" "74HC14PW,118" (at 226.06 217.805 0)
       (effects (font (size 1.27 1.27)))
     )
@@
       (effects (font (size 1.27 1.27)))
     )
-    (property "Value" "74HC14" (at 245.745 113.665 0)
+    (property "Value" "74HC14PW,118" (at 247.015 113.665 0)
       (effects (font (size 1.27 1.27)))
     )
@@
       (effects (font (size 1.27 1.27)) hide)
     )
+    (property "LCSC" "C5606" (at 239.395 116.205 0)
+      (effects (font (size 1.524 1.524)) hide)
+    )
     (pin "1")
     (pin "2")
@@
       (effects (font (size 1.27 1.27)) (justify left))
     )
-    (property "Value" "74HC14" (at 206.3749 88.265 0)
+    (property "Value" "74HC14PW,118" (at 206.3749 88.265 0)
       (effects (font (size 1.27 1.27)) (justify left))
     )
@@
       (effects (font (size 1.27 1.27)) hide)
     )
+    (property "LCSC" "C5606" (at 205.105 94.615 0)
+      (effects (font (size 1.524 1.524)) hide)
+    )
     (pin "1")
     (pin "2")
@@
       (effects (font (size 1.27 1.27)))
     )
-    (property "Value" "74HC14" (at 224.155 202.565 0)
+    (property "Value" "74HC14PW,118" (at 226.06 202.565 0)
       (effects (font (size 1.27 1.27)))
     )
@@
       (effects (font (size 1.27 1.27)) hide)
     )
-    (property "LCSC" "C5606" (at 217.805 205.105 0)
-      (effects (font (size 1.524 1.524)) hide)
-    )
     (pin "1")
     (pin "2")
@@
       (effects (font (size 1.27 1.27)))
     )
-    (property "Value" "74HC14" (at 245.745 128.905 0)
+    (property "Value" "74HC14PW,118" (at 247.015 128.905 0)
       (effects (font (size 1.27 1.27)))
     )
@@
       (effects (font (size 1.27 1.27)) hide)
     )
+    (property "LCSC" "C5606" (at 239.395 131.445 0)
+      (effects (font (size 1.524 1.524)) hide)
+    )
     (pin "1")
     (pin "2")
@@
       (effects (font (size 1.27 1.27)) hide)
     )
-    (property "LCSC" "C326973" (at 500.38 266.7 0)
+    (property "LCSC" "C525649" (at 500.38 266.7 0)
       (effects (font (size 1.27 1.27)) hide)
     )
@@
       (effects (font (size 1.016 1.016)))
     )
-    (property "Value" "Jumper-Pad-Pad" (at 424.18 77.978 0)
-      (effects (font (size 1.016 1.016)) hide)
+    (property "Value" "DNP" (at 424.18 76.2 0)
+      (effects (font (size 1.016 1.016)))
     )
     (property "Footprint" "hellen-one-common:PAD-0805-PAD" (at 424.18 80.01 0)
@@
       (effects (font (size 1.524 1.524)) hide)
     )
-    (property "LCSC" "C17477" (at 424.18 80.01 0)
+    (property "LCSC" "" (at 424.18 80.01 0)
       (effects (font (size 1.27 1.27)) hide)
     )
@@
       (effects (font (size 1.27 1.27)))
     )
-    (property "Value" "74HC14" (at 245.745 121.285 0)
+    (property "Value" "74HC14PW,118" (at 247.015 121.285 0)
       (effects (font (size 1.27 1.27)))
     )
@@
       (effects (font (size 1.27 1.27)) hide)
     )
+    (property "LCSC" "C5606" (at 239.395 123.825 0)
+      (effects (font (size 1.524 1.524)) hide)
+    )
     (pin "1")
     (pin "2")
@@
       (effects (font (size 1.27 1.27)))
     )
-    (property "Value" "74HC14" (at 245.745 98.425 0)
+    (property "Value" "74HC14PW,118" (at 247.015 98.425 0)
       (effects (font (size 1.27 1.27)))
     )
@@
     )
   )
-  (symbol (lib_id "hellen-one-common:Jumper-Pad-Pad") (at 424.18 73.66 0) (unit 1)
-    (in_bom yes) (on_board yes) (dnp no)
-    (property "Reference" "R121" (at 429.26 72.39 0)
-      (effects (font (size 1.016 1.016)))
-    )
-    (property "Value" "DNP" (at 424.18 73.66 0)
-      (effects (font (size 1.016 1.016)))
-    )
-    (property "Footprint" "hellen-one-common:PAD-0805-PAD" (at 424.18 77.47 0)
-      (effects (font (size 1.524 1.524)) hide)
-    )
-    (property "Datasheet" "" (at 424.18 73.66 0)
-      (effects (font (size 1.524 1.524)) hide)
-    )
-    (property "LCSC" "" (at 424.18 77.47 0)
-      (effects (font (size 1.27 1.27)) hide)
-    )
-    (pin "1")
-    (pin "2")
-    (instances
-      (project "GDI-4ch"
-        (path "/03caada9-9e22-4e2d-9035-b15433dfbb17"
-          (reference "R121") (unit 1)
-        )
-      )
-    )
-  )
   (symbol (lib_id "Device:R") (at 563.88 312.42 0) (unit 1)
     (in_bom yes) (on_board yes) (dnp no)
@@
       (effects (font (size 1.27 1.27)))
     )
-    (property "Value" "74HC14" (at 224.155 233.045 0)
+    (property "Value" "74HC14PW,118" (at 226.06 233.045 0)
       (effects (font (size 1.27 1.27)))
     )

Commit message: #200 note
Other:
- note added: "Use IN_A3 as board ID Remove R59 to disconnect this line from the main connector ID R32 ADC_PA4 0 DNP 0V 1 470k 1.48V 2 100k 2.45V"
Changed lines of the file:
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@@
+    (effects (font (size 1.524 1.524)) (justify left bottom))
+  )
+  (text "Use IN_A3 as board ID\n\nRemove R59 to disconnect\nthis line from the \nmain connector\n\nID   R32  ADC_PA4\n0    DNP      0V\n1    470k   1.48V \n2    100k   2.45V\n\n"
+    (at 87.63 347.98 0)
     (effects (font (size 1.524 1.524)) (justify left bottom))
   )

Commit message: #201, #202
Parts:
- D20: value BLUE -> RED; LCSC C72041 -> C2286
Other:
- note added: "CAN High"
- note added: "CAN Low"
- note added: "Injector Control 1"
- note added: "Injector Control 2"
- note added: "Injector Control 3"
- note added: "Injector Control 4"
- note added: "Injector Control 5"
- note added: "Injector Control 6"
- note added: "OK"
- note added: "blue"
- note added: "green"
- note added: "grey"
- note added: "orange/brown"
- note added: "white"
- note added: "yellow"
- note removed: "LED1"
- moved on the sheet: R9
Changed lines of the file:
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@@
     (stroke (width 0) (type default))
   )
-  (wire (pts (xy 72.39 180.34) (xy 54.61 180.34))
-    (stroke (width 0) (type default))
-  )
   (wire (pts (xy 147.955 154.305) (xy 150.495 154.305))
     (stroke (width 0) (type default))
@@
     (stroke (width 0) (type default))
   )
+  (wire (pts (xy 57.15 177.8) (xy 57.15 180.34))
+    (stroke (width 0) (type default))
+  )
   (wire (pts (xy 499.11 135.89) (xy 515.62 135.89))
     (stroke (width 0) (type default))
@@
     (stroke (width 0) (type default))
   )
+  (wire (pts (xy 340.36 104.14) (xy 345.44 104.14))
+    (stroke (width 0) (type default))
+  )
   (wire (pts (xy 250.825 306.705) (xy 253.365 306.705))
     (stroke (width 0) (type default))
@@
     (stroke (width 0) (type default))
   )
+  (wire (pts (xy 57.15 180.34) (xy 54.61 180.34))
+    (stroke (width 0) (type default))
+  )
   (wire (pts (xy 54.61 142.24) (xy 69.85 142.24))
     (stroke (width 0) (type default))
@@
     (effects (font (size 1.524 1.524)) (justify right bottom))
   )
+  (text "white" (at 33.02 173.355 0)
+    (effects (font (size 1.27 1.27)) (justify right bottom))
+  )
   (text "Use R122 option without R113, R121 for SENT" (at 469.9 80.645 0)
     (effects (font (size 1.524 1.524)) (justify right bottom))
   )
+  (text "yellow" (at 33.02 170.815 0)
+    (effects (font (size 1.27 1.27)) (justify right bottom))
+  )
   (text "rev. a: STTH802G-TR" (at 518.16 275.59 0)
     (effects (font (size 1.27 1.27)) (justify left bottom))
   )
-  (text "LED2" (at 351.61 104.0524 0)
+  (text "LED2" (at 342.265 104.14 0)
     (effects (font (size 1.524 1.524)) (justify left bottom))
   )
+  (text "Injector Control 3" (at 68.58 167.005 0)
+    (effects (font (size 1.27 1.27)) (justify left bottom))
+  )
   (text "     4ch+1  6ch\nR87    +    DNP\nR37    +    DNP\nR41   DNP    +\nR88   DNP    +\nR89    +    DNP"
     (at 88.9 161.925 0)
     (effects (font (size 1.524 1.524)) (justify left bottom))
   )
+  (text "orange/brown" (at 33.02 175.895 0)
+    (effects (font (size 1.27 1.27)) (justify right bottom))
+  )
+  (text "Injector Control 5" (at 68.58 164.465 0)
+    (effects (font (size 1.27 1.27)) (justify left bottom))
+  )
   (text "22V MAX\n" (at 25.4 25.4 0)
     (effects (font (size 1.524 1.524)) (justify left bottom))
   )
+  (text "Injector Control 4" (at 68.58 174.625 0)
+    (effects (font (size 1.27 1.27)) (justify left bottom))
+  )
   (text "PUMP BANK / INJECTOR LOW 5, 6" (at 287.02 322.58 0)
     (effects (font (size 1.524 1.524)) (justify left bottom))
   )
+  (text "grey" (at 33.02 165.735 0)
+    (effects (font (size 1.27 1.27)) (justify right bottom))
+  )
+  (text "CAN Low" (at 68.58 184.785 0)
+    (effects (font (size 1.27 1.27)) (justify left bottom))
+  )
   (text "OUT\n" (at 52.0045 74.7659 0)
     (effects (font (size 1.524 1.524)) (justify left bottom))
@@
     (effects (font (size 1.27 1.27)) (justify left bottom))
   )
-  (text "LED1" (at 422.91 97.79 0)
+  (text "OK" (at 424.18 97.155 0)
     (effects (font (size 1.524 1.524)) (justify left bottom))
   )
+  (text "blue" (at 33.02 168.275 0)
+    (effects (font (size 1.27 1.27)) (justify right bottom))
+  )
+  (text "green" (at 33.02 183.515 0)
+    (effects (font (size 1.27 1.27)) (justify right bottom))
+  )
   (text "Discharge\ncircuit" (at 575.31 293.37 0)
     (effects (font (size 1.27 1.27)) (justify right bottom))
@@
     (effects (font (size 1.524 1.524)) (justify left bottom))
   )
+  (text "Injector Control 2" (at 68.58 172.085 0)
+    (effects (font (size 1.27 1.27)) (justify left bottom))
+  )
   (text "UART / +5 / GND for integration" (at 534.67 66.675 0)
     (effects (font (size 1.27 1.27)) (justify left bottom))
   )
+  (text "Injector Control 1" (at 68.58 161.925 0)
+    (effects (font (size 1.27 1.27)) (justify left bottom))
+  )
+  (text "Injector Control 6" (at 68.58 169.545 0)
+    (effects (font (size 1.27 1.27)) (justify left bottom))
+  )
+  (text "green" (at 33.02 163.195 0)
+    (effects (font (size 1.27 1.27)) (justify right bottom))
+  )
+  (text "blue" (at 33.02 186.055 0)
+    (effects (font (size 1.27 1.27)) (justify right bottom))
+  )
+  (text "CAN High" (at 68.58 182.245 0)
+    (effects (font (size 1.27 1.27)) (justify left bottom))
+  )
   (label "OUT_INJ2_N" (at 58.42 43.18 180) (fields_autoplaced)
     (effects (font (size 1.524 1.524)) (justify right bottom))
@@
       (effects (font (size 1.27 1.27)) (justify right))
     )
-    (property "Value" "BLUE" (at 351.79 101.6 0)
+    (property "Value" "RED" (at 354.965 102.87 0)
       (effects (font (size 1.27 1.27)) (justify right))
     )
@@
       (effects (font (size 1.27 1.27)) hide)
     )
-    (property "LCSC" "C72041" (at 349.25 104.14 0)
+    (property "LCSC" "C2286" (at 349.25 104.14 0)
       (effects (font (size 1.27 1.27)) hide)
     )
@@
     )
   )
-  (symbol (lib_id "power:+BATT") (at 72.39 180.34 270) (unit 1)
+  (symbol (lib_id "power:+BATT") (at 57.15 177.8 270) (unit 1)
     (in_bom yes) (on_board yes) (dnp no)
-    (property "Reference" "#PWR04" (at 68.58 180.34 0)
+    (property "Reference" "#PWR04" (at 53.34 177.8 0)
       (effects (font (size 1.27 1.27)) hide)
     )
-    (property "Value" "+BATT" (at 78.74 180.34 90)
+    (property "Value" "+BATT" (at 63.5 177.8 90)
       (effects (font (size 1.27 1.27)))
     )
-    (property "Footprint" "" (at 72.39 180.34 0)
+    (property "Footprint" "" (at 57.15 177.8 0)
       (effects (font (size 1.27 1.27)) hide)
     )
-    (property "Datasheet" "" (at 72.39 180.34 0)
+    (property "Datasheet" "" (at 57.15 177.8 0)
       (effects (font (size 1.27 1.27)) hide)
     )
@@
     )
   )
-  (symbol (lib_id "power:GND") (at 337.82 104.14 270) (unit 1)
+  (symbol (lib_id "power:GND") (at 332.74 104.14 270) (unit 1)
     (in_bom yes) (on_board yes) (dnp no)
-    (property "Reference" "#PWR062" (at 331.47 104.14 0)
+    (property "Reference" "#PWR062" (at 326.39 104.14 0)
       (effects (font (size 1.27 1.27)) hide)
     )
-    (property "Value" "GND" (at 333.4258 104.267 0)
+    (property "Value" "GND" (at 327.66 104.14 90)
       (effects (font (size 1.27 1.27)))
     )
-    (property "Footprint" "" (at 337.82 104.14 0)
+    (property "Footprint" "" (at 332.74 104.14 0)
       (effects (font (size 1.27 1.27)) hide)
     )
-    (property "Datasheet" "" (at 337.82 104.14 0)
+    (property "Datasheet" "" (at 332.74 104.14 0)
       (effects (font (size 1.27 1.27)) hide)
     )
@@
     )
   )
-  (symbol (lib_id "Device:R") (at 341.63 104.14 270) (unit 1)
+  (symbol (lib_id "Device:R") (at 336.55 104.14 270) (unit 1)
     (in_bom yes) (on_board yes) (dnp no)
-    (property "Reference" "R9" (at 345.44 102.87 90)
+    (property "Reference" "R9" (at 340.36 102.87 90)
       (effects (font (size 1.016 1.016)))
     )
-    (property "Value" "1K" (at 341.6554 104.3178 90)
+    (property "Value" "1K" (at 336.5754 104.3178 90)
       (effects (font (size 1.016 1.016)))
     )
-    (property "Footprint" "Resistor_SMD:R_0603_1608Metric" (at 321.31 149.987 90)
+    (property "Footprint" "Resistor_SMD:R_0603_1608Metric" (at 316.23 149.987 90)
       (effects (font (size 1.524 1.524)) hide)
     )
-    (property "Datasheet" "" (at 321.945 239.395 0)
+    (property "Datasheet" "" (at 316.865 239.395 0)
       (effects (font (size 1.524 1.524)) hide)
     )
-    (property "LCSC" "C21190" (at 341.63 104.14 0)
+    (property "LCSC" "C21190" (at 336.55 104.14 0)
       (effects (font (size 1.27 1.27)) hide)
     )
