File: lambda-x2/lambda-x2.kicad_sch (KiCad schematic)
At the start: 75 parts, among them J1 FTSH-107-01-F-DV-K, P1 33311-24AW-2, Q2 BTS3028, U2 STM32F103C6Tx, U4 LM78M05_TO252, U5 XC6206P332MR, U6 REF3033, U7 MCP6002T-I/SN, U8 TJA1051T-3

Commit message: lambda-x2: some upadte
Parts:
- J3: value (none) -> Conn_02x02_Odd_Even; footprint (none) -> Connector_PinHeader_2.54mm:PinHeader_2x02_P2.54mm_Vertical
- J4: value (none) -> Conn_01x10; footprint (none) -> Connector_PinHeader_2.54mm:PinHeader_1x10_P2.54mm_Vertical
- TP1, TP2: value (none) -> TestPoint; footprint (none) -> Connector_PinHeader_2.54mm:PinHeader_1x01_P2.54mm_Vertical
- TP3, TP4, TP5: value (none) -> TestPoint; footprint (none) -> TestPoint:TestPoint_Pad_D1.0mm
Changed lines of the file:
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@@
     (in_bom no) (on_board yes)
     (property "Reference" "J3" (id 0) (at 553.085 57.3532 0))
-    (property "Value" "" (id 1) (at 553.085 59.6646 0))
-    (property "Footprint" "" (id 2) (at 551.815 62.865 0)
+    (property "Value" "Conn_02x02_Odd_Even" (id 1) (at 553.085 59.6646 0))
+    (property "Footprint" "Connector_PinHeader_2.54mm:PinHeader_2x02_P2.54mm_Vertical" (id 2) (at 551.815 62.865 0)
       (effects (font (size 1.27 1.27)) hide)
     )
@@
     (in_bom no) (on_board yes)
     (property "Reference" "TP1" (id 0) (at 383.6162 278.257 90))
-    (property "Value" "" (id 1) (at 383.6162 280.5684 90))
-    (property "Footprint" "" (id 2) (at 385.445 278.13 0)
+    (property "Value" "TestPoint" (id 1) (at 383.6162 280.5684 90))
+    (property "Footprint" "Connector_PinHeader_2.54mm:PinHeader_1x01_P2.54mm_Vertical" (id 2) (at 385.445 278.13 0)
       (effects (font (size 1.27 1.27)) hide)
     )
@@
       (effects (font (size 1.27 1.27)) (justify right))
     )
-    (property "Value" "" (id 1) (at 375.4882 294.4368 0)
-      (effects (font (size 1.27 1.27)) (justify right))
-    )
-    (property "Footprint" "" (id 2) (at 368.935 291.465 0)
+    (property "Value" "TestPoint" (id 1) (at 375.4882 294.4368 0)
+      (effects (font (size 1.27 1.27)) (justify right))
+    )
+    (property "Footprint" "Connector_PinHeader_2.54mm:PinHeader_1x01_P2.54mm_Vertical" (id 2) (at 368.935 291.465 0)
       (effects (font (size 1.27 1.27)) hide)
     )
@@
       (effects (font (size 1.27 1.27)) (justify left))
     )
-    (property "Value" "" (id 1) (at 480.822 306.0446 0)
-      (effects (font (size 1.27 1.27)) (justify left))
-    )
-    (property "Footprint" "" (id 2) (at 478.79 303.53 0)
+    (property "Value" "Conn_01x10" (id 1) (at 480.822 306.0446 0)
+      (effects (font (size 1.27 1.27)) (justify left))
+    )
+    (property "Footprint" "Connector_PinHeader_2.54mm:PinHeader_1x10_P2.54mm_Vertical" (id 2) (at 478.79 303.53 0)
       (effects (font (size 1.27 1.27)) hide)
     )
@@
       (effects (font (size 1.27 1.27)) (justify left))
     )
-    (property "Value" "" (id 1) (at 445.77 322.5799 90)
+    (property "Value" "TestPoint" (id 1) (at 445.77 322.5799 90)
       (effects (font (size 1.27 1.27)) (justify left) hide)
     )
-    (property "Footprint" "" (id 2) (at 440.69 326.39 0)
+    (property "Footprint" "TestPoint:TestPoint_Pad_D1.0mm" (id 2) (at 440.69 326.39 0)
       (effects (font (size 1.27 1.27)) hide)
     )
@@
       (effects (font (size 1.27 1.27)) (justify left))
     )
-    (property "Value" "" (id 1) (at 445.77 317.4999 90)
+    (property "Value" "TestPoint" (id 1) (at 445.77 317.4999 90)
       (effects (font (size 1.27 1.27)) (justify left) hide)
     )
-    (property "Footprint" "" (id 2) (at 440.69 321.31 0)
+    (property "Footprint" "TestPoint:TestPoint_Pad_D1.0mm" (id 2) (at 440.69 321.31 0)
       (effects (font (size 1.27 1.27)) hide)
     )
@@
       (effects (font (size 1.27 1.27)) (justify left))
     )
-    (property "Value" "" (id 1) (at 445.77 320.0399 90)
+    (property "Value" "TestPoint" (id 1) (at 445.77 320.0399 90)
       (effects (font (size 1.27 1.27)) (justify left) hide)
     )
-    (property "Footprint" "" (id 2) (at 440.69 323.85 0)
+    (property "Footprint" "TestPoint:TestPoint_Pad_D1.0mm" (id 2) (at 440.69 323.85 0)
       (effects (font (size 1.27 1.27)) hide)
     )
@@
       (reference "U9") (unit 3) (value "GS8332") (footprint "Package_SO:TSSOP-8_3x3mm_P0.65mm")
     )
-    (path "/8c53ed69-a65a-4bef-9bec-7173d9bbff28/bff1e8d7-556b-43e8-a4e1-923281a6eea9"
+    (path "/8c53ed69-a65a-4bef-9bec-7173d9bbff28/32efed2e-5629-49a3-a1b9-8e0addb8e454"
       (reference "U10") (unit 1) (value "MCP6004") (footprint "Package_SO:TSSOP-14_4.4x5mm_P0.65mm")
     )
@@
       (reference "U10") (unit 2) (value "MCP6004") (footprint "Package_SO:TSSOP-14_4.4x5mm_P0.65mm")
     )
-    (path "/8c53ed69-a65a-4bef-9bec-7173d9bbff28/32efed2e-5629-49a3-a1b9-8e0addb8e454"
+    (path "/8c53ed69-a65a-4bef-9bec-7173d9bbff28/7350c1a2-80c4-4998-9179-ac12ed459522"
       (reference "U10") (unit 3) (value "MCP6004") (footprint "Package_SO:TSSOP-14_4.4x5mm_P0.65mm")
     )
-    (path "/8c53ed69-a65a-4bef-9bec-7173d9bbff28/7350c1a2-80c4-4998-9179-ac12ed459522"
+    (path "/8c53ed69-a65a-4bef-9bec-7173d9bbff28/bff1e8d7-556b-43e8-a4e1-923281a6eea9"
       (reference "U10") (unit 4) (value "MCP6004") (footprint "Package_SO:TSSOP-14_4.4x5mm_P0.65mm")
     )

Commit message: more progress
Parts:
- removed TP3, TP4, TP5: TestPoint, TestPoint:TestPoint_Pad_D1.0mm, symbol Connector:TestPoint
- added C35: 100n, Capacitor_SMD:C_0402_1005Metric, symbol Device:C
- added D3: RED, LED_SMD:LED_0603_1608Metric, symbol Device:LED
- added Q1: BTS3028, Package_TO_SOT_SMD:TO-252-2, symbol Device:Q_NMOS_GDS
- added R79, R83: 1k, Resistor_SMD:R_0402_1005Metric, symbol Device:R
- added R80: 10k, Resistor_SMD:R_0402_1005Metric, symbol Device:R
- added R81: 100k 1%, Resistor_SMD:R_0402_1005Metric, symbol Device:R
- added R82: 10k 1%, Resistor_SMD:R_0402_1005Metric, symbol Device:R
Connections:
- net GND: now also C35.2, D3.1 (K), Q1.3 (S), R80.1, R82.1
- net L_Ip_sense: now also U2.15 (PA5); no longer U2.16 (PA6)
- net L_LSU_Heater-: now also P1.5 (A5); no longer P1.17 (C1)
- net L_LSU_Ip: now also P1.4 (A4); no longer P1.18 (C2)
- net L_LSU_Un: now also P1.3 (A3); no longer P1.19 (C3)
- net L_LSU_Vm: now also P1.12 (B4); no longer P1.10 (B2)
- net L_Un_3x_sense: now also U2.16 (PA6); no longer U2.17 (PA7)
- net L_Un_sense: now also U2.17 (PA7); no longer U2.15 (PA5)
- net R_Ip_sense: now also U2.12 (PA2)
- net R_LSU_Heater-: now also Q1.2 (D), R81.1
- net R_Un_3x_sense: now also U2.13 (PA3)
- net R_Un_sense: now also U2.14 (PA4)
- new net: D3.2 (A), R83.1
- new net: Q1.1 (G), R79.1
- new net R_Heater_sense: C35.1, R81.2, R82.2
- new net R_heater_pwm: R79.2, R80.2, R83.2
Other:
- note added: "ADC"

Commit message: progress
Connections:
- net 12V_RAW: now also P1.24 (C8); no longer P1.2 (A2)
- net CAN_H: no longer P1.21 (C5)
- net CAN_L: no longer P1.22 (C6)
- net GND: now also P1.17 (C1); no longer P1.1 (A1)
- net L_EGT-: now reaches P1.19 (C3)
- net L_EGT+: now reaches P1.20 (C4)
- net R_EGT+: now reaches P1.23 (C7)
- net DISP0: no longer names the net of J4.3 (Pin_3)
- net DISP0: no longer U2.38 (PA15)
- net DISP1: no longer names the net of J4.5 (Pin_5)
- net DISP1: no longer U2.40 (PB4)
- net DISP2: no longer names the net of J4.6 (Pin_6)
- net DISP2: no longer U2.41 (PB5)
- removed net SWO: J1.8 (Pin_8), J4.4 (Pin_4), U2.39 (PB3)
- new net R_EGT-: P1.22 (C6)
- new net SPI1_MISO: U2.40 (PB4)
- new net SPI1_MOSI: U2.41 (PB5)
- new net SPI1_NSS: U2.38 (PA15)
- new net SPI1_SCK: U2.39 (PB3)
- no-connect marks 4 -> 5
Other:
- added sheet EGT left (egt.kicad_sch)
- added sheet EGT right (egt.kicad_sch)
- note removed: "SPI1_MISO"
- note removed: "SPI1_MOSI"
- note removed: "SPI1_NSS"
- note removed: "SPI1_SCK"
- moved on the sheet: C7, R2, R6

Commit message: more progress
Parts:
- added C54: 1u, Capacitor_SMD:C_0402_1005Metric, symbol Device:C
- added C55, C56, C57: 100n, Capacitor_SMD:C_0402_1005Metric, symbol Device:C
- added D10, D11: RED, LED_SMD:LED_0603_1608Metric, symbol Device:LED
- added D12: NUP2105L, Package_TO_SOT_SMD:SOT-23, symbol Power_Protection:NUP2105L
- added Q3, Q4: BTS3028, Package_TO_SOT_SMD:TO-252-2, symbol Device:Q_NMOS_GDS
- added R100, R101: 160k, Resistor_SMD:R_0603_1608Metric, symbol Device:R
- added R86, R87, R90, R91: 1k, Resistor_SMD:R_0402_1005Metric, symbol Device:R
- added R88, R89: 10k, Resistor_SMD:R_0402_1005Metric, symbol Device:R
- added R96, R97: 10k 0.1%, Resistor_SMD:R_0603_1608Metric, symbol Device:R
- added R98, R99: 82k, Resistor_SMD:R_0603_1608Metric, symbol Device:R
- added U17: (no value), symbol Amplifier_Operational:MCP6002-xSN
- R34: value 3.3k -> (none); footprint Resistor_SMD:R_0402_1005Metric -> (none)
- R43: value 100k 1% -> 3.3k; LCSC C25741 -> C25890
- R44: value 10k 1% -> 3.3k; LCSC C25744 -> C25890
Connections:
- net R_Un_sense is gone; now on net R_Un_3x_sense: U2.14 (PA4)
- net SPI1_NSS is gone; now on net SPI1_CS2: U2.38 (PA15)
- net l_Heater_sense is gone; now on net L_Heater_sense: C10.1, R52.2, R53.2
- net +3V3: now also R43.1, R44.1, C57.1
- net +5V: now also C2.1, C54.1, C55.1, C56.1, U17.8 (V+); no longer R27.2
- net 12V_PROT: no longer R43.1
- net CAN_H: now also P1.20 (C4), D12.1 (K)
- net CAN_L: now also P1.21 (C5), D12.2 (K)
- net GND: now also R27.2, C54.2, C55.2, C56.2, C57.2, D10.1 (K), D11.1 (K), D12.3 (A), Q3.3 (S), Q4.3 (S), R100.1, R101.1, R88.1, R89.1, U17.4 (V-); no longer R44.1
- net L_EGT+: now also P1.19 (C3); no longer P1.20 (C4)
- net L_EGT-: now also P1.18 (C2); no longer P1.19 (C3)
- net L_Heater_sense: now also U2.18 (PB0); no longer U2.19 (PB1)
- net L_Ip_dac: now also U2.12 (PA2); no longer U2.11 (PA1)
- net L_LSU_Heater-: now also P1.1 (A1); no longer P1.5 (A5)
- net L_LSU_Ip: now also P1.3 (A3); no longer P1.4 (A4)
- net L_LSU_Rtrim: now also P1.10 (B2); no longer P1.11 (B3)
- net L_LSU_Un: now also P1.2 (A2); no longer P1.3 (A3)
- net L_LSU_Vm: now also P1.11 (B3); no longer P1.12 (B4)
- net L_Vm_sense: no longer U2.10 (PA0)
- net R_Heater_sense: now also U2.19 (PB1)
- net R_Ip_dac: now also U2.11 (PA1)
- net R_Ip_sense: now also U2.13 (PA3); no longer U2.12 (PA2)
- net R_Un_3x_sense: no longer U2.13 (PA3)
- net R_heater_pwm: now also U2.43 (PB7)
- net SPI1_MISO: now also J4.5 (Pin_5)
- net SPI1_MOSI: now also J4.6 (Pin_6)
- net SPI1_SCK: now also J4.4 (Pin_4)
- net Vout1: now also P1.13 (B5)
- net Vout2: now also P1.12 (B4)
- net SPI1_CS0: now reaches U2.5 (PD0)
- net SPI1_CS1: now reaches U2.6 (PD1)
- net R_OD: now reaches P1.16 (B8)
- net R_OD: now also Q4.2 (D)
- net L_OD: now reaches P1.9 (B1)
- net L_OD: now also Q3.2 (D)
- net DISP4 renamed SPI1_CS2
- net SPI1_CS2: no longer U2.43 (PB7)
- net DISP5 renamed I2C1_SCL
- net I2C1_SCL: now also R43.2
- net DISP6 renamed I2C1_SDA
- net I2C1_SDA: now also R44.2
- net L_Un_sense renamed L_AUX_ADC
- net L_AUX_ADC: now also R100.2, R98.1
- removed net Vbatt_sense: C2.1, R43.2, R44.2, U2.18 (PB0)
- new net: R99.2, U17.1, U17.2 (-)
- new net: R96.1, U17.5 (+)
- new net: R98.2, U17.6 (-), U17.7
- new net: Q3.1 (G), R86.1
- new net: Q4.1 (G), R87.1
- new net: R97.1, U17.3 (+)
- new net: D11.2 (A), R91.1
- new net: D10.2 (A), R90.1
- new net L_AUX: P1.4 (A4), R96.2
- new net L_OUT_en: R86.2, R88.2, R90.2
- new net R_AUX: P1.5 (A5), R97.2
- new net R_AUX_ADC: R101.2, R99.1, U2.10 (PA0)
- new net R_OUT_en: R87.2, R89.2, R91.2
- no-connect marks 5 -> 7
Other:
- sheet EGT left ports: added SPI_SI; removed none
- sheet EGT right ports: added SPI_SI; removed none
- note added: "No cap required needed according to DS"
- note added: "Optional OD outputs"
- note added: "TIM4_CH1"
- note added: "TIM4_CH2"
- note added: "booloader"
- note removed: "I2C1_SCL"
- note removed: "I2C1_SDA"
- note removed: "grey"
- moved on the sheet: C10, C27, C28, C32, C33, C34, C35, C36, C42, C7, D3, D5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
