File: lambda-x2/lambda-x2.kicad_sch (KiCad schematic)
At the start: 151 parts, among them J1 FTSH-107-01-F-DV-K, J3 Conn_02x02_Odd_Even, J4 Conn_01x10, P1 33311-24AW-2, Q1 BTS3028, Q2 BTS3028, Q3 BTS3028, Q4 BTS3028, U17 MCP6002T-I/SN, U18 JDY-33, U2 STM32F103C6Tx, U4 LM78M05_TO252, U5 XC6206P332MR, U6 REF3033, U7 MCP6002T-I/SN, U8 TJA1051T-3, Y1 XXDCELNANF-8MHZ

Commit message: lambda-x2: update
Parts:
- removed H2, H3: MountingHole_Pad, MountingHole:MountingHole_2.5mm_Pad_Via, symbol Mechanical:MountingHole_Pad
- J2: value (none) -> tc2030-idc-nl; footprint (none) -> rusefi:tc2030-idc-nl
Other:
- moved on the sheet: H1
Changed lines of the file:
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@@
   (junction (at 228.6 353.06) (diameter 0) (color 0 0 0 0)
   )
-  (junction (at 548.64 361.95) (diameter 0) (color 0 0 0 0)
-  )
   (junction (at 228.6 180.34) (diameter 0) (color 0 0 0 0)
   )
@@
     (stroke (width 0) (type default) (color 0 0 0 0))
   )
-  (wire (pts (xy 516.89 361.95) (xy 516.89 364.49))
-    (stroke (width 0) (type default) (color 0 0 0 0))
-  )
   (wire (pts (xy 234.95 381) (xy 209.55 381))
     (stroke (width 0) (type default) (color 0 0 0 0))
@@
     (stroke (width 0) (type default) (color 0 0 0 0))
   )
+  (wire (pts (xy 516.89 361.95) (xy 516.89 364.49))
+    (stroke (width 0) (type default) (color 0 0 0 0))
+  )
   (wire (pts (xy 154.94 278.13) (xy 158.75 278.13))
     (stroke (width 0) (type default) (color 0 0 0 0))
@@
     (stroke (width 0) (type default) (color 0 0 0 0))
   )
-  (wire (pts (xy 516.89 359.41) (xy 516.89 361.95))
-    (stroke (width 0) (type default) (color 0 0 0 0))
-  )
   (wire (pts (xy 142.24 323.85) (xy 135.89 323.85))
     (stroke (width 0) (type default) (color 0 0 0 0))
@@
     (stroke (width 0) (type default) (color 0 0 0 0))
   )
-  (wire (pts (xy 548.64 359.41) (xy 548.64 361.95))
-    (stroke (width 0) (type default) (color 0 0 0 0))
-  )
   (wire (pts (xy 443.23 195.58) (xy 443.23 198.12))
     (stroke (width 0) (type default) (color 0 0 0 0))
@@
     (pin "1")
   )
-  (symbol (lib_id "Mechanical:MountingHole_Pad") (at 516.89 367.03 180) (unit 1)
-    (in_bom no) (on_board yes) (fields_autoplaced)
-    (property "Reference" "H2" (id 0) (at 519.43 367.0299 0)
-      (effects (font (size 1.27 1.27)) (justify right))
-    )
-    (property "Value" "MountingHole_Pad" (id 1) (at 519.43 369.5699 0)
-      (effects (font (size 1.27 1.27)) (justify right))
-    )
-    (property "Footprint" "MountingHole:MountingHole_2.5mm_Pad_Via" (id 2) (at 516.89 367.03 0)
-      (effects (font (size 1.27 1.27)) hide)
-    )
-    (property "Datasheet" "~" (id 3) (at 516.89 367.03 0)
-      (effects (font (size 1.27 1.27)) hide)
-    )
-    (pin "1")
-  )
   (symbol (lib_name "GND_63") (lib_id "power:GND") (at 339.09 134.62 270) (unit 1)
     (in_bom yes) (on_board yes)
@@
     (pin "9")
   )
-  (symbol (lib_id "Mechanical:MountingHole_Pad") (at 516.89 356.87 0) (unit 1)
+  (symbol (lib_id "Mechanical:MountingHole_Pad") (at 516.89 367.03 180) (unit 1)
     (in_bom no) (on_board yes) (fields_autoplaced)
-    (property "Reference" "H1" (id 0) (at 519.43 354.3299 0)
-      (effects (font (size 1.27 1.27)) (justify left))
+    (property "Reference" "H1" (id 0) (at 519.43 367.0299 0)
+      (effects (font (size 1.27 1.27)) (justify right))
     )
-    (property "Value" "MountingHole_Pad" (id 1) (at 519.43 356.8699 0)
-      (effects (font (size 1.27 1.27)) (justify left))
+    (property "Value" "MountingHole_Pad" (id 1) (at 519.43 369.5699 0)
+      (effects (font (size 1.27 1.27)) (justify right))
     )
-    (property "Footprint" "MountingHole:MountingHole_2.5mm_Pad_Via" (id 2) (at 516.89 356.87 0)
+    (property "Footprint" "MountingHole:MountingHole_2.5mm_Pad_Via" (id 2) (at 516.89 367.03 0)
       (effects (font (size 1.27 1.27)) hide)
     )
-    (property "Datasheet" "~" (id 3) (at 516.89 356.87 0)
+    (property "Datasheet" "~" (id 3) (at 516.89 367.03 0)
       (effects (font (size 1.27 1.27)) hide)
     )
@@
     (pin "1")
   )
-  (symbol (lib_id "Mechanical:MountingHole_Pad") (at 548.64 356.87 0) (unit 1)
-    (in_bom no) (on_board yes) (fields_autoplaced)
-    (property "Reference" "H3" (id 0) (at 551.18 354.3299 0)
-      (effects (font (size 1.27 1.27)) (justify left))
-    )
-    (property "Value" "MountingHole_Pad" (id 1) (at 551.18 356.8699 0)
-      (effects (font (size 1.27 1.27)) (justify left))
-    )
-    (property "Footprint" "MountingHole:MountingHole_2.5mm_Pad_Via" (id 2) (at 548.64 356.87 0)
-      (effects (font (size 1.27 1.27)) hide)
-    )
-    (property "Datasheet" "~" (id 3) (at 548.64 356.87 0)
-      (effects (font (size 1.27 1.27)) hide)
-    )
-    (pin "1")
-  )
   (symbol (lib_id "Device:R") (at 203.2 246.38 90) (mirror x) (unit 1)
     (in_bom yes) (on_board yes)
@@
     (in_bom yes) (on_board yes) (fields_autoplaced)
     (property "Reference" "J2" (id 0) (at 542.29 149.86 0))
-    (property "Value" "" (id 1) (at 542.29 152.4 0))
-    (property "Footprint" "" (id 2) (at 538.48 168.91 0)
+    (property "Value" "tc2030-idc-nl" (id 1) (at 542.29 152.4 0))
+    (property "Footprint" "rusefi:tc2030-idc-nl" (id 2) (at 538.48 168.91 0)
       (effects (font (size 1.27 1.27)) hide)
     )
@@
       (reference "H1") (unit 1) (value "MountingHole_Pad") (footprint "MountingHole:MountingHole_2.5mm_Pad_Via")
     )
-    (path "/01d4ddc4-aab7-48e4-bb44-8d9a410eff5c"
-      (reference "H2") (unit 1) (value "MountingHole_Pad") (footprint "MountingHole:MountingHole_2.5mm_Pad_Via")
-    )
-    (path "/acb5489d-7f48-415d-95ac-a67b3110aa0e"
-      (reference "H3") (unit 1) (value "MountingHole_Pad") (footprint "MountingHole:MountingHole_2.5mm_Pad_Via")
-    )
     (path "/16d62a37-8b6b-4e51-bc7b-4763aa0a3148"
