File: lambda-x2/lsu.kicad_sch (KiCad schematic)
At the start: 39 parts

Commit message: Progress
Parts:
- added unit 3 of U3
- gave numbers to parts that had none: 34
Connections:
- net Vgnd is gone; now on an unnamed net: R45.2
- net at R20.2: now also U3.8, U3.9 (-)
- net Vm renamed Vgnd_ref
- net Vgnd_ref: now also U3.10 (+)
Other:
- note added: "Internal Virtual Ground Buffer"

Commit message: Update components
Parts:
- R17, R5: LCSC C25776 -> C22984
- R19, R20: LCSC C328415 -> C122538
Changed lines of the file:
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@@
       (effects (font (size 1.27 1.27)) hide)
     )
-    (property "LCSC" "C25776" (id 4) (at 138.43 160.655 0)
+    (property "LCSC" "C22984" (id 4) (at 138.43 160.655 0)
       (effects (font (size 1.27 1.27)) hide)
     )
@@
       (effects (font (size 1.27 1.27)) hide)
     )
-    (property "LCSC" "C25776" (id 4) (at 121.92 148.59 0)
+    (property "LCSC" "C22984" (id 4) (at 121.92 148.59 0)
       (effects (font (size 1.27 1.27)) hide)
     )
@@
       (effects (font (size 1.27 1.27)) hide)
     )
-    (property "LCSC" "C328415" (id 4) (at 139.7 215.9 0)
+    (property "LCSC" "C122538" (id 4) (at 139.7 215.9 0)
       (effects (font (size 1.27 1.27)) hide)
     )
@@
       (effects (font (size 1.27 1.27)) hide)
     )
-    (property "LCSC" "C328415" (id 4) (at 139.7 243.84 0)
-      (effects (font (size 1.27 1.27)) hide)
-    )
+    (property "LCSC" "C122538" (id 4) (at 139.7 243.84 0)
+      (effects (font (size 1.27 1.27)) hide)
+    )

Commit message: lambda-x2: some upadte
Parts:
- U3: value MCP6004 -> (none); footprint Package_SO:TSSOP-14_4.4x5mm_P0.65mm -> (none)
Connections:
- no-connect marks 0 -> 1
Changed lines of the file:
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@@
   (junction (at 176.53 116.84) (diameter 0) (color 0 0 0 0)
   )
+  (no_connect (at -57.15 238.76))
   (wire (pts (xy 88.9 114.3) (xy 93.98 114.3))
     (stroke (width 0) (type default) (color 0 0 0 0))
@@
     (in_bom yes) (on_board yes)
     (property "Reference" "U3" (id 0) (at 222.25 60.96 0))
-    (property "Value" "MCP6004" (id 1) (at 222.885 63.5 0))
-    (property "Footprint" "Package_SO:TSSOP-14_4.4x5mm_P0.65mm" (id 2) (at 217.17 64.77 0)
+    (property "Value" "" (id 1) (at 222.885 63.5 0))
+    (property "Footprint" "" (id 2) (at 217.17 64.77 0)
       (effects (font (size 1.27 1.27)) hide)
     )
@@
     (in_bom yes) (on_board yes)
     (property "Reference" "U3" (id 0) (at 127 64.77 0))
-    (property "Value" "MCP6004" (id 1) (at 126.365 67.31 0))
-    (property "Footprint" "Package_SO:TSSOP-14_4.4x5mm_P0.65mm" (id 2) (at 132.08 68.58 0)
+    (property "Value" "" (id 1) (at 126.365 67.31 0))
+    (property "Footprint" "" (id 2) (at 132.08 68.58 0)
       (effects (font (size 1.27 1.27)) hide)
     )
@@
     (in_bom yes) (on_board yes)
     (property "Reference" "U3" (id 0) (at 222.25 158.75 0))
-    (property "Value" "MCP6004" (id 1) (at 229.235 154.94 0)
-      (effects (font (size 1.27 1.27)) hide)
-    )
-    (property "Footprint" "Package_SO:TSSOP-14_4.4x5mm_P0.65mm" (id 2) (at 223.52 156.21 0)
+    (property "Value" "" (id 1) (at 229.235 154.94 0)
+      (effects (font (size 1.27 1.27)) hide)
+    )
+    (property "Footprint" "" (id 2) (at 223.52 156.21 0)
       (effects (font (size 1.27 1.27)) hide)
     )
@@
     (in_bom yes) (on_board yes)
     (property "Reference" "U3" (id 0) (at 139.7 194.31 0))
-    (property "Value" "MCP6004" (id 1) (at 136.525 184.785 0))
-    (property "Footprint" "Package_SO:TSSOP-14_4.4x5mm_P0.65mm" (id 2) (at 140.97 191.77 0)
+    (property "Value" "" (id 1) (at 136.525 184.785 0))
+    (property "Footprint" "" (id 2) (at 140.97 191.77 0)
       (effects (font (size 1.27 1.27)) hide)
     )
@@
     (in_bom yes) (on_board yes)
     (property "Reference" "U3" (id 0) (at 142.24 111.76 0))
-    (property "Value" "MCP6004" (id 1) (at 143.51 114.3 0))
-    (property "Footprint" "Package_SO:TSSOP-14_4.4x5mm_P0.65mm" (id 2) (at 135.89 114.3 0)
-      (effects (font (size 1.27 1.27)) hide)
-    )
+    (property "Value" "" (id 1) (at 143.51 114.3 0))
+    (property "Footprint" "" (id 2) (at 135.89 114.3 0)
+      (effects (font (size 1.27 1.27)) hide)
+    )

Commit message: more progress
Parts:
- removed unit 5 of U3
- removed unit 1 of U3
- added C24: 100n, Capacitor_SMD:C_0402_1005Metric, symbol Device:C
- added C30: (no value), symbol Device:C
- added unit 3 of U12
- added unit 3 of U3
- added unit 2 of U3
- U12: renamed from U3; symbol Amplifier_Operational:MCP6004 -> Amplifier_Operational:MCP6002-xMS
- U3: value (none) -> MCP6002T-I/SN; footprint (none) -> Package_SO:SOIC-8_3.9x4.9mm_P1.27mm; symbol Amplifier_Operational:MCP6004 -> Amplifier_Operational:MCP6002-xMS
- U9: value GS8332 -> GS8332-SR; footprint Package_SO:TSSOP-8_3x3mm_P0.65mm -> Package_SO:SOIC-8_3.9x4.9mm_P1.27mm; LCSC C157714 -> C157713
Connections:
- net +3V3: now also C24.1, U12.8 (V+), U3.8 (V+)
- net GND: now also C24.2, C30.2, U12.4 (V-), U3.4 (V-)
- net Un_sense: now also U3.7
- net Vgnd_ref: now also U3.3 (+); no longer U12.12 (+), U3.10 (+)
- net at R14.1: now also U3.6 (-)
- net at R4.2: now also U12.1, C30.1; no longer U12.14
- net at R20.2, R45.2: now also U12.3 (+), U3.1, U3.2 (-); no longer U3.8, U3.9 (-)
- net at R13.2: now also U12.2 (-); no longer U12.13 (-)
- net at R1.2: now also U3.5 (+)
Other:
- note added: "caps for 2 x dual opamp"
- note added: "na"
- note removed: "caps for quad opamp"
- moved on the sheet: C8, R4, U3A

Commit message: progress
Parts:
- added R84: (no value), symbol Device:R
- C30: value (none) -> 1u; footprint (none) -> Capacitor_SMD:C_0402_1005Metric
- U12: value (none) -> MCP6002T-I/SN; footprint (none) -> Package_SO:SOIC-8_3.9x4.9mm_P1.27mm
Connections:
- net at C30.1, R4.2, U12.1: now also R84.1
- net at R13.2, U12.2 (-): now also R84.2
Other:
- note added: "DNI"
- note removed: "na"
- moved on the sheet: R13
Changed lines of the file:
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@@
   (junction (at 148.59 186.69) (diameter 0) (color 0 0 0 0)
+  )
+  (junction (at 119.38 80.01) (diameter 0) (color 0 0 0 0)
   )
   (junction (at 222.25 149.86) (diameter 0) (color 0 0 0 0)
@@
     (stroke (width 0) (type default) (color 0 0 0 0))
   )
-  (polyline (pts (xy 104.14 73.66) (xy 104.14 54.61))
+  (polyline (pts (xy 104.14 78.74) (xy 104.14 54.61))
     (stroke (width 0) (type default) (color 0 0 0 0))
   )
@@
     (stroke (width 0) (type default) (color 0 0 0 0))
   )
-  (wire (pts (xy 140.97 80.01) (xy 134.62 80.01))
+  (wire (pts (xy 140.97 80.01) (xy 119.38 80.01))
     (stroke (width 0) (type default) (color 0 0 0 0))
   )
@@
     (stroke (width 0) (type default) (color 0 0 0 0))
   )
-  (wire (pts (xy 92.71 80.01) (xy 127 80.01))
+  (wire (pts (xy 92.71 80.01) (xy 95.25 80.01))
     (stroke (width 0) (type default) (color 0 0 0 0))
   )
@@
     (stroke (width 0) (type default) (color 0 0 0 0))
   )
+  (wire (pts (xy 107.95 71.12) (xy 107.95 76.2))
+    (stroke (width 0) (type default) (color 0 0 0 0))
+  )
   (wire (pts (xy 222.25 236.22) (xy 222.25 234.95))
     (stroke (width 0) (type default) (color 0 0 0 0))
@@
     (stroke (width 0) (type default) (color 0 0 0 0))
   )
+  (wire (pts (xy 119.38 80.01) (xy 102.87 80.01))
+    (stroke (width 0) (type default) (color 0 0 0 0))
+  )
   (wire (pts (xy 222.25 149.86) (xy 222.25 151.13))
     (stroke (width 0) (type default) (color 0 0 0 0))
@@
     (stroke (width 0) (type default) (color 0 0 0 0))
   )
+  (wire (pts (xy 119.38 76.2) (xy 119.38 80.01))
+    (stroke (width 0) (type default) (color 0 0 0 0))
+  )
   (wire (pts (xy 148.59 116.84) (xy 148.59 128.27))
     (stroke (width 0) (type default) (color 0 0 0 0))
   )
-  (polyline (pts (xy 104.14 54.61) (xy 114.3 54.61))
+  (polyline (pts (xy 104.14 54.61) (xy 118.11 54.61))
     (stroke (width 0) (type default) (color 0 0 0 0))
   )
@@
     (stroke (width 0) (type default) (color 0 0 0 0))
   )
+  (wire (pts (xy 107.95 76.2) (xy 109.22 76.2))
+    (stroke (width 0) (type default) (color 0 0 0 0))
+  )
   (wire (pts (xy 175.26 40.64) (xy 175.26 43.18))
     (stroke (width 0) (type default) (color 0 0 0 0))
@@
     (stroke (width 0) (type default) (color 0 0 0 0))
   )
-  (polyline (pts (xy 104.14 73.66) (xy 114.3 73.66))
+  (polyline (pts (xy 104.14 78.74) (xy 118.11 78.74))
     (stroke (width 0) (type default) (color 0 0 0 0))
   )
@@
     (stroke (width 0) (type default) (color 0 0 0 0))
   )
+  (wire (pts (xy 116.84 76.2) (xy 119.38 76.2))
+    (stroke (width 0) (type default) (color 0 0 0 0))
+  )
   (wire (pts (xy 135.89 97.79) (xy 135.89 92.71))
     (stroke (width 0) (type default) (color 0 0 0 0))
@@
     (stroke (width 0) (type default) (color 0 0 0 0))
   )
-  (polyline (pts (xy 114.3 54.61) (xy 114.3 73.66))
+  (polyline (pts (xy 118.11 54.61) (xy 118.11 78.74))
     (stroke (width 0) (type default) (color 0 0 0 0))
   )
@@
     (effects (font (size 1.27 1.27)) (justify right bottom))
   )
-  (text "na" (at 107.95 53.34 0)
+  (text "DNI" (at 107.95 53.34 0)
     (effects (font (size 1.27 1.27)) (justify left bottom))
   )
@@
     (pin "1")
   )
+  (symbol (lib_id "Device:R") (at 113.03 76.2 90) (mirror x) (unit 1)
+    (in_bom no) (on_board yes)
+    (property "Reference" "R84" (id 0) (at 114.3 72.39 90)
+      (effects (font (size 1.27 1.27)) (justify left))
+    )
+    (property "Value" "" (id 1) (at 116.84 73.66 90)
+      (effects (font (size 1.27 1.27)) (justify left))
+    )
+    (property "Footprint" "" (id 2) (at 113.03 74.422 90)
+      (effects (font (size 1.27 1.27)) hide)
+    )
+    (property "Datasheet" "~" (id 3) (at 113.03 76.2 0)
+      (effects (font (size 1.27 1.27)) hide)
+    )
+    (property "LCSC" "C25744" (id 4) (at 113.03 76.2 0)
+      (effects (font (size 1.27 1.27)) hide)
+    )
+    (pin "1")
+    (pin "2")
+  )
   (symbol (lib_id "Device:C") (at 213.36 158.75 0) (unit 1)
     (in_bom yes) (on_board yes)
@@
     (in_bom yes) (on_board yes)
     (property "Reference" "U12" (id 0) (at 127 64.77 0))
-    (property "Value" "" (id 1) (at 126.365 67.31 0))
-    (property "Footprint" "" (id 2) (at 130.81 71.12 0)
+    (property "Value" "MCP6002T-I/SN" (id 1) (at 126.365 67.31 0))
+    (property "Footprint" "Package_SO:SOIC-8_3.9x4.9mm_P1.27mm" (id 2) (at 130.81 71.12 0)
       (effects (font (size 1.27 1.27)) hide)
     )
@@
       (effects (font (size 1.27 1.27)) (justify left))
     )
-    (property "Value" "" (id 1) (at 110.871 63.627 0)
-      (effects (font (size 1.27 1.27)) (justify left))
-    )
-    (property "Footprint" "" (id 2) (at 108.9152 60.96 0)
+    (property "Value" "1u" (id 1) (at 110.871 63.627 0)
+      (effects (font (size 1.27 1.27)) (justify left))
+    )
+    (property "Footprint" "Capacitor_SMD:C_0402_1005Metric" (id 2) (at 108.9152 60.96 0)
       (effects (font (size 1.27 1.27)) hide)
     )
@@
     (in_bom yes) (on_board yes)
     (property "Reference" "U12" (id 0) (at 201.93 152.4 0))
-    (property "Value" "" (id 1) (at 201.295 154.94 0))
-    (property "Footprint" "" (id 2) (at 205.74 158.75 0)
+    (property "Value" "MCP6002T-I/SN" (id 1) (at 201.295 154.94 0))
+    (property "Footprint" "Package_SO:SOIC-8_3.9x4.9mm_P1.27mm" (id 2) (at 205.74 158.75 0)
       (effects (font (size 1.27 1.27)) hide)
     )
@@
     (in_bom yes) (on_board yes)
     (property "Reference" "U12" (id 0) (at 139.7 194.31 0))
-    (property "Value" "" (id 1) (at 136.525 184.785 0))
-    (property "Footprint" "" (id 2) (at 139.7 189.23 0)
+    (property "Value" "MCP6002T-I/SN" (id 1) (at 136.525 184.785 0))
+    (property "Footprint" "Package_SO:SOIC-8_3.9x4.9mm_P1.27mm" (id 2) (at 139.7 189.23 0)
       (effects (font (size 1.27 1.27)) hide)
     )
@@
     (pin "2")
   )
-  (symbol (lib_id "Device:R") (at 130.81 80.01 90) (mirror x) (unit 1)
-    (in_bom yes) (on_board yes)
-    (property "Reference" "R13" (id 0) (at 127 76.2 90)
-      (effects (font (size 1.27 1.27)) (justify left))
-    )
-    (property "Value" "10k 1%" (id 1) (at 127 78.74 90)
-      (effects (font (size 1.27 1.27)) (justify left))
-    )
-    (property "Footprint" "Resistor_SMD:R_0402_1005Metric" (id 2) (at 130.81 78.232 90)
-      (effects (font (size 1.27 1.27)) hide)
-    )
-    (property "Datasheet" "~" (id 3) (at 130.81 80.01 0)
-      (effects (font (size 1.27 1.27)) hide)
-    )
-    (property "LCSC" "C25744" (id 4) (at 130.81 80.01 0)
-      (effects (font (size 1.27 1.27)) hide)
-    )
+  (symbol (lib_id "Device:R") (at 99.06 80.01 90) (mirror x) (unit 1)
+    (in_bom yes) (on_board yes)
+    (property "Reference" "R13" (id 0) (at 100.33 82.55 90)
+      (effects (font (size 1.27 1.27)) (justify left))
+    )
+    (property "Value" "10k 1%" (id 1) (at 101.6 85.09 90)
+      (effects (font (size 1.27 1.27)) (justify left))
+    )
+    (property "Footprint" "Resistor_SMD:R_0402_1005Metric" (id 2) (at 99.06 78.232 90)
+      (effects (font (size 1.27 1.27)) hide)
+    )
+    (property "Datasheet" "~" (id 3) (at 99.06 80.01 0)
+      (effects (font (size 1.27 1.27)) hide)
+    )
+    (property "LCSC" "C25744" (id 4) (at 99.06 80.01 0)
+      (effects (font (size 1.27 1.27)) hide)
+    )

Commit message: more progress
Parts:
- R84: value (none) -> 10k 1%; footprint (none) -> Resistor_SMD:R_0402_1005Metric
Other:
- moved on the sheet: R1, R11, R12, R21, R3, R7, R9

Commit message: Progress
Parts:
- removed C12: 100n, Capacitor_SMD:C_0402_1005Metric, symbol Device:C
- removed R46: 100k 1%, Resistor_SMD:R_0402_1005Metric, symbol Device:R
- removed R51: 10k 1%, Resistor_SMD:R_0402_1005Metric, symbol Device:R
Changed lines of the file:
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@@
   (junction (at 128.27 148.59) (diameter 0) (color 0 0 0 0)
   )
-  (junction (at 181.61 40.64) (diameter 0) (color 0 0 0 0)
-  )
   (junction (at 148.59 151.13) (diameter 0) (color 0 0 0 0)
   )
@@
   )
   (junction (at 149.86 226.06) (diameter 0) (color 0 0 0 0)
-  )
-  (junction (at 175.26 40.64) (diameter 0) (color 0 0 0 0)
   )
   (junction (at 195.58 68.58) (diameter 0) (color 0 0 0 0)
@@
     (stroke (width 0) (type default) (color 0 0 0 0))
   )
-  (wire (pts (xy 181.61 52.07) (xy 181.61 50.8))
-    (stroke (width 0) (type default) (color 0 0 0 0))
-  )
   (wire (pts (xy 128.27 160.655) (xy 134.62 160.655))
     (stroke (width 0) (type default) (color 0 0 0 0))
@@
     (stroke (width 0) (type default) (color 0 0 0 0))
   )
-  (wire (pts (xy 175.26 40.64) (xy 181.61 40.64))
-    (stroke (width 0) (type default) (color 0 0 0 0))
-  )
   (wire (pts (xy 157.48 92.71) (xy 187.96 92.71))
     (stroke (width 0) (type default) (color 0 0 0 0))
@@
     (stroke (width 0) (type default) (color 0 0 0 0))
   )
-  (wire (pts (xy 152.4 40.64) (xy 82.55 40.64))
-    (stroke (width 0) (type default) (color 0 0 0 0))
-  )
   (wire (pts (xy 227.33 149.86) (xy 227.33 154.94))
     (stroke (width 0) (type default) (color 0 0 0 0))
@@
     (stroke (width 0) (type default) (color 0 0 0 0))
   )
-  (wire (pts (xy 175.26 40.64) (xy 175.26 43.18))
-    (stroke (width 0) (type default) (color 0 0 0 0))
-  )
   (wire (pts (xy 149.86 226.06) (xy 152.4 226.06))
     (stroke (width 0) (type default) (color 0 0 0 0))
@@
     (stroke (width 0) (type default) (color 0 0 0 0))
   )
-  (wire (pts (xy 160.02 40.64) (xy 175.26 40.64))
-    (stroke (width 0) (type default) (color 0 0 0 0))
-  )
   (wire (pts (xy 129.54 179.07) (xy 129.54 189.23))
     (stroke (width 0) (type default) (color 0 0 0 0))
@@
     (stroke (width 0) (type default) (color 0 0 0 0))
   )
-  (wire (pts (xy 181.61 40.64) (xy 187.96 40.64))
-    (stroke (width 0) (type default) (color 0 0 0 0))
-  )
   (wire (pts (xy 147.32 186.69) (xy 148.59 186.69))
     (stroke (width 0) (type default) (color 0 0 0 0))
@@
     (stroke (width 0) (type default) (color 0 0 0 0))
   )
-  (wire (pts (xy 181.61 40.64) (xy 181.61 43.18))
-    (stroke (width 0) (type default) (color 0 0 0 0))
-  )
   (wire (pts (xy 97.79 189.23) (xy 100.33 189.23))
     (stroke (width 0) (type default) (color 0 0 0 0))
@@
   )
   (wire (pts (xy 90.17 189.23) (xy 87.63 189.23))
-    (stroke (width 0) (type default) (color 0 0 0 0))
-  )
-  (wire (pts (xy 82.55 40.64) (xy 82.55 71.12))
-    (stroke (width 0) (type default) (color 0 0 0 0))
-  )
-  (wire (pts (xy 175.26 52.07) (xy 175.26 50.8))
     (stroke (width 0) (type default) (color 0 0 0 0))
   )
@@
     (effects (font (size 1.27 1.27)) (justify left))
   )
-  (hierarchical_label "Vm_sense" (shape output) (at 187.96 40.64 0)
-    (effects (font (size 1.27 1.27)) (justify left))
-  )
   (hierarchical_label "Nernst_4.9_esr_drive" (shape input) (at 187.96 97.79 0)
     (effects (font (size 1.27 1.27)) (justify left))
@@
     (pin "2")
   )
-  (symbol (lib_id "Device:R") (at 156.21 40.64 90) (mirror x) (unit 1)
-    (in_bom yes) (on_board yes)
-    (property "Reference" "R46" (id 0) (at 157.48 35.56 90)
-      (effects (font (size 1.27 1.27)) (justify left))
-    )
-    (property "Value" "100k 1%" (id 1) (at 160.02 38.1 90)
-      (effects (font (size 1.27 1.27)) (justify left))
-    )
-    (property "Footprint" "Resistor_SMD:R_0402_1005Metric" (id 2) (at 156.21 38.862 90)
-      (effects (font (size 1.27 1.27)) hide)
-    )
-    (property "Datasheet" "~" (id 3) (at 156.21 40.64 0)
-      (effects (font (size 1.27 1.27)) hide)
-    )
-    (property "LCSC" "C25741" (id 4) (at 156.21 40.64 0)
-      (effects (font (size 1.27 1.27)) hide)
-    )
-    (pin "1")
-    (pin "2")
-  )
   (symbol (lib_id "power:GND") (at 222.25 236.22 0) (unit 1)
     (in_bom yes) (on_board yes)
@@
     )
     (property "Datasheet" "" (id 3) (at 222.25 236.22 0)
-      (effects (font (size 1.27 1.27)) hide)
-    )
-    (pin "1")
-  )
-  (symbol (lib_id "power:GND") (at 181.61 52.07 0) (unit 1)
-    (in_bom yes) (on_board yes)
-    (property "Reference" "#PWR0129" (id 0) (at 181.61 58.42 0)
-      (effects (font (size 1.27 1.27)) hide)
-    )
-    (property "Value" "GND" (id 1) (at 181.737 56.4642 0))
-    (property "Footprint" "" (id 2) (at 181.61 52.07 0)
-      (effects (font (size 1.27 1.27)) hide)
-    )
-    (property "Datasheet" "" (id 3) (at 181.61 52.07 0)
       (effects (font (size 1.27 1.27)) hide)
     )
@@
     (pin "1")
   )
-  (symbol (lib_id "power:GND") (at 175.26 52.07 0) (unit 1)
-    (in_bom yes) (on_board yes)
-    (property "Reference" "#PWR0128" (id 0) (at 175.26 58.42 0)
-      (effects (font (size 1.27 1.27)) hide)
-    )
-    (property "Value" "GND" (id 1) (at 175.387 56.4642 0))
-    (property "Footprint" "" (id 2) (at 175.26 52.07 0)
-      (effects (font (size 1.27 1.27)) hide)
-    )
-    (property "Datasheet" "" (id 3) (at 175.26 52.07 0)
-      (effects (font (size 1.27 1.27)) hide)
-    )
-    (pin "1")
-  )
   (symbol (lib_id "Device:R") (at 113.03 76.2 90) (mirror x) (unit 1)
     (in_bom no) (on_board yes)
@@
     (pin "2")
   )
-  (symbol (lib_id "Device:C") (at 181.61 46.99 0) (mirror y) (unit 1)
-    (in_bom yes) (on_board yes)
-    (property "Reference" "C12" (id 0) (at 186.69 44.45 0)
-      (effects (font (size 1.27 1.27)) (justify left))
-    )
-    (property "Value" "100n" (id 1) (at 189.23 48.26 0)
-      (effects (font (size 1.27 1.27)) (justify left))
-    )
-    (property "Footprint" "Capacitor_SMD:C_0402_1005Metric" (id 2) (at 180.6448 50.8 0)
-      (effects (font (size 1.27 1.27)) hide)
-    )
-    (property "Datasheet" "~" (id 3) (at 181.61 46.99 0)
-      (effects (font (size 1.27 1.27)) hide)
-    )
-    (property "LCSC" "C1525" (id 4) (at 181.61 46.99 0)
-      (effects (font (size 1.27 1.27)) hide)
-    )
-    (pin "1")
-    (pin "2")
-  )
   (symbol (lib_id "Device:C") (at 107.95 64.77 0) (mirror x) (unit 1)
     (in_bom no) (on_board yes)
@@
       (effects (font (size 1.27 1.27)) hide)
     )
-    (pin "1")
-    (pin "2")
-  )
-  (symbol (lib_id "Device:R") (at 175.26 46.99 0) (mirror x) (unit 1)
-    (in_bom yes) (on_board yes)
-    (property "Reference" "R51" (id 0) (at 168.91 45.72 0)
-      (effects (font (size 1.27 1.27)) (justify left))
-    )
-    (property "Value" "10k 1%" (id 1) (at 165.1 48.26 0)
-      (effects (font (size 1.27 1.27)) (justify left))
-    )
-    (property "Footprint" "Resistor_SMD:R_0402_1005Metric" (id 2) (at 173.482 46.99 90)
-      (effects (font (size 1.27 1.27)) hide)
-    )
-    (property "Datasheet" "~" (id 3) (at 175.26 46.99 0)
-      (effects (font (size 1.27 1.27)) hide)
-    )
-    (property "LCSC" "C25744" (id 4) (at 175.26 46.99 0)
-      (effects (font (size 1.27 1.27)) hide)
-    )

Commit message: Progress
Parts:
- added D13, D14, D15, D16, D17, D27: DF2B7AFS,L3M, Diode_SMD:D_SOD-923, symbol Diode:ESD9B5.0ST5G
- added Q5, Q6, Q7, Q8: BSS169H6327, Package_TO_SOT_SMD:SOT-23, symbol Transistor_FET:BSS123
- added R76, R78: 75R, Resistor_SMD:R_0603_1608Metric, symbol Device:R
- added TP10, TP11, TP12, TP3: (no value), symbol Connector:TestPoint_Probe
- added TP13, TP14: Un, TestPoint:TestPoint_Pad_D1.0mm, symbol Connector:TestPoint_Probe
- added TP15: Ip_DAC, TestPoint:TestPoint_Pad_D1.0mm, symbol Connector:TestPoint_Probe
- added TP16: Ip_Sense, TestPoint:TestPoint_Pad_D1.0mm, symbol Connector:TestPoint_Probe
- added TP5: 3xUn, TestPoint:TestPoint_Pad_D1.0mm, symbol Connector:TestPoint_Probe
Connections:
- net GND: now also D13.2 (A2), D14.2 (A2), D15.2 (A2), D16.2 (A2), D17.2 (A2), D27.2 (A2)
- net Ip_dac: now also TP15.1
- net Ip_sense: now also TP16.1
- net LSU_Ip: now also TP10.1
- net LSU_Rtrim: now also Q8.3 (D), TP11.1
- net LSU_Un: now also TP13.1
- net LSU_Vm: now also Q6.3 (D), TP12.1
- net Un_3x_sense: now also TP5.1
- net Un_sense: now also TP3.1
- net at C9.1, R12.2, R18.1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: now also Q7.3 (D)
- net at R19.2, R9.1, U9.2 (-): now also D16.1 (A1)
- net at R17.1, R7.1, U9.6 (-): now also D14.1 (A1)
- net at C30.1, R4.2, R84.1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: now also Q5.3 (D)
- net at R20.2, R45.2, U12.3 (+)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: now also TP14.1
- net at R13.2, R84.2, U12.2 (-): now also D17.1 (A1)
- net at R21.2, R45.1, U12.5 (+): now also D27.1 (A1)
- net at R1.2, U3.5 (+): now also D13.1 (A1)
- net at R11.1, R20.1, U9.3 (+): now also D15.1 (A1)
- new net: Q5.1 (G), Q6.2 (S), R76.1
- new net: Q5.2 (S), Q6.1 (G), R76.2
- new net: Q7.2 (S), Q8.1 (G), R78.2
- new net: Q7.1 (G), Q8.2 (S), R78.1
Other:
- note added: "Current limiter (25 mA)"
- note added: "Virtual ground should be at least 1.8 for this circuit to work"
- moved on the sheet: C11, C14, C30, C9, R11, R12, R18, R19, R20, R21, R3, R42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
