File: lambda-x2/lsu.kicad_sch (KiCad schematic)
At the start: 56 parts, among them Q5 BSS169H6327, Q6 BSS169H6327, Q7 BSS169H6327, Q8 BSS169H6327, U12 MCP6002T-I/SN, U3 MCP6002T-I/SN, U9 GS8332-SR

Commit message: Lambda x2 rev1 (#180)
* lambda-x2: revork aux outputs, remove useless protection in LSU

* lambda-x2: switch to 64-pin MCU

* lambda-x2: add HSE, move pump to DAC outputs

* lambda-x2: move BT to UART4/USART3

* lambda-x2: ocsillator fix

* lambda-x2: fix RC filter values on heater voltage ADC inputs

* lambda-x2: fuse, Vbat sense, resistor in sense

* lambda-x2: diagnostic for AUX out, PWM noise cancelation, etc

* lambda-x2: jtag, adc channels, one more led, BT en, etc

* lambda-x2: update PCB dimentions, connector footprint, etx

* lambda-x2: update

* lambda-x2: final update, rev1

* lambda-x2: rev1: fabrication files
Parts:
- removed Q5, Q6, Q7, Q8: BSS169H6327, Package_TO_SOT_SMD:SOT-23, symbol Transistor_FET:BSS123
- removed R76, R78: 75R, Resistor_SMD:R_0603_1608Metric, symbol Device:R
- added R107: 10k, Resistor_SMD:R_0402_1005Metric, symbol Device:R
- C9: now left out of the parts list
- R15: value 10k 0.1% -> 2.7k 0.1%; LCSC C309083 -> C318131
- R5: value 30k 1% -> 10k 0.1%; LCSC C22984 -> C309083
Connections:
- net Ip_dac: now also R107.1
- net at R20.2, R45.2, TP14.1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: now also R107.2
Other:
- note added: "Un_3x_sense = 0.247 + 3.15 * (Un - Vm)"
- note added: "Zero current while in reset"
- note removed: "Current limiter (25 mA)"
- note removed: "Un_sense = 3.000 * (Un - Vm)"
- note removed: "Virtual ground should be at least 1.8 for this circuit to work"
- moved on the sheet: R15, R5
