File: lambda-x2/lambda-x2.kicad_pcb (KiCad board)
At the start: 4 copper layers, 87 x 106 mm, 143 parts, among them J1 FTSH-107-01-F-DV-K, J3 Conn_02x02_Odd_Even, J4 Conn_01x10, P1 33311-24AW-2, Q2 BTS3028, U10 MCP6004, U11 GS8332, U2 STM32F103C6Tx, U3 MCP6004, U4 LM78M05_TO252, U5 XC6206P332MR, U6 REF3033, U7 MCP6002T-I/SN, U8 TJA1051T-3, U9 GS8332

Commit message: lambda-x2: some upadte
Parts:
- moved C16 80.8 mm to (147.6, 50.9), turned to 90 degrees
- moved R62 79.7 mm to (149.7, 53.3)
- moved C15 77.7 mm to (149.9, 56.5)
- moved R72 73.4 mm to (152.0, 58.7), turned to -90 degrees
- moved R54 71.8 mm to (149.9, 55.5)
- moved R71 70.5 mm to (150.4, 58.7), turned to -90 degrees
- moved R56 68.5 mm to (150.4, 51.3)
- moved R73 67.3 mm to (148.7, 58.7), turned to -90 degrees
- moved R70 66.0 mm to (147.1, 58.7), turned to 90 degrees
- moved C18 62.8 mm to (173.3, 47.6), turned to 180 degrees
- moved R60 62.6 mm to (162.7, 51.7), turned to 180 degrees
- moved R69 62.2 mm to (162.9, 57.7), turned to -90 degrees
- moved R61 61.6 mm to (164.2, 57.1), turned to -90 degrees
- moved R59 61.4 mm to (162.7, 53.6), turned to 180 degrees
- moved C23 60.6 mm to (171.7, 52.5), turned to 90 degrees
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Connections:
- U10 pad 1: /R_Un_sense -> Net-(R68-Pad2)
- U10 pad 12: /LSU analog left/Vgnd_ref -> Net-(R54-Pad2)
- U10 pad 13: Net-(R62-Pad2) -> Net-(R63-Pad1)
- U10 pad 14: Net-(R56-Pad2) -> /R_Un_sense
- U10 pad 2: Net-(R63-Pad1) -> Net-(R68-Pad2)
- U10 pad 3: Net-(R54-Pad2) -> /LSU analog left/Vgnd_ref
- U10 pad 8: Net-(R68-Pad2) -> Net-(R56-Pad2)
- U10 pad 9: Net-(R68-Pad2) -> Net-(R62-Pad2)
Routing:
- net /R_LSU_Rtrim: track 0.00 -> 37.9 mm, vias 0 -> 1
- net /L_LSU_Vm: track 41.5 -> 78.4 mm, vias 0 -> 3
- net /L_LSU_Un: track 33.7 -> 0.00 mm, vias 2 -> 0
- net /R_LSU_Vm: track 0.00 -> 30.8 mm, vias 0 -> 1
- net Net-(R20-Pad2): track 34.9 -> 62.0 mm, vias 2 -> 5
- net /R_LSU_Ip: track 0.00 -> 26.1 mm, vias 0 -> 1
- net Net-(R68-Pad2): track 0.00 -> 25.4 mm, vias 0 -> 2
- net /R_LSU_Un: track 0.00 -> 23.3 mm
- net /Nernst_4.9_esr_drive: track 10.9 -> 33.7 mm, vias 0 -> 2
- net Net-(R62-Pad2): track 0.00 -> 20.2 mm
- net Net-(R54-Pad2): track 0.00 -> 18.6 mm
- net Net-(R56-Pad2): track 0.00 -> 18.3 mm
- net Net-(C9-Pad2): track 61.1 -> 45.6 mm, vias 4 -> 2
- net Net-(C9-Pad1): track 27.1 -> 12.3 mm, vias 3 -> 0
- net /R_Un_sense: track 0.00 -> 12.9 mm, vias 0 -> 2
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
Commit message: more progress
Parts:
- removed TP3, TP4, TP5: TestPoint, TestPoint:TestPoint_Pad_D1.0mm
- added C24: 100n, Capacitor_SMD:C_0402_1005Metric, F.Cu at (151.0, 56.0)
- added C29: 100n, Capacitor_SMD:C_0402_1005Metric, F.Cu at (172.8, 56.0)
- added C30: 1u, Capacitor_SMD:C_0402_1005Metric, F.Cu at (143.4, 51.4)
- added C31: 1u, Capacitor_SMD:C_0402_1005Metric, F.Cu at (165.5, 51.4)
- added C35: 100n, Capacitor_SMD:C_0402_1005Metric, F.Cu at (107.7, 76.6)
- added D3: RED, LED_SMD:LED_0603_1608Metric, F.Cu at (112.2, 70.3)
- added Q1: BTS3028, Package_TO_SOT_SMD:TO-252-2, F.Cu at (110.5, 63.9)
- added R79: 1k, Resistor_SMD:R_0402_1005Metric, F.Cu at (110.6, 72.6)
- added R80: 10k, Resistor_SMD:R_0402_1005Metric, F.Cu at (107.7, 74.6)
- added R81: 100k 1%, Resistor_SMD:R_0402_1005Metric, F.Cu at (118.5, 70.0)
- added R82: 10k 1%, Resistor_SMD:R_0402_1005Metric, F.Cu at (115.6, 70.0)
- added R83: 1k, Resistor_SMD:R_0402_1005Metric, F.Cu at (107.7, 72.6)
- added U12: MCP6002T-I/SN, Package_SO:SOIC-8_3.9x4.9mm_P1.27mm, F.Cu at (147.7, 56.0)
- added U13: MCP6002T-I/SN, Package_SO:SOIC-8_3.9x4.9mm_P1.27mm, F.Cu at (169.6, 56.0)
- U10, U3: value MCP6004 -> MCP6002T-I/SN; footprint Package_SO:TSSOP-14_4.4x5mm_P0.65mm -> Package_SO:SOIC-8_3.9x4.9mm_P1.27mm
- U11, U9: value GS8332 -> GS8332-SR; footprint Package_SO:TSSOP-8_3x3mm_P0.65mm -> Package_SO:SOIC-8_3.9x4.9mm_P1.27mm
- moved C3 49.7 mm to (136.4, 57.4), turned to 180 degrees
- moved R4 48.1 mm to (142.0, 49.7), turned to 0 degrees
- moved R21 45.0 mm to (144.0, 56.1), turned to 0 degrees
- moved R18 44.9 mm to (147.7, 60.3), turned to 180 degrees
- moved R13 44.6 mm to (142.0, 52.6), turned to 0 degrees
- moved R11 43.8 mm to (140.7, 58.8)
- moved R41 42.9 mm to (132.6, 59.4), turned to -90 degrees
- moved R47 41.6 mm to (144.9, 65.3)
- moved D4 39.6 mm to (96.8, 68.3)
- moved R3 37.4 mm to (139.4, 54.9)
- moved Q2 37.3 mm to (110.5, 55.0), turned to 0 degrees
- moved C13 37.0 mm to (131.7, 67.2), turned to -90 degrees
- moved R12 35.0 mm to (143.5, 54.9), turned to 0 degrees
- moved R1 34.8 mm to (138.4, 59.4), turned to -90 degrees
- moved R9 34.0 mm to (142.5, 58.8), turned to 90 degrees
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Connections:
- P1 pad 10: /L_LSU_Vm -> unconnected-(P1-Pad10)
- P1 pad 12: unconnected-(P1-Pad12) -> /L_LSU_Vm
- P1 pad 17: /L_LSU_Heater- -> unconnected-(P1-Pad17)
- P1 pad 18: /L_LSU_Ip -> unconnected-(P1-Pad18)
- P1 pad 19: /L_LSU_Un -> unconnected-(P1-Pad19)
- P1 pad 3: unconnected-(P1-Pad3) -> /L_LSU_Un
- P1 pad 4: unconnected-(P1-Pad4) -> /L_LSU_Ip
- P1 pad 5: unconnected-(P1-Pad5) -> /L_LSU_Heater-
- R70 pad 1: /LSU analog right/Nernst_4.9_bias -> /Nernst_4.9_bias
- R71 pad 2: /LSU analog right/Nernst_4.9_esr_drive -> /Nernst_4.9_esr_drive
- R72 pad 2: /LSU analog right/Nernst_ADV_esr_drive -> /Nernst_ADV_esr_drive
- R73 pad 2: /LSU analog right/Nernst_4.2_esr_drive -> /Nernst_4.2_esr_drive
- U10 pad 4: +3V3 -> GND
- U10 pad 5: Net-(R69-Pad2) -> Net-(R54-Pad2)
- U10 pad 6: Net-(C17-Pad2) -> Net-(R63-Pad1)
- U10 pad 7: Net-(C17-Pad1) -> /R_Un_sense
- U10 pad 8: Net-(R56-Pad2) -> +3V3
- U2 pad 12: Net-(TP5-Pad1) -> /R_Ip_sense
- U2 pad 13: Net-(TP3-Pad1) -> /R_Un_3x_sense
- U2 pad 14: Net-(TP4-Pad1) -> /R_Un_sense
- U2 pad 15: /L_Un_sense -> /L_Ip_sense
- U2 pad 16: /L_Ip_sense -> /L_Un_3x_sense
- U2 pad 17: /L_Un_3x_sense -> /L_Un_sense
- U3 pad 1: /L_Un_sense -> Net-(R20-Pad2)
- U3 pad 2: Net-(R14-Pad1) -> Net-(R20-Pad2)
- U3 pad 3: Net-(R1-Pad2) -> /LSU analog left/Vgnd_ref
- U3 pad 4: +3V3 -> GND
- U3 pad 5: Net-(R21-Pad2) -> Net-(R1-Pad2)
- U3 pad 6: Net-(C9-Pad2) -> Net-(R14-Pad1)
- U3 pad 7: Net-(C9-Pad1) -> /L_Un_sense
- U3 pad 8: Net-(R20-Pad2) -> +3V3
Routing:
- net /R_LSU_Vm: track 30.8 -> 99.3 mm, vias 1 -> 2
- net GND: track 126.1 -> 177.5 mm, vias 99 -> 94
- net VDDA: track 95.3 -> 47.5 mm
- net /R_LSU_Heater-: track 0.00 -> 47.5 mm, vias 0 -> 4
- net 12V_PROT: track 58.6 -> 16.4 mm
- net Net-(C9-Pad2): track 45.6 -> 3.95 mm, vias 2 -> 0
- net /Nernst_4.2_esr_drive: track 3.53 -> 44.2 mm, vias 0 -> 3
- net Net-(C3-Pad2): track 44.2 -> 4.40 mm, vias 3 -> 0
- net /L_Un_sense: track 0.00 -> 34.7 mm
- net 12V_RAW: track 0.00 -> 34.5 mm
- net /R_Ip_sense: track 1.04 -> 32.7 mm
- net /L_LSU_Rtrim: track 0.00 -> 29.1 mm
- net /Nernst_4.9_bias: track 5.11 -> 33.2 mm, vias 0 -> 3
- net /R_Un_3x_sense: track 2.35 -> 29.1 mm
- net /l_Heater_sense: track 26.5 -> 0.00 mm, vias 2 -> 0
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
Commit message: progress
Parts:
- added C37: 100n, Capacitor_SMD:C_0402_1005Metric, F.Cu at (164.1, 105.4)
- added C43: 1u, Capacitor_SMD:C_0402_1005Metric, F.Cu at (164.1, 104.4)
- added C46: 100n, Capacitor_SMD:C_0402_1005Metric, F.Cu at (164.0, 113.3)
- added C47: 1u, Capacitor_SMD:C_0402_1005Metric, F.Cu at (164.0, 112.3)
- added C48: 10nF 50V, Capacitor_SMD:C_0402_1005Metric, F.Cu at (190.0, 64.3)
- added C49: 100n, Capacitor_SMD:C_0402_1005Metric, F.Cu at (184.2, 80.6)
- added C50: 10nF 50V, Capacitor_SMD:C_0402_1005Metric, F.Cu at (187.1, 64.3)
- added C51: 10nF 50V, Capacitor_SMD:C_0402_1005Metric, F.Cu at (200.9, 64.3)
- added C52: 100n, Capacitor_SMD:C_0402_1005Metric, F.Cu at (198.0, 66.2)
- added C53: 10nF 50V, Capacitor_SMD:C_0402_1005Metric, F.Cu at (198.0, 64.3)
- added D7: NUP2105L, Package_TO_SOT_SMD:SOT-23, F.Cu at (167.8, 108.2)
- added D9: NUP2105L, Package_TO_SOT_SMD:SOT-23, F.Cu at (179.8, 108.2)
- added L1: 470R@100MHz, Inductor_SMD:L_0603_1608Metric, F.Cu at (168.9, 108.1)
- added L2: 470R@100MHz, Inductor_SMD:L_0603_1608Metric, F.Cu at (168.6, 116.0)
- added L3: 470R@100MHz, Inductor_SMD:L_0603_1608Metric, F.Cu at (172.2, 107.2)
- added L4: 470R@100MHz, Inductor_SMD:L_0603_1608Metric, F.Cu at (184.2, 107.2)
- added R84: 10k 1%, Resistor_SMD:R_0402_1005Metric, F.Cu at (145.4, 50.3)
- added R85: 10k 1%, Resistor_SMD:R_0402_1005Metric, F.Cu at (167.5, 50.3)
- added U1: MAX31855KASA, Package_SO:SOIC-8_3.9x4.9mm_P1.27mm, F.Cu at (162.1, 108.7)
- added U14: MAX31855KASA, Package_SO:SOIC-8_3.9x4.9mm_P1.27mm, F.Cu at (162.1, 116.6)
Connections:
- J1 pad 8: /SWO -> unconnected-(J1-Pad8)
- J4 pad 3: /DISP0 -> unconnected-(J4-Pad3)
- J4 pad 4: /SWO -> unconnected-(J4-Pad4)
- J4 pad 5: /DISP1 -> unconnected-(J4-Pad5)
- J4 pad 6: /DISP2 -> unconnected-(J4-Pad6)
- P1 pad 19: unconnected-(P1-Pad19) -> /L_EGT+
- P1 pad 20: unconnected-(P1-Pad20) -> /L_EGT-
- P1 pad 21: /CAN_H -> unconnected-(P1-Pad21)
- P1 pad 22: /CAN_L -> /R_EGT+
- P1 pad 23: unconnected-(P1-Pad23) -> /R_EGT-
- U2 pad 38: /DISP0 -> /SPI1_NSS
- U2 pad 39: /SWO -> /SPI1_SCK
- U2 pad 40: /DISP1 -> /SPI1_MISO
- U2 pad 41: /DISP2 -> /SPI1_MOSI
Routing:
- net /SWO: track 41.8 -> 0.00 mm, vias 2 -> 0
- net unconnected-(J1-Pad8): track 0.00 -> 23.9 mm, vias 0 -> 1
- net /DISP0: track 20.0 -> 0.00 mm
- net unconnected-(J4-Pad5): track 0.00 -> 15.9 mm
- net /DISP1: track 15.9 -> 0.00 mm
- net unconnected-(J4-Pad3): track 0.00 -> 14.8 mm
- net unconnected-(J4-Pad6): track 0.00 -> 14.4 mm
- net /DISP2: track 14.4 -> 0.00 mm
- net unconnected-(J4-Pad4): track 0.00 -> 13.7 mm
- net /Nernst_ADV_esr_drive: track 42.8 -> 33.0 mm
- net /Nernst_4.9_esr_drive: track 43.8 -> 34.5 mm
- net /Nernst_4.2_esr_drive: track 44.2 -> 35.2 mm
- net /SPI1_NSS: track 0.00 -> 5.16 mm
- net /SPI1_SCK: track 0.00 -> 4.19 mm, vias 0 -> 1
- net Net-(C31-Pad1): track 11.1 -> 13.8 mm
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
Commit message: more progress
Parts:
- added C54: 1u, Capacitor_SMD:C_0402_1005Metric, F.Cu at (102.4, 95.6)
- added C55: 100n, Capacitor_SMD:C_0402_1005Metric, F.Cu at (103.4, 95.6)
- added C56: 100n, Capacitor_SMD:C_0402_1005Metric, F.Cu at (103.4, 100.4)
- added C57: 100n, Capacitor_SMD:C_0402_1005Metric, F.Cu at (111.1, 117.0)
- added C58: 10nF 50V, Capacitor_SMD:C_0402_1005Metric, F.Cu at (163.1, 100.8)
- added C59: 100n, Capacitor_SMD:C_0402_1005Metric, F.Cu at (163.1, 98.8)
- added C60: 10nF 50V, Capacitor_SMD:C_0402_1005Metric, F.Cu at (163.1, 96.8)
- added C61: 100n, Capacitor_SMD:C_0402_1005Metric, F.Cu at (157.6, 95.2)
- added C62: 100n, Capacitor_SMD:C_0402_1005Metric, F.Cu at (159.5, 95.2)
- added C63: 10nF 50V, Capacitor_SMD:C_0402_1005Metric, F.Cu at (163.1, 114.8)
- added C64: 100n, Capacitor_SMD:C_0402_1005Metric, F.Cu at (163.1, 112.8)
- added C65: 10nF 50V, Capacitor_SMD:C_0402_1005Metric, F.Cu at (163.1, 110.7)
- added C66: 100n, Capacitor_SMD:C_0402_1005Metric, F.Cu at (157.6, 109.2)
- added C67: 100n, Capacitor_SMD:C_0402_1005Metric, F.Cu at (159.5, 109.2)
- added D10: RED, LED_SMD:LED_0603_1608Metric, F.Cu at (102.7, 53.1)
- added D11: RED, LED_SMD:LED_0603_1608Metric, F.Cu at (102.7, 80.3)
- added D12: NUP2105L, Package_TO_SOT_SMD:SOT-23, F.Cu at (106.4, 113.7)
- added Q3: BTS3028, Package_TO_SOT_SMD:TO-252-2, F.Cu at (110.5, 53.3)
- added Q4: BTS3028, Package_TO_SOT_SMD:TO-252-2, F.Cu at (110.5, 80.4)
- added R100: 160k, Resistor_SMD:R_0603_1608Metric, F.Cu at (127.4, 73.4)
- added R101: 160k, Resistor_SMD:R_0603_1608Metric, F.Cu at (71.9, 90.8)
- added R86: 1k, Resistor_SMD:R_0402_1005Metric, F.Cu at (104.1, 50.5)
- added R87: 1k, Resistor_SMD:R_0402_1005Metric, F.Cu at (104.1, 77.6)
- added R88: 10k, Resistor_SMD:R_0402_1005Metric, F.Cu at (104.1, 52.6)
- added R89: 10k, Resistor_SMD:R_0402_1005Metric, F.Cu at (104.1, 79.6)
- added R90: 1k, Resistor_SMD:R_0402_1005Metric, F.Cu at (102.7, 50.5)
- added R91: 1k, Resistor_SMD:R_0402_1005Metric, F.Cu at (102.7, 77.6)
- added R92: 100R, Resistor_SMD:R_0402_1005Metric, F.Cu at (164.6, 98.3)
- added R93: 100R, Resistor_SMD:R_0402_1005Metric, F.Cu at (164.6, 99.3)
- added R94: 100R, Resistor_SMD:R_0402_1005Metric, F.Cu at (164.6, 112.3)
- added R95: 100R, Resistor_SMD:R_0402_1005Metric, F.Cu at (164.6, 113.3)
- added R96: 10k 0.1%, Resistor_SMD:R_0603_1608Metric, F.Cu at (122.8, 61.6)
- added R97: 10k 0.1%, Resistor_SMD:R_0603_1608Metric, F.Cu at (124.7, 61.6)
- added R98: 82k, Resistor_SMD:R_0603_1608Metric, F.Cu at (75.9, 90.8)
- added R99: 82k, Resistor_SMD:R_0603_1608Metric, F.Cu at (67.9, 90.8)
- added U15: MAX31856, Package_SO:TSSOP-14_4.4x5mm_P0.65mm, F.Cu at (158.6, 98.6)
- added U16: MAX31856, Package_SO:TSSOP-14_4.4x5mm_P0.65mm, F.Cu at (158.6, 112.5)
- added U17: MCP6002T-I/SN, Package_SO:SO-8_3.9x4.9mm_P1.27mm, F.Cu at (125.3, 67.2)
- R43: value 100k 1% -> 3.3k
- R44: value 10k 1% -> 3.3k
- moved C51 68.4 mm to (163.1, 121.3), turned to -90 degrees
- moved C52 63.5 mm to (163.1, 119.3), turned to 90 degrees
- moved C53 63.5 mm to (163.1, 117.2), turned to 90 degrees
- moved R29 62.6 mm to (102.7, 59.6), turned to 90 degrees
- moved D8 57.6 mm to (102.7, 62.1), turned to 90 degrees
- moved J4 53.4 mm to (173.0, 134.4), turned to -90 degrees
- moved C48 50.8 mm to (163.1, 107.3), turned to -90 degrees
- moved C50 45.8 mm to (163.1, 103.3), turned to 90 degrees
- moved R8 41.4 mm to (128.5, 83.6), turned to 0 degrees
- moved R26 41.4 mm to (104.1, 59.6), turned to 90 degrees
- moved D1 40.3 mm to (131.1, 83.6), turned to 0 degrees
- moved R10 39.9 mm to (128.5, 86.1), turned to 0 degrees
- moved D2 39.1 mm to (131.1, 86.1), turned to 0 degrees
- moved R30 38.9 mm to (104.1, 61.6), turned to 90 degrees
- moved R23 38.7 mm to (128.5, 88.6), turned to 0 degrees
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Connections:
- C10 pad 1: /l_Heater_sense -> /L_Heater_sense
- C2 pad 1: /Vbatt_sense -> +5V
- C48 pad 1: Net-(U1-Pad2) -> Net-(C48-Pad1)
- C49 pad 1: Net-(U1-Pad2) -> Net-(C48-Pad1)
- C49 pad 2: Net-(L1-Pad2) -> Net-(C49-Pad2)
- C50 pad 1: Net-(L1-Pad2) -> Net-(C49-Pad2)
- C51 pad 1: Net-(U14-Pad2) -> Net-(C51-Pad1)
- C52 pad 1: Net-(U14-Pad2) -> Net-(C51-Pad1)
- C52 pad 2: Net-(L2-Pad2) -> Net-(C52-Pad2)
- C53 pad 1: Net-(L2-Pad2) -> Net-(C52-Pad2)
- D7 pad 1: Net-(U1-Pad2) -> Net-(C49-Pad2)
- D7 pad 2: Net-(L1-Pad2) -> Net-(C48-Pad1)
- D9 pad 1: Net-(U14-Pad2) -> Net-(C52-Pad2)
- D9 pad 2: Net-(L2-Pad2) -> Net-(C51-Pad1)
- J4 pad 4: unconnected-(J4-Pad4) -> /SPI1_SCK
- J4 pad 5: unconnected-(J4-Pad5) -> /SPI1_MISO
- J4 pad 6: unconnected-(J4-Pad6) -> /SPI1_MOSI
- J4 pad 7: /DISP4 -> /SPI1_CS2
- J4 pad 8: /DISP5 -> /I2C1_SCL
- J4 pad 9: /DISP6 -> /I2C1_SDA
- L1 pad 2: Net-(L1-Pad2) -> Net-(C49-Pad2)
- L2 pad 2: Net-(L2-Pad2) -> Net-(C52-Pad2)
- L3 pad 2: Net-(U1-Pad2) -> Net-(C48-Pad1)
- L4 pad 2: Net-(U14-Pad2) -> Net-(C51-Pad1)
- P1 pad 1: GND -> /L_LSU_Heater-
- P1 pad 10: unconnected-(P1-Pad10) -> /L_LSU_Rtrim
- P1 pad 11: /L_LSU_Rtrim -> /L_LSU_Vm
- P1 pad 12: /L_LSU_Vm -> /Vout2
- P1 pad 13: unconnected-(P1-Pad13) -> /Vout1
- P1 pad 16: unconnected-(P1-Pad16) -> /R_OD
- P1 pad 17: unconnected-(P1-Pad17) -> GND
- P1 pad 18: unconnected-(P1-Pad18) -> /L_EGT-
- P1 pad 2: 12V_RAW -> /L_LSU_Un
- P1 pad 20: /L_EGT- -> /CAN_H
- P1 pad 21: unconnected-(P1-Pad21) -> /CAN_L
- P1 pad 22: /R_EGT+ -> /R_EGT-
- P1 pad 23: /R_EGT- -> /R_EGT+
- P1 pad 24: unconnected-(P1-Pad24) -> 12V_RAW
- P1 pad 3: /L_LSU_Un -> /L_LSU_Ip
- P1 pad 4: /L_LSU_Ip -> /L_AUX
- P1 pad 5: /L_LSU_Heater- -> /R_AUX
- P1 pad 9: unconnected-(P1-Pad9) -> /L_OD
- R14 pad 2: /L_Un_sense -> /LSU analog left/Un_sense
- R15 pad 2: /L_Un_sense -> /LSU analog left/Un_sense
- R27 pad 2: +5V -> GND
- R43 pad 1: 12V_PROT -> +3V3
- R43 pad 2: /Vbatt_sense -> /I2C1_SCL
- R44 pad 1: GND -> +3V3
- R44 pad 2: /Vbatt_sense -> /I2C1_SDA
- R52 pad 2: /l_Heater_sense -> /L_Heater_sense
- R53 pad 2: /l_Heater_sense -> /L_Heater_sense
- R63 pad 2: /R_Un_sense -> /LSU analog right/Un_sense
- R64 pad 2: /R_Un_sense -> /LSU analog right/Un_sense
- U1 pad 2: Net-(U1-Pad2) -> Net-(C48-Pad1)
- U1 pad 3: Net-(L1-Pad2) -> Net-(C49-Pad2)
- U1 pad 6: /SPI1_NSS -> /SPI1_CS0
- U10 pad 7: /R_Un_sense -> /LSU analog right/Un_sense
- U14 pad 2: Net-(U14-Pad2) -> Net-(C51-Pad1)
- U14 pad 3: Net-(L2-Pad2) -> Net-(C52-Pad2)
- U14 pad 6: /EGT right/SPI_CS -> /SPI1_CS1
- U2 pad 10: /L_Vm_sense -> /R_AUX_ADC
- U2 pad 11: /L_Ip_dac -> /R_Ip_dac
- U2 pad 12: /R_Ip_sense -> /L_Ip_dac
- U2 pad 13: /R_Un_3x_sense -> /R_Ip_sense
- U2 pad 14: /R_Un_sense -> /R_Un_3x_sense
- U2 pad 17: /L_Un_sense -> /L_AUX_ADC
- U2 pad 18: /Vbatt_sense -> /L_Heater_sense
- U2 pad 19: /L_Heater_sense -> /R_Heater_sense
- U2 pad 38: /SPI1_NSS -> /SPI1_CS2
- U2 pad 43: /DISP4 -> /R_heater_pwm
- U2 pad 45: /DISP5 -> /I2C1_SCL
- U2 pad 46: /DISP6 -> /I2C1_SDA
- U2 pad 5: unconnected-(U2-Pad5) -> /SPI1_CS0
- U2 pad 6: unconnected-(U2-Pad6) -> /SPI1_CS1
- U3 pad 7: /L_Un_sense -> /LSU analog left/Un_sense
Routing:
- net /L_EGT-: track 0.00 -> 129.9 mm, vias 0 -> 1
- net /Vout1: track 0.00 -> 129.2 mm, vias 0 -> 1
- net /L_EGT+: track 0.00 -> 127.7 mm, vias 0 -> 1
- net /Vout2: track 0.00 -> 127.0 mm, vias 0 -> 1
- net /R_EGT-: track 0.00 -> 124.9 mm, vias 0 -> 1
- net /R_EGT+: track 0.00 -> 122.8 mm, vias 0 -> 1
- net /CAN_H: track 50.8 -> 144.3 mm
- net /CAN_L: track 51.0 -> 144.1 mm
- net GND: track 177.5 -> 254.4 mm, vias 94 -> 99
- net /R_OD: track 0.00 -> 73.1 mm, vias 0 -> 4
- net /UART_RX: track 39.4 -> 110.6 mm
- net +5V: track 108.7 -> 40.0 mm, vias 5 -> 3
- net /SPI1_SCK: track 4.19 -> 70.4 mm, vias 1 -> 4
- net /SPI1_MISO: track 0.00 -> 64.1 mm, vias 0 -> 5
- net /nRESET: track 41.7 -> 102.9 mm, vias 1 -> 2
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- removed copper zone on F.Cu, net /L_LSU_Heater-

Commit message: Progress
Parts:
- removed C12, C19: 100n, Capacitor_SMD:C_0402_1005Metric
- removed R46, R76: 100k 1%, Resistor_SMD:R_0402_1005Metric
- removed R51, R78: 10k 1%, Resistor_SMD:R_0402_1005Metric
- added H1: MountingHole_Pad, MountingHole:MountingHole_2.5mm_Pad_Via, F.Cu at (164.5, 119.3)
- added H2: MountingHole_Pad, MountingHole:MountingHole_2.5mm_Pad_Via, F.Cu at (164.5, 125.3)
- added H3: MountingHole_Pad, MountingHole:MountingHole_2.5mm_Pad_Via, F.Cu at (102.5, 125.3)
- added H4: MountingHole_Pad, MountingHole:MountingHole_2.5mm_Pad_Via, F.Cu at (102.5, 119.3)
- moved R99 62.0 mm to (127.3, 73.0), turned to 90 degrees
- moved R101 57.3 mm to (127.3, 76.1), turned to 90 degrees
- moved R98 52.0 mm to (124.7, 73.0), turned to 90 degrees
- moved J3 41.1 mm to (136.0, 108.3)
- moved J4 37.2 mm to (145.0, 109.9), turned to 90 degrees
- moved R43 35.8 mm to (162.8, 106.8), turned to -90 degrees
- moved R44 35.5 mm to (165.4, 106.8), turned to -90 degrees
- moved J1 27.6 mm to (128.0, 107.1), turned to 90 degrees
- moved C47 24.8 mm to (150.9, 91.2)
- moved C43 18.6 mm to (150.9, 83.4)
- moved C46 18.6 mm to (158.7, 97.4)
- moved C48 18.6 mm to (163.1, 88.7)
- moved C49 18.6 mm to (163.1, 86.7)
- moved C50 18.6 mm to (163.1, 84.7)
- moved C51 18.6 mm to (163.1, 102.7)
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Connections:
- U2 pad 2: /config0 -> /SPI1_CS2
- U2 pad 3: /config1 -> /config0
- U2 pad 38: /SPI1_CS2 -> unconnected-(U2-Pad38)
- U2 pad 4: unconnected-(U2-Pad4) -> /config1
- U2 pad 5: /SPI1_CS0 -> /SPI1_CS1
- U2 pad 6: /SPI1_CS1 -> /SPI1_CS0
Routing:
- net /UART_RX: track 110.6 -> 44.2 mm
- net /UART_TX: track 95.6 -> 35.3 mm
- net /SWCLK: track 78.6 -> 23.4 mm
- net /SWDIO: track 74.1 -> 23.2 mm
- net /I2C1_SDA: track 0.00 -> 42.8 mm, vias 0 -> 2
- net /I2C1_SCL: track 0.00 -> 40.5 mm, vias 0 -> 2
- net /SPI1_CS2: track 0.00 -> 37.4 mm, vias 0 -> 2
- net /R_AUX_ADC: track 0.00 -> 25.9 mm, vias 0 -> 2
- net /Boot0: track 25.3 -> 50.7 mm
- net /L_EGT+: track 127.7 -> 104.0 mm
- net /L_EGT-: track 129.9 -> 107.2 mm
- net /nRESET: track 102.9 -> 80.8 mm
- net /L_AUX_ADC: track 0.00 -> 21.8 mm, vias 0 -> 2
- net /R_EGT-: track 124.9 -> 105.6 mm, vias 1 -> 2
- net /SPI1_CS1: track 47.0 -> 29.3 mm
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Other:
- board size 87 x 106 mm -> 82.4 x 102.3 mm
