File: lambda-x2/egt.kicad_sch (KiCad schematic)
At the start: 17 parts, among them U1 MAX31855KASA

Commit message: Lambda x2 rev1 (#180)
* lambda-x2: revork aux outputs, remove useless protection in LSU

* lambda-x2: switch to 64-pin MCU

* lambda-x2: add HSE, move pump to DAC outputs

* lambda-x2: move BT to UART4/USART3

* lambda-x2: ocsillator fix

* lambda-x2: fix RC filter values on heater voltage ADC inputs

* lambda-x2: fuse, Vbat sense, resistor in sense

* lambda-x2: diagnostic for AUX out, PWM noise cancelation, etc

* lambda-x2: jtag, adc channels, one more led, BT en, etc

* lambda-x2: update PCB dimentions, connector footprint, etx

* lambda-x2: update

* lambda-x2: final update, rev1

* lambda-x2: rev1: fabrication files
Parts:
- U1: value MAX31855KASA -> (none); footprint Package_SO:SOIC-8_3.9x4.9mm_P1.27mm -> (none); LCSC (none) -> C52028
- U15: value (none) -> MAX31856; footprint (none) -> Package_SO:TSSOP-14_4.4x5mm_P0.65mm
Changed lines of the file:
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@@
       (effects (font (size 1.27 1.27)) (justify left))
     )
-    (property "Value" "MAX31855KASA" (id 1) (at 82.0294 34.29 0)
+    (property "Value" "" (id 1) (at 82.0294 34.29 0)
       (effects (font (size 1.27 1.27)) (justify left))
     )
-    (property "Footprint" "Package_SO:SOIC-8_3.9x4.9mm_P1.27mm" (id 2) (at 105.41 53.34 0)
+    (property "Footprint" "" (id 2) (at 105.41 53.34 0)
       (effects (font (size 1.27 1.27) italic) hide)
     )
     (property "Datasheet" "http://datasheets.maximintegrated.com/en/ds/MAX31855.pdf" (id 3) (at 80.01 44.45 0)
+      (effects (font (size 1.27 1.27)) hide)
+    )
+    (property "LCSC" "C52028" (id 4) (at 80.01 44.45 0)
       (effects (font (size 1.27 1.27)) hide)
     )
@@
       (effects (font (size 1.27 1.27)) (justify left))
     )
-    (property "Value" "" (id 1) (at 83.2994 88.9 0)
+    (property "Value" "MAX31856" (id 1) (at 83.2994 88.9 0)
       (effects (font (size 1.27 1.27)) (justify left))
     )
-    (property "Footprint" "" (id 2) (at 82.55 118.11 0)
+    (property "Footprint" "Package_SO:TSSOP-14_4.4x5mm_P0.65mm" (id 2) (at 82.55 118.11 0)
       (effects (font (size 1.27 1.27)) (justify left) hide)
     )
