File: quad-igbt/quad-igbt.kicad_pcb (KiCad board)
At the start: 2 copper layers, 31 x 57 mm, 21 parts, among them P1 Pad, P2 Pad, P3 Pad, P4 Pad, P5 Pad, P6 Pad, P7 Pad, P8 Pad, P9 Pad, Q1 ISL9V3040D3S, Q2 ISL9V3040D3S, Q3 ISL9V3040D3S, Q4 ISL9V3040D3S

Commit message: logo+export
Parts:
- added G***: LOGO, rusefi_lib:mre_logo, B.Cu at (212.1, 119.9)
- added J1: Conn_01x01, MountingHole:MountingHole_5mm, F.Cu at (196.0, 100.0)
- added J2: Conn_01x01, MountingHole:MountingHole_5mm, F.Cu at (196.0, 151.0)
- added J3: Conn_01x01, MountingHole:MountingHole_5mm, F.Cu at (221.0, 100.0)
- added J4: Conn_01x01, MountingHole:MountingHole_5mm, F.Cu at (221.0, 151.0)
