File: quad-igbt/quad-igbt.kicad_sch (KiCad schematic)
At the start: 21 parts, among them P1 Pad, P2 Pad, P3 Pad, P4 Pad, P5 Pad, P6 Pad, P7 Pad, P8 Pad, P9 Pad, Q1 ISL9V3040D3S, Q2 ISL9V3040D3S, Q3 ISL9V3040D3S, Q4 ISL9V3040D3S

Commit message: logo+export
Parts:
- added J1, J2, J3, J4: Conn_01x01, MountingHole:MountingHole_5mm, symbol Connector_Generic:Conn_01x01
Changed lines of the file:
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@@
     (pin "1")
+  )
+  (symbol (lib_name "Conn_01x01_1") (lib_id "Connector_Generic:Conn_01x01") (at 210.82 161.29 180) (unit 1)
+    (in_bom yes) (on_board yes)
+    (property "Reference" "J3" (id 0) (at 209.55 161.29 0)
+      (effects (font (size 1.27 1.27)) (justify left))
+    )
+    (property "Value" "Conn_01x01" (id 1) (at 212.852 162.5346 0)
+      (effects (font (size 1.27 1.27)) (justify left) hide)
+    )
+    (property "Footprint" "MountingHole:MountingHole_5mm" (id 2) (at 210.82 161.29 0)
+      (effects (font (size 1.27 1.27)) hide)
+    )
+    (property "Datasheet" "~" (id 3) (at 210.82 161.29 0)
+      (effects (font (size 1.27 1.27)) hide)
+    )
+  )
+  (symbol (lib_name "Conn_01x01_1") (lib_id "Connector_Generic:Conn_01x01") (at 210.82 165.1 180) (unit 1)
+    (in_bom yes) (on_board yes)
+    (property "Reference" "J4" (id 0) (at 209.55 165.1 0)
+      (effects (font (size 1.27 1.27)) (justify left))
+    )
+    (property "Value" "Conn_01x01" (id 1) (at 212.852 166.3446 0)
+      (effects (font (size 1.27 1.27)) (justify left) hide)
+    )
+    (property "Footprint" "MountingHole:MountingHole_5mm" (id 2) (at 210.82 165.1 0)
+      (effects (font (size 1.27 1.27)) hide)
+    )
+    (property "Datasheet" "~" (id 3) (at 210.82 165.1 0)
+      (effects (font (size 1.27 1.27)) hide)
+    )
   )
   (symbol (lib_name "Res_1") (lib_id "hellen-one-common:Res") (at 132.08 91.44 180) (unit 1)
@@
     (pin "2")
   )
+  (symbol (lib_name "Conn_01x01_1") (lib_id "Connector_Generic:Conn_01x01") (at 210.82 157.48 180) (unit 1)
+    (in_bom yes) (on_board yes)
+    (property "Reference" "J2" (id 0) (at 209.55 157.48 0)
+      (effects (font (size 1.27 1.27)) (justify left))
+    )
+    (property "Value" "Conn_01x01" (id 1) (at 212.852 158.7246 0)
+      (effects (font (size 1.27 1.27)) (justify left) hide)
+    )
+    (property "Footprint" "MountingHole:MountingHole_5mm" (id 2) (at 210.82 157.48 0)
+      (effects (font (size 1.27 1.27)) hide)
+    )
+    (property "Datasheet" "~" (id 3) (at 210.82 157.48 0)
+      (effects (font (size 1.27 1.27)) hide)
+    )
+  )
   (symbol (lib_id "hellen-one-common:Pad") (at 114.3 91.44 0) (mirror y) (unit 1)
     (in_bom yes) (on_board yes)
@@
     (pin "1")
   )
+  (symbol (lib_name "Conn_01x01_1") (lib_id "Connector_Generic:Conn_01x01") (at 210.82 153.67 180) (unit 1)
+    (in_bom yes) (on_board yes)
+    (property "Reference" "J1" (id 0) (at 209.55 153.67 0)
+      (effects (font (size 1.27 1.27)) (justify left))
+    )
+    (property "Value" "Conn_01x01" (id 1) (at 212.852 154.9146 0)
+      (effects (font (size 1.27 1.27)) (justify left) hide)
+    )
+    (property "Footprint" "MountingHole:MountingHole_5mm" (id 2) (at 210.82 153.67 0)
+      (effects (font (size 1.27 1.27)) hide)
+    )
+    (property "Datasheet" "~" (id 3) (at 210.82 153.67 0)
+      (effects (font (size 1.27 1.27)) hide)
+    )
+  )
   (symbol (lib_id "power:GND") (at 148.59 99.06 0) (mirror y) (unit 1)
     (in_bom yes) (on_board yes)
@@
       (reference "#PWR0104") (unit 1) (value "GND") (footprint "")
     )
+    (path "/cf38b252-15b3-47cf-a195-57c8cf943175"
+      (reference "J1") (unit 1) (value "Conn_01x01") (footprint "MountingHole:MountingHole_5mm")
+    )
+    (path "/7247004c-171d-4a1b-ac09-209b906f44e2"
+      (reference "J2") (unit 1) (value "Conn_01x01") (footprint "MountingHole:MountingHole_5mm")
+    )
+    (path "/29309ac9-7e80-43ee-b1be-d347d31ed2f2"
+      (reference "J3") (unit 1) (value "Conn_01x01") (footprint "MountingHole:MountingHole_5mm")
+    )
+    (path "/2c3888d1-262d-4fd7-8b6d-7ddcd8ab4c86"
+      (reference "J4") (unit 1) (value "Conn_01x01") (footprint "MountingHole:MountingHole_5mm")
+    )
     (path "/03346a1b-c58d-41cb-989c-2c53ae0e733d"
