File: breakout-boards/Breakout_154pin_284617-1-Connector/284617-1.kicad_pcb (KiCad board)
At the start: 2 copper layers, 150 x 51.8 mm, 27 parts, among them P1 284617-1, P10 CONN_5, P11 CONN_9, P12 CONN_5, P13 CONN_9, P14 CONN_22, P15 CONN_22, P16 CONN_22, P17 CONN_22, P18 CONN_1, P19 CONN_1, P2 CONN_1, P20 CONN_1, P21 CONN_1, P22 CONN_1, P23 CONN_1, P24 CONN_1, P25 CONN_1, P3 CONN_1, P4 CONN_1, P5 CONN_1, P6 CONN_5, P7 CONN_9, P8 CONN_5, P9 CONN_9

Commit message: added Breakout_154pin_284617-1 v0.4 #160
Parts:
- moved P13 3.56 mm to (121.1, 113.0)
- moved P11 3.50 mm to (121.1, 109.0)
- moved P9 3.45 mm to (121.1, 105.0)
- moved P7 3.41 mm to (121.1, 101.0)
- moved P12 1.24 mm to (99.1, 113.0)
- moved P5 1.24 mm to (135.9, 113.0)
- moved P10 1.05 mm to (99.1, 109.0)
- moved P4 1.05 mm to (135.9, 109.0)
- moved P3 0.86 mm to (135.9, 105.0)
- moved P8 0.86 mm to (99.1, 105.0)
- moved P14 0.85 mm to (187.4, 101.0)
- moved P2 0.67 mm to (135.9, 101.0)
- moved P6 0.67 mm to (99.1, 101.0)
- moved P15 0.59 mm to (188.4, 105.0)
- moved P16 0.48 mm to (188.4, 109.0)
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Routing:
- net N-0000022: track 36.9 -> 41.6 mm
- net N-00000136: track 133.7 -> 136.9 mm
- net N-0000061: track 104.5 -> 107.2 mm
- net N-00000100: track 15.0 -> 12.4 mm
- net N-0000030: track 91.3 -> 93.8 mm
- net N-0000073: track 12.2 -> 14.6 mm
- net N-00000122: track 88.6 -> 91.0 mm
- net N-00000120: track 74.9 -> 77.2 mm
- net N-0000026: track 65.0 -> 67.1 mm
- net N-0000064: track 90.4 -> 92.4 mm
- net N-0000062: track 112.1 -> 114.0 mm
- net N-0000016: track 29.3 -> 31.3 mm
- net N-0000024: track 52.0 -> 50.0 mm
- net N-00000109: track 61.6 -> 63.6 mm
- net N-0000065: track 82.3 -> 84.2 mm
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Other:
- net class 1.5A removed
- net class 1A removed
- net class 4A removed
- net class Default removed
- board text added: "11"
- board text added: "12"
- board text added: "13"
- board text added: "14"
- board text added: "17"
- board text added: "19"
- board text added: "21"
- board text added: "22"
- board text added: "23"
- board text added: "24"
- board text added: "25"
- board text added: "26"
- board text added: "27"
- board text added: "32"
- board text added: "33"
- board text added: "34"
- board text added: "36"
- board text added: "37"
- board text added: "38"
- board text added: "39"
- board text added: "40"
- board text added: "41"
- board text added: "42"
- board text added: "43"
- board text added: "44"
- board text added: "47"
- board text added: "48"
- board text added: "49"
- board text added: "52"
- board text added: "53"
- board text added: "54"
- board text added: "56"
- board text added: "57"
- board text added: "58"
- board text added: "59"
- board text added: "61"
- board text added: "62"
- board text added: "63"
- board text added: "64"
- board text added: "65"
- board text added: "67"
- board text added: "68"
- board text added: "69"
- board text added: "70"
- board text added: "71"
- board text added: "74"
- board text added: "75"
- board text added: "76"
- board text added: "77"
- board text added: "78"
- board text added: "79"
- board text added: "8"
- board text added: "80"
- board text added: "81"
- board text added: "82"
- board text added: "83"
- board text added: "84"
- board text added: "85"
- board text added: "86"
- board text added: "87"
- board text added: "88"
- board text added: "9"
- board text added: "90"
- board text added: "91"
- board text added: "92"
- board text added: "93"
- board text added: "Connector 154pin rev0.4"
- board text removed: "Connector 154pin rev0.3"
