File: breakout-boards/Breakout_154pin_284617-1-Connector/284617-1.kicad_pcb (KiCad board)
At the start: 2 copper layers, 150 x 51.8 mm, 27 parts, among them P1 284617-1, P10 CONN_5, P11 CONN_9, P12 CONN_5, P13 CONN_9, P14 CONN_22, P15 CONN_22, P16 CONN_22, P17 CONN_22, P18 CONN_1, P19 CONN_1, P2 CONN_1, P20 CONN_1, P21 CONN_1, P22 CONN_1, P23 CONN_1, P24 CONN_1, P25 CONN_1, P3 CONN_1, P4 CONN_1, P5 CONN_1, P6 CONN_5, P7 CONN_9, P8 CONN_5, P9 CONN_9

Commit message: #218
Routing:
- net N-00000136: track 136.9 -> 46.3 mm
- net N-00000128: track 55.3 -> 63.7 mm
- net N-00000125: track 78.7 -> 83.7 mm
- net N-0000073: track 14.6 -> 16.8 mm
- net N-0000037: track 21.6 -> 23.4 mm
- net N-0000023: track 43.6 -> 44.8 mm
Other:
- board text added: "Connector 154pin rev0.5"
- board text removed: "Connector 154pin rev0.4"
