File: breakout-boards/Breakout-24pin/24pins_In_3conn.kicad_pcb (KiCad board)
At the start: 2 copper layers, 63 x 50 mm, 10 parts, among them J1 DB125-2.54-8P-GN-S, J2 DB125-2.54-8P-GN-S, J3 DB125-2.54-8P-GN-S, P1 33311-24AW-2

Commit message: #260
Parts:
- moved H3 2.00 mm to (64.0, 96.0)
- moved H4 2.00 mm to (119.0, 96.0)
- moved P1 0.27 mm to (78.5, 106.5)
Routing:
- net Net-(J1-Pad8): track 64.5 -> 88.2 mm
- net Net-(J1-Pad5): track 66.0 -> 49.7 mm
- net Net-(J1-Pad7): track 54.5 -> 60.1 mm
- net Net-(J1-Pad4): track 61.8 -> 57.9 mm
- net Net-(J1-Pad3): track 54.2 -> 51.3 mm
- net Net-(J1-Pad2): track 50.5 -> 47.9 mm
- net Net-(J1-Pad6): track 50.5 -> 52.9 mm
- net Net-(J1-Pad1): track 45.3 -> 42.9 mm
Other:
- board size 63 x 50 mm -> 63 x 48 mm

Commit message: #260
v 0.2
Other:
- board text added: "24pins_In_3conn rev 0.2"
- board text removed: "24pins_In_3conn rev 0.1"
Changed lines of the file:
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@@
     (effects (font (size 1 1) (thickness 0.15)) (justify mirror))
   )
-  (gr_text "24pins_In_3conn rev 0.1" (at 81.684286 111.9) (layer "B.SilkS")
+  (gr_text "24pins_In_3conn rev 0.2" (at 81.684286 111.9) (layer "B.SilkS")
     (effects (font (size 2 2) (thickness 0.2)) (justify mirror))
   )
@@
     (effects (font (size 1 1) (thickness 0.15)))
   )
-  (gr_text "24pins_In_3conn rev 0.1" (at 100.61 111.8) (layer "F.SilkS")
+  (gr_text "24pins_In_3conn rev 0.2" (at 100.61 111.8) (layer "F.SilkS")
     (effects (font (size 2 2) (thickness 0.2)))
   )
