File: tle9104-breakout/tle9104-breakout.kicad_pcb (KiCad board)
At the start: 4 copper layers, 34.5 x 42.2 mm, 20 parts, among them J1 Conn_01x13, J2 Conn_01x03_Female, J3 Conn_01x03_Female, J4 Conn_01x13, J5 Conn_01x03_Female, U1 TLE9104SH

Commit message: #261
kicad7
Other:
- net class Default removed

Commit message: #261
Connections:
- J5 pad 2: Net-(J5-Pad2) -> unconnected-(J5-Pin_2-Pad2)
