File: GDI-6ch/GDI-6ch.kicad_pcb (KiCad board)
At the start: 4 copper layers, 154 x 160 mm, 280 parts, among them J1 Conn_02x02_Odd_Even, J10 Conn_01x01, J2 FTSH-107-01-F-DV-K, J3 TC2030, J4 Conn_01x06, J5 Conn_01x04, J6 Conn_01x01, J7 Conn_01x01, J8 Conn_01x01, J9 Conn_01x01, P1 368255-2, P10 Pad, P18 Pad, P19 Pad, P2 Pad, P20 Pad, P3 Pad, P32 Pad, P36 Pad, P4 Pad, P5 Pad, P7 Pad, P8 Pad, P9 Pad, Q1 BUK9230-100B, Q10 BUK9230-100B, Q11 BUK9230-100B, Q12 BUK9230-100B, Q13 AOD4185, Q14 VND14NV04TR-E, Q15 VND14NV04TR-E, Q16 BUK9230-100B, Q17 BUK9230-100B, Q18 BUK9230-100B, Q2 BUK9230-100B, Q3 BUK9230-100B, Q4 BUK9230-100B, Q5 BUK9230-100B, Q6 BUK9230-100B, Q7 BUK9230-100B, Q8 BUK9230-100B, Q9 BUK9230-100B, U1 74HC14, U2 TJA1051T-3, U3 LM78M05_TO252, U4 74HC14, U5 XC6206P332MR, U6 MCP6004, U7 STM32F103C8Tx, U8 PT2000, Y2 1MHz

Commit message: Cleanup GDI6
Parts:
- moved R96 32.4 mm to (23.5, 63.7)
Changed lines of the file:
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@@
   )
   (footprint "hellen-one-common:PAD-0805-PAD" placed (layer "F.Cu")
-    (at 41.705391 90.450391)
+    (at 23.5 63.7)
     (property "LCSC" "")
     (property "Sheetfile" "GDI-6ch.kicad_sch")

Commit message: Upd GDI6
Parts:
- added R100: 56k, Resistor_SMD:R_0805_2012Metric, F.Cu at (343.2, 38.6)
- added R101: 56k, Resistor_SMD:R_0805_2012Metric, F.Cu at (347.7, 32.8)
- added R102: 56k, Resistor_SMD:R_0805_2012Metric, F.Cu at (347.7, 35.7)
- added R103: 56k, Resistor_SMD:R_0805_2012Metric, F.Cu at (347.7, 38.6)
- added R104: 56k, Resistor_SMD:R_0805_2012Metric, F.Cu at (352.1, 32.8)
- added R105: 56k, Resistor_SMD:R_0805_2012Metric, F.Cu at (352.1, 35.7)
- added R106: 56k, Resistor_SMD:R_0805_2012Metric, F.Cu at (352.1, 38.6)
- added R97: 56k, Resistor_SMD:R_0805_2012Metric, F.Cu at (343.2, 32.8)
- added R98: 2K, Resistor_SMD:R_1206_3216Metric, F.Cu at (343.9, 45.1)
- added R99: 56k, Resistor_SMD:R_0805_2012Metric, F.Cu at (343.2, 35.7)
- C1, C12, C18, C19, C29, C30, C35, C36, C37, C38, C5, C51, C52, C53, C54, C56, C57, C58, C6, C62, C63, C7, C75, C76, C77, C78, C79, C8, C84, C85, C86, C87, C88, C93, C94, C95, D12, D13, D14, D15, D16, D19, D22, D9, R10, R11, R13, R15, R16, R17, R19, R20, R29, R31, R33, R46, R51, R52, R53, R54, R6, R91, R92, R93: moved to B.Cu
- R45: value 0.01 -> 2K; footprint kicad6-libraries:Shunt_1206 -> Resistor_SMD:R_1206_3216Metric
- moved J1 247.3 mm to (116.5, 171.8)
- moved J2 245.4 mm to (138.1, 159.7)
- moved J3 245.4 mm to (137.7, 166.7)
- moved R45 243.8 mm to (343.9, 41.8), turned to 0 degrees
- moved J4 241.3 mm to (136.8, 151.5)
- moved C12 238.9 mm to (112.8, 163.0), turned to -90 degrees
- moved C78 236.9 mm to (110.2, 160.0), turned to 90 degrees
- moved R44 235.5 mm to (127.8, 172.5), turned to 180 degrees
- moved R55 232.4 mm to (127.8, 170.0), turned to 180 degrees
- moved P4 232.3 mm to (112.0, 151.5)
- moved C75 232.2 mm to (108.8, 160.0)
- moved C77 231.8 mm to (109.8, 163.0), turned to 180 degrees
- moved D20 230.9 mm to (120.7, 164.5)
- moved D21 230.9 mm to (120.7, 161.5)
- moved R23 230.9 mm to (124.2, 161.5)
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Connections:
- C59 pad 2: Net-(C59-Pad2) -> +3V3
- C87 pad 2: Net-(C87-Pad2) -> Net-(RN2-R1.2)
- C88 pad 2: Net-(C88-Pad2) -> Net-(RN2-R2.2)
- D8 pad 1: unconnected-(D8-Pad1) -> Net-(RN2-R2.2)
- D8 pad 3: unconnected-(D8-Pad3) -> Net-(RN2-R1.2)
- R45 pad 1: +3V3 -> /+Batt_filtered
- R45 pad 2: unconnected-(R45-Pad2) -> GND
- R84 pad 2: /L5 -> /L6
- R86 pad 2: /L6 -> /L5
- RN2 pad 7: Net-(C88-Pad2) -> Net-(RN2-R2.2)
- RN2 pad 8: Net-(C87-Pad2) -> Net-(RN2-R1.2)
- U4 pad 11: Net-(C87-Pad2) -> Net-(RN2-R1.2)
- U4 pad 13: Net-(C88-Pad2) -> Net-(RN2-R2.2)
- U8 pad 18: Net-(C59-Pad2) -> +3V3
Routing:
- net /LS1: track 226.2 -> 148.0 mm
- net /LS2: track 188.5 -> 121.9 mm
- net /L7: track 2.05 -> 42.4 mm
- net /H1: track 6.05 -> 27.6 mm, vias 0 -> 1
- net /H3: track 5.55 -> 27.1 mm, vias 0 -> 1
- net /H5: track 0.00 -> 15.4 mm, vias 0 -> 1
- net Net-(Q7-S): track 0.00 -> 14.7 mm, vias 0 -> 1
- net Net-(Q17-S): track 0.00 -> 14.7 mm, vias 0 -> 1
- net Net-(Q10-S): track 0.00 -> 14.7 mm, vias 0 -> 1
- net Net-(Q5-S): track 0.00 -> 11.9 mm, vias 0 -> 1
- net Net-(Q3-S): track 0.00 -> 11.9 mm, vias 0 -> 1
- net Net-(Q1-S): track 0.00 -> 11.9 mm, vias 0 -> 1
- net Vdrive: track 0.00 -> 9.60 mm
- net Net-(Q7-G): track 0.00 -> 5.85 mm
- net Net-(Q18-G): track 0.00 -> 5.85 mm
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Other:
- board text added: "C52"
- board text added: "C53"
- board text added: "C54"
- board text added: "C55"
- board text added: "D10"
- board text added: "D12"
- board text added: "D9"
- board text added: "HS1"
- board text added: "HS2"
- board text added: "HS3"
- board text added: "HS4"
- board text added: "HS5"
- board text added: "HS6"
- board text added: "HS7"
- board text added: "LS3"
- board text added: "LS4"
- board text added: "LS5"
- board text added: "LS6"
- board text added: "LS8"
- board text added: "Q4"
- board text added: "Q7"
- board text added: "Q8"
- board text added: "R10"
- board text added: "R11"
- board text added: "R13"
- board text added: "R14"
- board text added: "R21"
- board text added: "https://rusefi.com GDI-6ch rev.a https://rusefi.com/s/gdi6"
- board text removed: "BOOT0"
- board text removed: "CSB FLAG3"
- board text removed: "DBG SCLK"
- board text removed: "DRVEN"
- board text removed: "FLAG1 FLAG0"
- board text removed: "IRQ"
- board text removed: "MISO MOSI"
- board text removed: "RESETB"
- board text removed: "https://rusefi.com GDI-4ch rev.b https://rusefi.com/s/gdi4"

Commit message: Update GDI-6ch.kicad_pcb
Parts:
- C17, C31, C33, C4, C60, C68, C80, R100, R101, R102, R103, R104, R105, R106, R38, R45, R97, R98, R99: moved to B.Cu
- moved R104 218.3 mm to (151.1, 118.0), turned to 180 degrees
- moved R105 217.9 mm to (151.1, 120.0), turned to 180 degrees
- moved R101 215.9 mm to (151.1, 122.0), turned to 180 degrees
- moved R106 215.4 mm to (151.1, 116.0), turned to 180 degrees
- moved R97 212.7 mm to (151.1, 124.0), turned to 180 degrees
- moved R99 212.3 mm to (151.1, 126.0), turned to 180 degrees
- moved R103 210.5 mm to (151.1, 114.0), turned to 180 degrees
- moved R102 210.1 mm to (151.1, 110.0), turned to 180 degrees
- moved R100 205.7 mm to (151.1, 112.0), turned to 180 degrees
- moved R45 174.4 mm to (193.5, 130.0), turned to 180 degrees
- moved R98 174.2 mm to (193.5, 133.0), turned to 180 degrees
- moved G1 148.8 mm to (180.9, 168.0)
- moved C73 76.0 mm to (148.0, 143.0)
- moved R42 75.0 mm to (151.0, 141.8), turned to 90 degrees
- moved C81 74.3 mm to (148.0, 141.0), turned to 180 degrees
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Routing:
- net +BATT: track 0.00 -> 134.3 mm, vias 0 -> 15
- net /L5: track 5.14 -> 126.3 mm, vias 3 -> 6
- net Vdrive: track 9.60 -> 108.5 mm, vias 0 -> 13
- net /H5: track 15.4 -> 111.7 mm, vias 1 -> 3
- net /L6: track 4.21 -> 80.6 mm
- net Net-(U8-G_LS1): track 0.00 -> 70.7 mm, vias 0 -> 3
- net Net-(U8-G_HS1): track 0.00 -> 65.7 mm, vias 0 -> 2
- net Net-(U8-G_LS2): track 0.00 -> 64.5 mm, vias 0 -> 2
- net /H1: track 27.6 -> 90.0 mm, vias 1 -> 2
- net Net-(Q3-S): track 11.9 -> 72.3 mm, vias 1 -> 2
- net /H7: track 2.05 -> 62.4 mm, vias 0 -> 3
- net Net-(U8-G_LS5): track 0.00 -> 48.0 mm, vias 0 -> 3
- net Net-(U8-G_HS5): track 0.00 -> 43.7 mm, vias 0 -> 3
- net /L1: track 7.19 -> 49.7 mm
- net /L3: track 7.19 -> 48.0 mm
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- added copper zone on F.Cu, net +BATT
- added copper zone on F.Cu, net /+Batt_filtered
- added copper zone on F.Cu, net /H7
- added copper zone on F.Cu, net /Vdrive_coil
- added copper zone on F.Cu, net /Vdrive_shunt
- added copper zone on F.Cu, net Vdrive
