File: GDI-STM/GDI-STM.kicad_sch (KiCad schematic)
At the start: 250 parts, among them J1 Conn_02x02_Odd_Even, J10 Conn_01x08, J11 Conn_01x08, J12 Conn_01x04, J2 FTSH-107-01-F-DV-K, J3 TC2030, J4 Conn_01x06, J5 Conn_01x05, J6 Conn_01x01, J7 Conn_01x01, J8 Conn_01x01, J9 Conn_01x01, P1 368255-2, Q1 BUK9230-100B, Q10 BUK9230-100B, Q11 BUK9230-100B, Q12 BUK9230-100B, Q13 AOD4185, Q14 VND14NV04TR-E, Q15 VND14NV04TR-E, Q16 BUK9230-100B, Q17 BUK9230-100B, Q18 BUK9230-100B, Q2 BUK9230-100B, Q3 BUK9230-100B, Q4 BUK9230-100B, Q5 BUK9230-100B, Q6 BUK9230-100B, Q7 BUK9230-100B, Q8 BUK9230-100B, Q9 BUK9230-100B, U1 74HC14, U2 TJA1051T-3, U3 LM78M05_TO252, U4 74HC14, U5 XC6206P332MR, U6 MCP6004, U7 STM32F103C8Tx, U8 PT2000, Y2 1MHz

Commit message: Upd SCH
Parts:
- removed C66, C69, C70, C72, C8: 100n, hellen-one-common:C0603, symbol hellen-one-common:Cap
- removed D18: SRV05-4, Package_TO_SOT_SMD:SOT-23-6, symbol Power_Protection:NUP4202
- removed D5, D6: D_Schottky, Diode_SMD:D_SMA, symbol Device:D_Schottky
- removed J1: Conn_02x02_Odd_Even, Connector_PinHeader_2.54mm:PinHeader_2x02_P2.54mm_Vertical, symbol Connector_Generic:Conn_02x02_Odd_Even
- removed J11: Conn_01x08, Connector_PinHeader_2.54mm:PinHeader_1x08_P2.54mm_Vertical, symbol Connector_Generic:Conn_01x08
- removed J12: Conn_01x04, Connector_PinHeader_2.54mm:PinHeader_1x04_P2.54mm_Vertical, symbol Connector_Generic:Conn_01x04
- removed J2: FTSH-107-01-F-DV-K, Connector_PinHeader_1.27mm:PinHeader_2x07_P1.27mm_Vertical_SMD, symbol Connector_Generic:Conn_02x07_Odd_Even
- removed Q14, Q15: VND14NV04TR-E, Package_TO_SOT_SMD:TO-252-2, symbol semiconductors:VND14NV04TR-E
- removed R28, R30, R32, R5: DNP, Resistor_SMD:R_0603_1608Metric, symbol Device:R
- removed R29, R31, R33, R6: 470K, Resistor_SMD:R_0603_1608Metric, symbol Device:R
- removed R34, R35: 10k, hellen-one-common:R0603, symbol hellen-one-common:Res
- removed R44, R55: DNP, hellen-one-common:PAD-0805-PAD, symbol hellen-one-common:Jumper-Pad-Pad
- removed R46, R47, R48, R49: 6.8K, Resistor_SMD:R_0603_1608Metric, symbol Device:R
- removed R50, R51, R52, R53: 10K, Resistor_SMD:R_0603_1608Metric, symbol Device:R
- removed RN3: 10k, Resistor_SMD:R_Array_Convex_4x0603, symbol Device:R_Pack04
- removed U6: MCP6004, Package_SO:TSSOP-14_4.4x5mm_P0.65mm, symbol Amplifier_Operational:MCP6004
- removed U7: STM32F103C8Tx, Package_QFP:LQFP-48_7x7mm_P0.5mm, symbol MCU_ST_STM32F1:STM32F103C6Tx
- added C163: 100n, hellen-one-common:C0603, symbol hellen-one-common:Cap
- added U23: STM32G474M_B-C-E_Tx, Package_QFP:LQFP-80_12x12mm_P0.5mm, symbol MCU_ST_STM32G4:STM32G474M_B-C-E_Tx
Connections:
- net +3V3: now also C163.2, U23.1 (VBAT), U23.16 (VDD), U23.29 (VDDA), U23.41 (VDD), U23.51 (VDD), U23.62 (VDD), U23.80 (VDD)
- net GND: now also C163.1
- net LED_GREEN: no longer names the net of D21.2 (A)
- new net: U23.15 (VSS), U23.40 (VSS), U23.50 (VSS), U23.61 (VSS), U23.79 (VSS)
- no-connect marks 88 -> 84
Other:
- added sheet BANK2 (bank.kicad_sch)
- added sheet BANK3 (bank.kicad_sch)
- added sheet BANK4 (bank.kicad_sch)
- sheet BANK1 ports: added H1, H2, HS_VBAT, HS_VBOOST, Isense+, Isense-, L1, L2, LS1, LS2, REF, Vsense1, Vsense2; removed none
- note removed: "Debug"
- note removed: "LED2"
- note removed: "UART / +5 / GND for integration"
- moved on the sheet: C10, C11, C12, C13, C14, C15, C16, C17, C2, C20, C21, C22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

Commit message: Upd GDI-STM
Parts:
- removed R100, R101, R102, R103, R104, R105, R106, R97, R99: 56k, Resistor_SMD:R_0805_2012Metric, symbol Device:R
- removed R45, R98: 2K, Resistor_SMD:R_1206_3216Metric, symbol Device:R
Other:
- added sheet BOOST (boost.kicad_sch)
- sheet BANK1 ports: added VinM, VinP, Vo; removed Isense+, Isense-
- sheet BANK2 ports: added VinM, VinP, Vo; removed Isense+, Isense-
- sheet BANK3 ports: added VinM, VinP, Vo; removed Isense+, Isense-
- sheet BANK4 ports: added VinM, VinP, Vo; removed Isense+, Isense-
- note removed: "Discharge circuit"

Commit message: Upd PCB
Parts:
- removed C10, C11, C13, C24, C60, C73, C99: 330p, hellen-one-common:C0603, symbol hellen-one-common:Cap
- removed C14, C15, C16, C21, C22, C25, C27, C83: 470uF, Capacitor_THT:CP_Radial_D16.0mm_P7.50mm, symbol Device:C_Polarized_US
- removed C17, C80, C81, C82: 0.22uF, Capacitor_SMD:C_0805_2012Metric, symbol Device:C
- removed C26: 4.7u, hellen-one-common:C0603, symbol hellen-one-common:Cap
- removed C32, C34, C59: 100n, hellen-one-common:C0603, symbol hellen-one-common:Cap
- removed C39, C40, C41, C42, C64, C97, C98: 0.33uF, Capacitor_SMD:C_0603_1608Metric, symbol Device:C
- removed C43, C44, C45, C46, C47, C48, C49, C50, C65, C67, C89, C90, C91, C92: 4700p, hellen-one-common:C0603, symbol hellen-one-common:Cap
- removed C52, C53, C54, C55, C56, C57, C58, C61, C62, C63, C71, C93, C94, C95, C96: 1000pF, Capacitor_SMD:C_0603_1608Metric, symbol Device:C
- removed C74: 470p, hellen-one-common:C0603, symbol hellen-one-common:Cap
- removed C9: 1u, hellen-one-common:C0603, symbol hellen-one-common:Cap
- removed D10, D11, D17: SBR10200CTL, Package_TO_SOT_SMD:TO-252-2, symbol Device:D_Schottky_Dual_CommonCathode_AKA
- removed D12, D13, D14, D15, D16, D19, D22, D9: STPS2H100UY, Diode_SMD:D_SMB, symbol Device:D_Schottky_Small
- removed D31: LED_Small, LED_SMD:LED_0805_2012Metric, symbol Device:LED_Small
- removed D34: STTH802G-TR, Package_TO_SOT_SMD:TO-263-2, symbol Device:D_Schottky_AKA
- removed J10: Conn_01x08, Connector_PinHeader_2.54mm:PinHeader_1x08_P2.54mm_Vertical, symbol Connector_Generic:Conn_01x08
- removed L1: 6.8uH, Inductor_SMD:L_Wuerth_HCI-1350, symbol Device:L
- removed L2: 10uH, Inductor_SMD:L_Vishay_IHLP-6767, symbol Device:L
- removed Q1, Q10, Q11, Q12, Q16, Q17, Q18, Q2, Q3, Q4, Q5, Q6, Q7, Q8, Q9: BUK9230-100B, Package_TO_SOT_SMD:TO-252-2, symbol Device:Q_NMOS_GDS
- removed R10, R11, R13, R14, R15, R16, R17, R18, R19, R20, R24, R91, R92, R93, R94: 10, Resistor_SMD:R_0603_1608Metric, symbol Device:R
- removed R12, R21, R22, R26, R90: 0.01, kicad6-libraries:Shunt_1206, symbol Device:R_Shunt
- removed R2: 10k, hellen-one-common:R0603, symbol hellen-one-common:Res
- removed R38, R42: 5.1, Resistor_SMD:R_0603_1608Metric, symbol Device:R
- removed R43: 75K, Resistor_SMD:R_0603_1608Metric, symbol Device:R
- removed R60, R80, R81, R82, R83, R95, R96: DNP, hellen-one-common:PAD-0805-PAD, symbol hellen-one-common:Jumper-Pad-Pad
- removed U8: PT2000, kicad6-libraries:LQFP-80-1EP_12x12mm_P0.5mm, symbol chips:PT2000
- removed Y2: 1MHz, Oscillator:Oscillator_SMD_Diodes_FN-4Pin_7.0x5.0mm, symbol Oscillator:ABLNO
- added C119, C29: 100n, hellen-one-common:C0603, symbol hellen-one-common:Cap
- added C27: 12p, hellen-one-common:C0603, symbol hellen-one-common:Cap
- added R2: 10K, Resistor_SMD:R_0603_1608Metric, symbol Device:R
- added U5: REF2033, Package_TO_SOT_SMD:SOT-23-5, symbol Reference_Voltage:REF2033
- added Y1: 20MHz, Crystal:Crystal_SMD_5032-2Pin_5.0x3.2mm, symbol Device:Crystal
- C28: value 100n -> 12p; LCSC C14663 -> C38523
- D10: renamed from D21; LCSC C965804 -> C12624
- D11: renamed from D20; value BLUE -> RED; LCSC C497940 -> C2286
- F1: value 10A -> 20A; LCSC C136354 -> C136357
- G1: now left out of the parts list
- J5: now not fitted; now left out of the parts list
- U4: renamed from U5; footprint Package_TO_SOT_SMD:SOT-23 -> Package_TO_SOT_SMD:SOT-23-3
- renumbered C4 to C1, C31 to C10, C86 to C11, C1 to C12, C33 to C13, C30 to C14, C87 to C15, C35 to C16, C88 to C17, C36 to C18, C37 to C19, C5 to C2, C38 to C20, C51 to C21, C68 to C22, C2 to C24, C3 to C25, C20 to C26, C84 to C3, C12 to C30, C75 to C31, C76 to C32, C77 to C33, C78 to C34, C79 to C35, C163 to C36, C6 to C4, C85 to C5, C7 to C6, C18 to C7, C19 to C8, C29 to C9, D28 to D5, D32 to D6, D33 to D7, D7 to D8, D8 to D9, J6 to J1, J8 to J2, J7 to J3, J9 to J4, J3 to J6, J4 to J7, Q13 to Q1, R27 to R10, R36 to R11, R39 to R12, R40 to R13, R23 to R14, R9 to R15, R54 to R16, R88 to R4, R4 to R5, R89 to R6, R25 to R9, U3 to U1, U1 to U2, U4 to U3, U2 to U6, U23 to U7
Connections:
- net VCCP is gone; now on an unnamed net: C28.2
- net +5V: now also C23.2, U5.3 (EN), U5.4 (IN)
- net +BATT: no longer C23.2
- net BANK1/REF: now also C119.2, U5.1 (Vbias)
- net Boot0: now also U7.77 (PB8)
- net CAN_RX: now also U7.59 (PA11)
- net CAN_TX: now also U7.60 (PA12)
- net GND: now also U7.15 (VSS), U7.27 (VSSA), U7.40 (VSS), U7.50 (VSS), U7.61 (VSS), U7.79 (VSS), C119.1, C27.2, C29.1, R2.1, U5.2 (GND)
- net H1: no longer P1.121
- net H3: no longer P1.96, P1.97
- net H5: no longer P1.120
- net IN_PUMP2: now also P1.40
- net START1: now also U7.57 (PA9)
- net START2: now also U7.58 (PA10)
- net START3: now also U7.72 (PB3)
- net START4: now also U7.73 (PB4)
- net START5: now also U7.65 (PA15)
- net START6: now also U7.74 (PB5)
- net START7: now also U7.75 (PB6)
- net START8: now also U7.78 (PB9)
- net SWCLK: now also U7.64 (PA14)
- net SWDIO: now also U7.63 (PA13)
- net VinM1: now also U7.23 (PC5)
- net VinM2: now also U7.19 (PA5)
- net VinM3: now also U7.26 (PB2)
- net VinM4: now also U7.39 (PB10)
- net VinP1: now also U7.21 (PA7)
- net VinP2: now also U7.24 (PB0)
- net VinP3: now also U7.44 (PB13)
- net VinP4: now also U7.42 (PB11)
- net Vinj1: now also U7.8 (PC0)
- net Vinj2: now also U7.9 (PC1)
- net Vinj3: now also U7.10 (PC2)
- net Vinj4: now also U7.12 (PA0)
- net Vinj5: now also U7.13 (PA1)
- net Vinj6: now also U7.17 (PA3)
- net Vinj7: now also U7.18 (PA4)
- net Vinj8: now also U7.22 (PC4)
- net Vo1: now also U7.14 (PA2)
- net Vo2: now also U7.20 (PA6)
- net Vo3: now also U7.25 (PB1)
- net Vo4: now also U7.43 (PB12)
- net nRESET: now also U7.7 (PG10)
- net at D4.2 (A), Q1.1 (G): now also R2.2
- net H8: now reaches P1.86
- net H8: now also P1.87
- net L8: now reaches P1.88
- net L8: now also P1.89
- net +12V_C: now reaches F1.1, P1.4
- net at D11.2 (A): now also U7.4 (PC15)
- net at D10.2 (A): now also U7.3 (PC14)
- net VinPboost: now reaches U7.11 (PC3)
- net HS_VBOOST4: now reaches U7.2 (PC13)
- net at U7.28 (VREF+): now also C29.2, U5.5 (Vref)
- net Vboost: now reaches U7.30 (PE7)
- net INJ1: now reaches U7.31 (PE8)
- net INJ2: now reaches U7.32 (PE9)
- net INJ3: now reaches U7.33 (PE10)
- net INJ4: now reaches U7.34 (PE11)
- net INJ5: now reaches U7.35 (PE12)
- net INJ6: now reaches U7.36 (PE13)
- net INJ7: now reaches U7.37 (PE14)
- net INJ8: now reaches U7.38 (PE15)
- net VinMboost: now reaches U7.46 (PB15)
- net at U7.5 (PF0): now also C27.1, Y1.2
- net HS_VBAT1: now reaches U7.52 (PC6)
- net HS_VBAT2: now reaches U7.53 (PC7)
- net HS_VBAT3: now reaches U7.54 (PC8)
- net HS_VBAT4: now reaches U7.55 (PC9)
- net Voboost: now reaches U7.56 (PA8)
- net at U7.6 (PF1): now also Y1.1
- net HS_VBOOST1: now reaches U7.66 (PC10)
- net HS_VBOOST2: now reaches U7.67 (PC11)
- net HS_VBOOST3: now reaches U7.68 (PC12)
- net BOOST_PWM: now reaches U7.69 (PD0)
- net IN_A0: no longer names the net of P1.6
- net IN_A1: no longer names the net of P1.7
- net IN_A2: no longer names the net of P1.8
- net IN_A3: no longer names the net of P1.9
- net OUT_LS1: no longer names the net of P1.21
- net OUT_LS1: no longer P1.22
- net OUT_LS2: no longer names the net of P1.23
- net OUT_LS2: no longer P1.24
- new net H2: P1.121
- new net H4: P1.96, P1.97
- new net H6: P1.120
- no-connect marks 84 -> 94
Other:
- note removed: "Cap height 17mm"
- note removed: "INJECTOR BANK 1"
- note removed: "INJECTOR BANK 2"
- note removed: "INJECTOR BANK 3"
- note removed: "LED1"
- note removed: "Non-JLC: EEE-TP1K391V"
- note removed: "PUMP BANK"
- title: GDI 6ch -> GDI-STM
- moved on the sheet: C1, C10, C13, C22, C24, C25, C26, D1, D10, D11, D2, D3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
