File: GDI-STM/boost.kicad_sch (KiCad schematic)
At the start: 38 parts, among them Q33 IPB107N20N3G, U21 IRS21867S

Commit message: Upd PCB
Parts:
- Q18: renamed from Q33; symbol Device:Q_NMOS_GDS -> Transistor_FET:Q_NMOS_GDS
- renumbered C170 to C105, C168 to C106, C160 to C107, C159 to C108, C161 to C109, C153 to C110, C164 to C111, C162 to C112, C154 to C113, C157 to C114, C171 to C115, C156 to C116, C158 to C117, C155 to C118, D41 to D32, L4 to L1, L3 to L2, R124 to R100, R106 to R101, R123 to R102, R122 to R103, R128 to R85, R129 to R86, R45 to R87, R97 to R88, R125 to R89, R98 to R90, R99 to R91, R100 to R92, R101 to R93, R127 to R94, R102 to R95, R103 to R96, R126 to R97, R104 to R98, R105 to R99, U21 to U24
Other:
- title: GDI 6ch -> GDI-STM
