File: uaBrain-gm-e38/HS5.kicad_sch (KiCad schematic)
At the start: 30 parts, among them U10 BSP762TXUMA1, U5 BSP762TXUMA1, U6 BSP762TXUMA1, U8 BSP762TXUMA1, U9 BSP762TXUMA1

Commit message: Upd SCH
Parts:
- renumbered R33 to R36, R36 to R37, R37 to R38, R38 to R39, R39 to R40, R40 to R41, R41 to R42, R42 to R43, R43 to R44, R44 to R45, R45 to R46, R46 to R47, R47 to R48, R50 to R49, R51 to R50, U8 to U7, U9 to U8, U10 to U9

Commit message: uaBrain-e38 rev a
Changed lines of the file:
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@@
 			)
 		)
-		(property "Description" ""
+		(property "Description" "Unpolarized capacitor, small symbol"
 			(at 115.57 156.21 0)
 			(hide yes)
@@
 			)
 		)
-		(property "Description" ""
+		(property "Description" "Unpolarized capacitor, small symbol"
 			(at 115.57 36.83 0)
 			(hide yes)
@@
 			)
 		)
-		(property "Description" ""
+		(property "Description" "Unpolarized capacitor, small symbol"
 			(at 115.57 127 0)
 			(hide yes)
@@
 			)
 		)
-		(property "Description" ""
+		(property "Description" "Unpolarized capacitor, small symbol"
 			(at 115.57 68.58 0)
 			(hide yes)
@@
 			)
 		)
-		(property "Description" ""
+		(property "Description" "Unpolarized capacitor, small symbol"
 			(at 115.57 97.79 0)
 			(hide yes)
