File: uaBrain-gm-e38/i2c-adc.kicad_sch (KiCad schematic)
At the start: 58 parts, among them U1 MCP6004, U2 MCP6004, U3 ADS7128

Commit message: Upd SCH
Parts:
- renumbered C17 to C10, C12 to C11, C18 to C12, C19 to C14, C14 to C15, C20 to C16, C15 to C17, C21 to C18, C9 to C19, C6 to C2, C7 to C20, C8 to C21, C2 to C3, C10 to C4, C3 to C5, C11 to C6, C4 to C7, C16 to C8, C5 to C9, R19 to R10, R20 to R11, R3 to R12, R2 to R13, R21 to R14, R22 to R15, R5 to R16, R8 to R17, R23 to R18, R24 to R19, R9 to R20, R10 to R21, R11 to R22, R12 to R23, R25 to R24, R26 to R25, R27 to R26, R28 to R27, R13 to R28, R16 to R29, R17 to R30, R18 to R31, R29 to R32, R30 to R33, R31 to R34, R32 to R35, R7 to R4, R6 to R5, R14 to R6, R15 to R7, R1 to R8, R4 to R9, U1 to U2, U2 to U3, U3 to U4

Commit message: uaBrain-e38 rev a
Parts:
- D1, D2: LCSC C85364 -> C6454456
- R10, R12, R16, R6, R8: now not fitted
- R11, R13, R17, R7, R9: value 470k -> 680k; LCSC C23178 -> C25822
- R14: value DNP -> 10k; LCSC (none) -> C15401
- R15, R19, R5: value 470k -> DNP; LCSC C23178 -> (none); now not fitted
- R18, R4: value DNP -> 4.7k; LCSC (none) -> C23162
- U2, U3: LCSC C248577 -> C50282
Connections:
- net ADC0: no longer R20.2, R4.1, R5.2
- net ADC1: no longer R21.2, R8.1, R9.2
- net ADC2: no longer R12.1, R13.2, R22.2
- net ADC3: no longer R16.1, R17.2, R23.2
- net ADC4: no longer R24.2, R6.1, R7.2
- net ADC5: no longer R10.1, R11.2, R25.2
- net ADC6: no longer R14.1, R15.2, R26.2
- net ADC7: no longer R18.1, R19.2, R27.2
- net GND renamed GNDA
- new net IN_ADC0: R20.2, R4.1, R5.2
- new net IN_ADC1: R21.2, R8.1, R9.2
- new net IN_ADC2: R12.1, R13.2, R22.2
- new net IN_ADC3: R16.1, R17.2, R23.2
- new net IN_ADC4: R24.2, R6.1, R7.2
- new net IN_ADC5: R10.1, R11.2, R25.2
- new net IN_ADC6: R14.1, R15.2, R26.2
- new net IN_ADC7: R18.1, R19.2, R27.2
Other:
- moved on the sheet: R14, R18
