File: uaBrain-gm-e38/ls6.kicad_sch (KiCad schematic)
At the start: 15 parts, among them U10 VNLD5160TR-E, U11 VNLD5160TR-E, U12 VNLD5160TR-E

Commit message: Upd SCH
Parts:
- renumbered R51 to R63, R52 to R64, R53 to R65, R54 to R66, R55 to R67, R56 to R68, R57 to R69, R58 to R70, R59 to R71, R60 to R72, R61 to R73, R62 to R74, U10 to U13, U11 to U14, U12 to U15
Connections:
- net IN2: now reaches R64.1, R70.2
- net IN6: now reaches R68.1, R74.2
- net IN1: now reaches R63.1, R69.2
- net IN5: now reaches R67.1, R73.2
- net IN4: now reaches R66.1, R72.2
- net OUT2: now reaches U13.6 (D2)
- net OUT1: now reaches U13.8 (D1)
- net IN3: now reaches R65.1, R71.2
- net OUT6: now reaches U15.6 (D2)
- net OUT5: now reaches U15.8 (D1)
- net OUT4: now reaches U14.6 (D2)
- net OUT3: now reaches U14.8 (D1)
Changed lines of the file:
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@@
+		)
+	)
+	(hierarchical_label "OUT2"
+		(shape output)
+		(at 88.9 77.47 180)
+		(effects
+			(font
+				(size 1.27 1.27)
+			)
+			(justify right)
+		)
+	)
+	(hierarchical_label "IN1"
+		(shape input)
+		(at 162.56 72.39 0)
+		(effects
+			(font
+				(size 1.27 1.27)
+			)
+			(justify left)
+		)
+	)
+	(hierarchical_label "OUT1"
+		(shape output)
+		(at 88.9 72.39 180)
+		(effects
+			(font
+				(size 1.27 1.27)
+			)
+			(justify right)
+		)
+	)
+	(hierarchical_label "OUT4"
+		(shape output)
+		(at 88.9 97.79 180)
+		(effects
+			(font
+				(size 1.27 1.27)
+			)
+			(justify right)
+		)
+	)
+	(hierarchical_label "IN5"
+		(shape input)
+		(at 162.56 113.03 0)
+		(effects
+			(font
+				(size 1.27 1.27)
+			)
+			(justify left)
+		)
+	)
+	(hierarchical_label "OUT3"
+		(shape output)
+		(at 88.9 92.71 180)
+		(effects
+			(font
+				(size 1.27 1.27)
+			)
+			(justify right)
+		)
+	)
+	(hierarchical_label "OUT6"
+		(shape output)
+		(at 88.9 118.11 180)
+		(effects
+			(font
+				(size 1.27 1.27)
+			)
+			(justify right)
+		)
+	)
+	(hierarchical_label "IN6"
+		(shape input)
+		(at 162.56 118.11 0)
+		(effects
+			(font
+				(size 1.27 1.27)
+			)
+			(justify left)
+		)
+	)
+	(hierarchical_label "OUT5"
+		(shape output)
+		(at 88.9 113.03 180)
+		(effects
+			(font
+				(size 1.27 1.27)
+			)
+			(justify right)
+		)
+	)
+	(hierarchical_label "IN3"
+		(shape input)
+		(at 162.56 92.71 0)
+		(effects
+			(font
+				(size 1.27 1.27)
+			)
+			(justify left)
+		)
+	)
+	(hierarchical_label "IN4"
+		(shape input)
+		(at 162.56 97.79 0)
+		(effects
+			(font
+				(size 1.27 1.27)
+			)
+			(justify left)
+		)
+	)
+	(hierarchical_label "IN2"
+		(shape input)
+		(at 162.56 77.47 0)
+		(effects
+			(font
+				(size 1.27 1.27)
+			)
+			(justify left)
 		)
 	)
@@
 		(in_pos_files yes)
 		(dnp no)
-		(property "Reference" "R58"
+		(property "Reference" "R70"
 			(at 146.05 73.66 0)
 			(show_name no)
@@
 		(in_pos_files yes)
 		(dnp no)
-		(property "Reference" "#PWR0166"
+		(property "Reference" "#PWR0175"
 			(at 104.14 88.9 0)
 			(hide yes)
@@
 		(in_pos_files yes)
 		(dnp no)
-		(property "Reference" "R56"
+		(property "Reference" "R68"
 			(at 139.7 115.57 0)
 			(show_name no)
@@
 		(in_pos_files yes)
 		(dnp no)
-		(property "Reference" "#PWR0167"
+		(property "Reference" "#PWR0176"
 			(at 104.14 109.22 0)
 			(hide yes)
@@
 		(in_pos_files yes)
 		(dnp no)
-		(property "Reference" "#PWR0172"
+		(property "Reference" "#PWR0181"
 			(at 162.56 95.25 0)
 			(hide yes)
@@
 		(in_pos_files yes)
 		(dnp no)
-		(property "Reference" "R51"
+		(property "Reference" "R63"
 			(at 139.7 69.85 0)
 			(show_name no)
@@
 		(in_pos_files yes)
 		(dnp no)
-		(property "Reference" "R55"
+		(property "Reference" "R67"
 			(at 139.7 110.49 0)
 			(show_name no)
@@
 		(in_pos_files yes)
 		(dnp no)
-		(property "Reference" "#PWR0169"
+		(property "Reference" "#PWR0178"
 			(at 162.56 69.85 0)
 			(hide yes)
@@
 		(in_pos_files yes)
 		(dnp no)
-		(property "Reference" "#PWR0168"
+		(property "Reference" "#PWR0177"
 			(at 104.14 129.54 0)
 			(hide yes)
@@
 		(in_pos_files yes)
 		(dnp no)
-		(property "Reference" "R57"
+		(property "Reference" "R69"
 			(at 146.05 68.58 0)
 			(show_name no)
@@
 		(in_pos_files yes)
 		(dnp no)
-		(property "Reference" "R60"
+		(property "Reference" "R72"
 			(at 146.05 93.98 0)
 			(show_name no)
@@
 		(in_pos_files yes)
 		(dnp no)
-		(property "Reference" "U10"
+		(property "Reference" "U13"
 			(at 120.65 64.77 0)
 			(show_name no)
@@
 		(in_pos_files yes)
 		(dnp no)
-		(property "Reference" "R54"
+		(property "Reference" "R66"
 			(at 139.7 95.25 0)
 			(show_name no)
@@
 		(in_pos_files yes)
 		(dnp no)
-		(property "Reference" "R62"
+		(property "Reference" "R74"
 			(at 146.05 114.3 0)
 			(show_name no)
@@
 		(in_pos_files yes)
 		(dnp no)
-		(property "Reference" "R52"
+		(property "Reference" "R64"
 			(at 139.7 74.93 0)
 			(show_name no)
@@
 		(in_pos_files yes)
 		(dnp no)
-		(property "Reference" "R53"
+		(property "Reference" "R65"
 			(at 139.7 90.17 0)
 			(show_name no)
@@
 		(in_pos_files yes)
 		(dnp no)
-		(property "Reference" "#PWR0173"
+		(property "Reference" "#PWR0182"
 			(at 162.56 110.49 0)
 			(hide yes)
@@
 		(in_pos_files yes)
 		(dnp no)
-		(property "Reference" "#PWR0174"
+		(property "Reference" "#PWR0183"
 			(at 162.56 115.57 0)
 			(hide yes)
@@
 		(in_pos_files yes)
 		(dnp no)
-		(property "Reference" "R59"
+		(property "Reference" "R71"
 			(at 146.05 88.9 0)
 			(show_name no)
@@
 		(in_pos_files yes)
 		(dnp no)
-		(property "Reference" "#PWR0170"
+		(property "Reference" "#PWR0179"
 			(at 162.56 74.93 0)
 			(hide yes)
@@
 		(in_pos_files yes)
 		(dnp no)
-		(property "Reference" "R61"
+		(property "Reference" "R73"
 			(at 146.05 109.22 0)
 			(show_name no)
@@
 		(in_pos_files yes)
 		(dnp no)
-		(property "Reference" "U12"
+		(property "Reference" "U15"
 			(at 120.65 105.41 0)
 			(show_name no)
@@
 		(in_pos_files yes)
 		(dnp no)
-		(property "Reference" "U11"
+		(property "Reference" "U14"
 			(at 120.65 85.09 0)
 			(show_name no)
@@
 		(in_pos_files yes)
 		(dnp no)
-		(property "Reference" "#PWR0171"
+		(property "Reference" "#PWR0180"
 			(at 162.56 90.17 0)
 			(hide yes)
