File: uaBrain-gm-e38/uaBrain-gm-e38.kicad_sch (KiCad schematic)
At the start: 3 parts, among them J1 Molex_313874018 80-pin grey, J2 Molex_313872014 73-pin black, M1 hw-uaBrain

Commit message: Upd SCH
Parts:
- added J10: 5569-16A2, Connector_Molex:Molex_Mini-Fit_Jr_5569-16A2_2x08_P4.20mm_Horizontal, symbol Connector_Generic:Conn_02x08_Top_Bottom
- added J3, J4: 5569-06A2, Connector_Molex:Molex_Mini-Fit_Jr_5569-06A2_2x03_P4.20mm_Horizontal, symbol Connector_Generic:Conn_02x03_Top_Bottom
- added J5: 5569-04A2, Connector_Molex:Molex_Mini-Fit_Jr_5569-04A2_2x02_P4.20mm_Horizontal, symbol Connector_Generic:Conn_02x02_Top_Bottom
- added unit 2 of M1
- added unit 3 of M1
- added R34, R35, R48, R49: 4.7k, hellen-one-common:R0603, symbol hellen-one-common:Res
- added U4: PCA9685PW, Package_SO:TSSOP-28_4.4x9.7mm_P0.65mm, symbol Driver_LED:PCA9685PW
- added U7: VNLD5160TR-E, Package_SO:SOIC-8_3.9x4.9mm_P1.27mm, symbol chips:VNLD5160
- J1: value Molex_313874018 80-pin grey -> Molex_313874018_singleside; symbol e38-connectors:Molex_313874018_singleside -> Molex_313874018_80pin_Connector:Molex_313874018_singleside
- J2: value Molex_313872014 73-pin black -> Molex_313872014_singleside; symbol e38-connectors:Molex_313872014_singleside -> Molex_313872014_73pin_Connector:Molex_313872014_singleside
Connections:
- net +12V: now also J2.47, M1.M1 (+12V); no longer J2.20, M1.M1 (+12V)
- net +12V_RAW: now also J3.1 (Pin_1), J4.1 (Pin_1), J5.3 (Pin_3), M1.H6 (+12V_RAW); no longer J2.47, M1.H6 (+12V_RAW)
- net +5VP: now also M1.E5 (+5VP), M1.F4 (+5VP), M1.F7 (+5VP), M1.K5 (+5VP), M1.L3 (+5VP), M1.N3 (+5VP), M1.P7 (+5VP); no longer M1.E5 (+5VP), M1.F4 (+5VP), M1.F7 (+5VP), M1.K5 (+5VP), M1.L3 (+5VP), M1.N3 (+5VP), M1.P7 (+5VP)
- net 12V_KEY: now also M1.M2 (12V_KEY); no longer M1.M2 (12V_KEY)
- net CAN_H: now also M1.N5 (CAN1+); no longer M1.N5 (CAN1+)
- net CAN_L: now also M1.N6 (CAN1-); no longer M1.N6 (CAN1-)
- net GND: now also J5.4 (Pin_4), M1.G8 (GND), M1.K3 (GND), M1.K8 (GND), M1.M3 (GND), M1.M4 (GND), M1.P5 (GND), R34.1, R35.1, U4.1 (A0), U4.14 (VSS), U4.2 (A1), U4.23 (~{OE}), U4.24 (A5), U4.25 (EXTCLK), U4.3 (A2), U4.4 (A3), U4.5 (A4), U7.5 (S2), U7.7 (S1); no longer J2.72, M1.G8 (GND), M1.K3 (GND), M1.K8 (GND), M1.M3 (GND), M1.M4 (GND), M1.P5 (GND)
- net GNDA: now also M1.E6 (GNDA), M1.E8 (GNDA), M1.F5 (GNDA), M1.F8 (GNDA), M1.G2 (GNDA), M1.J8 (GNDA), M1.K6 (GNDA), M1.L4 (GNDA), M1.N4 (GNDA), M1.P8 (GNDA); no longer M1.E6 (GNDA), M1.E8 (GNDA), M1.F5 (GNDA), M1.F8 (GNDA), M1.G2 (GNDA), M1.J8 (GNDA), M1.K6 (GNDA), M1.L4 (GNDA), M1.N4 (GNDA), M1.P8 (GNDA)
- net IN_CAM: now also M1.G3 (IN_HALL2); no longer M1.G3 (IN_HALL2)
- net IN_CLT: now also M1.E7 (IN_CLT); no longer M1.E7 (IN_CLT)
- net IN_CLUTCH_SWITCH: now also M1.N8 (IN_BUTTON2); no longer M1.N8 (IN_BUTTON2)
- net IN_DIN1: now also M1.P6 (IN_FLEX); no longer M1.P6 (IN_FLEX)
- net IN_IAT: now also M1.G1 (IN_IAT); no longer M1.G1 (IN_IAT)
- net IN_KNOCK2: now also M1.J7 (IN_KNOCK2_RAW); no longer M1.J7 (IN_KNOCK2_RAW)
- net IN_MAF: now also M1.F3 (IN_AUX2); no longer M1.F3 (IN_AUX2)
- net IN_MAP: now also M1.F6 (IN_MAP); no longer M1.F6 (IN_MAP)
- net IN_P/N_SWITCH: now also M1.L2 (IN_BUTTON3); no longer M1.L2 (IN_BUTTON3)
- net IN_PPS1: now also M1.N1 (IN_PPS1); no longer M1.N1 (IN_PPS1)
- net IN_PPS2: now also M1.N2 (IN_PPS2); no longer M1.N2 (IN_PPS2)
- net IN_STOP_SWITCH: now also M1.N7 (IN_BUTTON1); no longer M1.N7 (IN_BUTTON1)
- net IN_TPS1: now also M1.E3 (IN_TPS1); no longer M1.E3 (IN_TPS1)
- net IN_TPS2: now also M1.E4 (IN_TPS2); no longer M1.E4 (IN_TPS2)
- net IN_VSS+: now also M1.C2 (VR_DISCRETE+); no longer M1.K4 (IN_HALL3)
- net OUT_BK1S1HTR: no longer M1.M5 (OUT_LS9)
- net OUT_BK2S1HTR: no longer M1.M6 (OUT_LS10)
- net OUT_CHECK_ENGINE: now also M1.K7 (OUT_LS5); no longer M1.K7 (OUT_LS5)
- net OUT_ETB+: now also M1.E2 (OUT_DC1+); no longer M1.E2 (OUT_DC1+)
- net OUT_ETB-: now also M1.E1 (OUT_DC1-); no longer M1.E1 (OUT_DC1-)
- net OUT_EVAP_PURGE: no longer M1.G6 (OUT_LS7)
- net OUT_FAN1_RELAY: now also M1.M8 (OUT_LS2); no longer M1.M8 (OUT_LS2)
- net OUT_INJ4: now also M1.J4 (OUT_INJ4); no longer M1.J4 (OUT_INJ4)
- net OUT_INJ5: now also M1.J5 (OUT_INJ5); no longer M1.J5 (OUT_INJ5)
- net OUT_INJ6: now also M1.J6 (OUT_INJ6); no longer M1.J6 (OUT_INJ6)
- net OUT_MAIN_RELAY: now also M1.M7 (OUT_LS1); no longer M1.M7 (OUT_LS1)
- net OUT_STARTER_RELAY: now also M1.G7 (OUT_LS8); no longer M1.G7 (OUT_LS8)
- net OUT_TACH: now also M1.L1 (OUT_LS6); no longer M1.L1 (OUT_LS6)
- net IN_AC_PRESSURE: now reaches J2.12
- net IN_PRIM_FUEL_LEVEL: now reaches J2.16
- net IN_FTPS: now reaches J2.24
- net IN_CLUTCH_POSITION: now reaches J2.26
- net OUT_FUEL_PUMP1_RELAY_HS: now reaches J2.50
- net OUT_FUEL_PUMP2_RELAY_HS: now reaches J2.51
- net OUT_STARTER_RELAY_HS: now reaches J2.52
- net OUT_VSS_HS: now reaches J2.57
- net OUT_EVAP_VENT: now reaches J2.61
- net OUT_SKIP_SHIFT_SOLENOID: now reaches J2.66
- net OUT_SKIP_SHIFT_SOLENOID: now also M1.G6 (OUT_LS7)
- net IN_SEC_FUEL_LEVEL: now reaches J2.70
- net IN_REVERSE_SWITCH: now reaches J2.8
- net IN_REVERSE_SWITCH: now also M1.K4 (IN_HALL3)
- net OUT_DOD_CYL1: now reaches J1.10
- net OUT_DOD_CYL2: now reaches J1.11
- net OUT_DOD_CYL4: now reaches J1.14
- net OUT_VVT_HS: now reaches J1.16
- net OUT_INJ8: now reaches J1.17
- net OUT_INJ8: now also M1.M6 (OUT_LS10)
- net IN_ATF_TEMP: now reaches J1.23
- net IN_OIL_LEVEL_SWITCH: now reaches J1.33
- net OUT_INJ7: now reaches J1.40
- net OUT_INJ7: now also M1.M5 (OUT_LS9)
- net IN_BK1S1SIG: now reaches J1.57
- net OUT_ALT_LIGHT: now reaches J1.61
- net OUT_ALT_LIGHT: now also U7.8 (D1)
- net OUT_IGN8_5: now reaches J1.71
- net OUT_IGN8_5: now also J1.75, M1.B2 (OUT_IGN2)
- net OUT_IGN7_4: now reaches J1.72
- net OUT_IGN7_4: now also J1.76, M1.B3 (OUT_IGN3)
- net OUT_DOD_CYL3: now reaches J1.9
- net 6_WBO1_Un: now reaches M1.A1 (6_WBO1_Un)
- net 6_WBO1_Un: now also J3.4 (Pin_4)
- net 5_WBO1_Rtrim: now reaches M1.A2 (5_WBO1_Rtrim)
- net 5_WBO1_Rtrim: now also J3.2 (Pin_2)
- net 1_WBO1_Ip: now reaches M1.A3 (1_WBO1_Ip)
- net 1_WBO1_Ip: now also J3.5 (Pin_5)
- net 2_WBO1_Vm: now reaches M1.A4 (2_WBO1_Vm)
- net 2_WBO1_Vm: now also J3.6 (Pin_6)
- net 3_WBO1_Heater: now reaches M1.A5 (3_WBO1_Heater)
- net 3_WBO1_Heater: now also J3.3 (Pin_3)
- net EGT1-: now reaches M1.A7 (EGT1-)
- net EGT1-: now also J10.13 (Pin_13)
- net EGT1+: now reaches M1.A8 (EGT1+)
- net EGT1+: now also J10.14 (Pin_14)
- net IN_VSS-: now reaches M1.C1 (VR_DISCRETE-)
- net IN_VSS-: now also J2.72
- net +3.3VA: now reaches M1.D5 (+3.3VA)
- net +3.3VA: now also M1.L5 (+3.3VA)
- net +3.3V: now reaches M1.D6 (+3.3V)
- net +3.3V: now also U4.28 (VDD)
- net +5VA: now reaches M1.D7 (+5VA)
- net +5VA: now also M1.L7 (+5VA)
- net +5V: now reaches M1.D8 (+5V)
- net OUT_IGN1 renamed OUT_IGN1_6
- net OUT_IGN1_6: now also J1.74
- net OUT_IGN2 renamed OUT_IGN2_3
- net OUT_IGN2_3: now also J1.77, M1.J1 (OUT_IGN4); no longer M1.B2 (OUT_IGN2)
- removed net OUT_IGN3: J1.77, M1.B3 (OUT_IGN3)
- removed net OUT_IGN4: J1.76, M1.J1 (OUT_IGN4)
- removed net OUT_IGN5: J1.75, M1.J2 (OUT_IGN5)
- removed net OUT_IGN6: J1.74, M1.J3 (OUT_IGN6)
- new net: R48.2, U7.1 (IN1)
- new net: R49.2, U7.3 (IN2)
- new net 1_WBO2_Ip: J4.5 (Pin_5), M1.H3 (1_WBO2_Ip)
- new net 2_WBO2_Vm: J4.6 (Pin_6), M1.H4 (2_WBO2_Vm)
- new net 3_WBO2_Heater: J4.3 (Pin_3), M1.H5 (3_WBO2_Heater)
- new net 5_WBO2_Rtrim: J4.2 (Pin_2), M1.H2 (5_WBO2_Rtrim)
- new net 6_WBO2_Un: J4.4 (Pin_4), M1.H1 (6_WBO2_Un)
- new net ALT_LIGHT: M1.J2 (OUT_IGN5), R34.2, R48.1
- new net AUX_LS1: M1.J3 (OUT_IGN6), R35.2, R49.1
- new net CAN2+: J10.8 (Pin_8), J5.1 (Pin_1), M1.G4 (CAN2+)
- new net CAN2-: J10.7 (Pin_7), J5.2 (Pin_2), M1.G5 (CAN2-)
- new net EGT2+: J10.12 (Pin_12), M1.H8 (EGT2+)
- new net EGT2-: J10.11 (Pin_11), M1.H7 (EGT2-)
- new net HS5/IN1: U4.6 (LED0)
- new net HS5/IN2: U4.7 (LED1)
- new net HS5/IN3: U4.8 (LED2)
- new net HS5/IN4: U4.9 (LED3)
- new net HS5/IN5: U4.10 (LED4)
- new net OUT_AUX_LS1: U7.6 (D2)
- new net OUT_DC2+: J10.16 (Pin_16), M1.F2 (OUT_DC2+)
- new net OUT_DC2-: J10.15 (Pin_15), M1.F1 (OUT_DC2-)
- new net SCL: M1.L8 (SCL), U4.26 (SCL)
- new net SDA: M1.L6 (SDA), U4.27 (SDA)
- new net VR_MAX9924+: J10.10 (Pin_10), M1.K2 (VR_MAX9924+)
- new net VR_MAX9924-: J10.9 (Pin_9), M1.K1 (VR_MAX9924-)
- no-connect marks 106 -> 54
Other:
- added sheet HS5 (HS5.kicad_sch)
- added sheet I2C ADC inputs (i2c-adc.kicad_sch)
- note added: "8 nets | DOD / EVAP / O2"
- note added: "DEFERRED: NOT USED"
- note added: "E"
- note added: "J1.10"
- note added: "J1.11"
- note added: "J1.12"
- note added: "J1.13"
- note added: "J1.14"
- note added: "J1.8"
- note added: "J1.9"
- note added: "J2.61"
- note added: "LOW-SIDE OUTPUTS / O2 HEATERS"
- note added: "LOW-SIDE OUTPUTS / SOLENOIDS"
- note removed: "IN_AC_PRESSURE (E38, unused)"
- note removed: "IN_ATF_TEMP (E38, unused)"
- note removed: "IN_BK1S1SIG (E38, unused)"
- note removed: "IN_CLUTCH_POSITION (E38, unused)"
- note removed: "IN_FTPS (E38, unused)"
- note removed: "IN_OIL_LEVEL_SWITCH (E38, unused)"
- note removed: "IN_PRIM_FUEL_LEVEL (E38, unused)"
- note removed: "IN_REVERSE_SWITCH (E38, unused)"
- note removed: "IN_SEC_FUEL_LEVEL (E38, unused)"
- note removed: "OUT_ALT_LIGHT (E38, unused)"
- note removed: "OUT_DOD_CYL1 (E38, unused)"
- note removed: "OUT_DOD_CYL2 (E38, unused)"
- note removed: "OUT_DOD_CYL3 (E38, unused)"
- note removed: "OUT_DOD_CYL4 (E38, unused)"
- note removed: "OUT_EVAP_VENT (E38, unused)"
- note removed: "OUT_FUEL_PUMP1_RELAY_HS (E38, unused)"
- note removed: "OUT_FUEL_PUMP2_RELAY_HS (E38, unused)"
- note removed: "OUT_IGN7 (E38, unused)"
- note removed: "OUT_IGN8 (E38, unused)"
- note removed: "OUT_INJ7 (E38, unused)"
- note removed: "OUT_INJ8 (E38, unused)"
- note removed: "OUT_SKIP_SHIFT_SOLENOID (E38, unused)"
- note removed: "OUT_STARTER_RELAY_HS (E38, unused)"
- note removed: "OUT_VSS_HS (E38, unused)"
- note removed: "OUT_VVT_HS (E38, unused)"
- note removed: "P1_SPARE (E38, unused)"
- note removed: "uaBrain-gm-e38: hw-uaBrain module on a GM E38 carrier. J1 = 80-pin grey (Molex 31387-4018), J2 = 73-pin black (Molex 31387-2014). Pin functions copied from hellen-gm-e38 rev c; grey text = E38 function not wired to the module."
- moved on the sheet: J1, J2, M1A

Commit message: Upd SCH
Parts:
- removed R34, R35, R48, R49: 4.7k, hellen-one-common:R0603, symbol hellen-one-common:Res
- removed U7: VNLD5160TR-E, Package_SO:SOIC-8_3.9x4.9mm_P1.27mm, symbol chips:VNLD5160
- added R1, R2, R3: 100, Resistor_SMD:R_2512_6332Metric_Pad1.40x3.35mm_HandSolder, symbol hellen-one-common:Res
- M1: footprint kicad6-libraries:hw-uaBrain -> kicad6-libraries:hw-uaBrain-PinHeader
- renumbered J2 to J1, J1 to J2, J10 to J6, U4 to U1
Connections:
- net +5VA: now also R1.1, R2.1, R3.1
- net +5VP: now also J6.2 (Pin_2)
- net CAN2+: no longer J6.8 (Pin_8)
- net CAN2-: no longer J6.7 (Pin_7)
- net GND: now also J6.1 (Pin_1)
- net GNDA: now also J6.3 (Pin_3)
- net IN_BK1S1SIG: now also J6.8 (Pin_8)
- net IN_PRIM_FUEL_LEVEL: now also R1.2
- net IN_SEC_FUEL_LEVEL: now also R2.2
- net OUT_ALT_LIGHT: now also R3.2
- net OUT_CHECK_ENGINE: no longer M1.K7 (OUT_LS5)
- net OUT_DOD_CYL1: now also J6.7 (Pin_7), M1.G7 (OUT_LS8)
- net OUT_DOD_CYL2: now also J6.6 (Pin_6), M1.K7 (OUT_LS5)
- net OUT_DOD_CYL3: now also J6.5 (Pin_5), M1.M7 (OUT_LS1)
- net OUT_DOD_CYL4: now also J6.4 (Pin_4), M1.M8 (OUT_LS2)
- net OUT_FAN1_RELAY: no longer M1.M8 (OUT_LS2)
- net OUT_MAIN_RELAY: no longer M1.M7 (OUT_LS1)
- net OUT_STARTER_RELAY: no longer M1.G7 (OUT_LS8)
- net STARTER_RELAY: now reaches U1.11 (LED5)
- net CHECK_ENGINE: now reaches U1.12 (LED6)
- net EVAP_VENT: now reaches U1.13 (LED7)
- net FAN1_RELAY: now reaches U1.15 (LED8)
- net AUX_LS1 renamed MAIN_RELAY
- net OUT_BK1S1HTR: no longer names the net of J2.12
- net OUT_BK2S1HTR: no longer names the net of J2.13
- net OUT_EVAP_PURGE: no longer names the net of J2.8
- no-connect marks 54 -> 62
Other:
- added sheet LS6 (ls6.kicad_sch)
- note removed: "8 nets | DOD / EVAP / O2"
- note removed: "DEFERRED: NOT USED"
- note removed: "J1.10"
- note removed: "J1.11"
- note removed: "J1.12"
- note removed: "J1.13"
- note removed: "J1.14"
- note removed: "J1.8"
- note removed: "J1.9"
- note removed: "J2.61"
- note removed: "LOW-SIDE OUTPUTS / O2 HEATERS"
- note removed: "LOW-SIDE OUTPUTS / SOLENOIDS"
- moved on the sheet: J5, J6, U1

Commit message: uaBrain-e38 rev a
Parts:
- added C27: 1u, hellen-one-common:C0603, symbol hellen-one-common:Cap
- added H1, H2, H3, H4: M3, MountingHole:MountingHole_3.2mm_M3_Pad_Via, symbol Mechanical:MountingHole_Pad
- added J10, J11, J12, J13, J14, J8, J9: PH2.54-01-16PZD, Connector_PinHeader_2.54mm:PinHeader_1x16_P2.54mm_Vertical, symbol Mechanical:Mechanical_Shape
- added J7: C4201WR-F-2x8P, Connector_Molex:Molex_Mini-Fit_Jr_5569-16A2_2x08_P4.20mm_Horizontal, symbol Connector_Generic:Conn_02x08_Top_Bottom
- J6: value 5569-16A2 -> C4201WR-F-2x8P; LCSC C485577 -> C5355564
- M1: now left out of the parts list
Connections:
- net +3.3V: now also C27.2
- net +5VP: now also J7.2 (Pin_2)
- net GND: now also C27.1, H1.1, H2.1, H3.1, H4.1, J7.1 (Pin_1)
- net GNDA: now also J7.3 (Pin_3)
- net IN_CLUTCH_POSITION: now also J7.5 (Pin_5)
- net IN_CLUTCH_SWITCH: now also J7.4 (Pin_4)
- net IN_MAF: now also J7.15 (Pin_15)
- net IN_P/N_SWITCH: now also J7.6 (Pin_6)
- net IN_PRIM_FUEL_LEVEL: now also J7.14 (Pin_14)
- net IN_REVERSE_SWITCH: now also J7.10 (Pin_10)
- net IN_SEC_FUEL_LEVEL: now also J7.13 (Pin_13)
- net IN_STOP_SWITCH: now also J7.12 (Pin_12)
- net OUT_EVAP_VENT: now also J7.11 (Pin_11)
- net OUT_FUEL_PUMP2_RELAY_HS: now also J7.7 (Pin_7)
- net OUT_SKIP_SHIFT_SOLENOID: now also J7.8 (Pin_8)
- net OUT_TACH: now also J7.9 (Pin_9)
- net IN_DIN1 renamed IN_FLEX
- net IN_FLEX: now also J7.16 (Pin_16)
- net IN_FTPS renamed IN_FUEL_TANK_PRESSURE
Other:
- sheet I2C ADC inputs ports: added IN_ADC0, IN_ADC1, IN_ADC2, IN_ADC3, IN_ADC4, IN_ADC5, IN_ADC6, IN_ADC7; removed ADC0, ADC1, ADC2, ADC3, ADC4, ADC5, ADC6, ADC7
- note added: "M1: A1-A8, B1-B8"
- note added: "M1: C1-C8, D1-D8"
- note added: "M1: E1-E8, F1-F8"
- note added: "M1: G1-G8, H1-H8"
- note added: "M1: J1-J8, K1-K8"
- note added: "M1: L1-L8, M1-M8"
- note added: "M1: N1-N8, P1-P8"
- note added: "uaBrain mounting headers"
